File: design/PCBs/MOTORDRIVER/_autosave-voltageregulatros.kicad_sch (KiCad schematic)
At the start: 35 parts, among them IC15 REF3425TIDBVR, IC2 LD1117S33CTR, IC3 TPS552882RPMR, IC4 BQ24133RGYR, IC5 REF3450TIDBVR

Commit message: more
Other:
- note added: "these might be configured wrong. look at examples, might need op-amp and diff value capacitors"
- moved on the sheet: 100nF, 100nF28, C16, C17, IC15, IC3, IC5, R11, R12, R13
