File: design/PCBs/MOTORDRIVER/microcontroller.kicad_sch (KiCad schematic)
At the start: 14 parts, among them IC1 ATSAME53J18A-MF

Commit message: LED
Parts:
- added ERROR, POWER, PROCESS: LED, symbol Device:LED
- added R21, R22, R23: R, symbol Device:R
Connections:
- net +3.3V: now also R23.1
- net ERR_LED: now also R22.1
- net GND: now also ERROR.1 (K), POWER.1 (K), PROCESS.1 (K)
- new net: POWER.2 (A), R23.2
- new net: PROCESS.2 (A), R21.2
- new net: ERROR.2 (A), R22.2
- new net PROCESS: R21.1
