File: design/PCBs/MOTORDRIVER/motordriver.kicad_sch (KiCad schematic)
At the start: 0 parts

Commit message: documentation, values, double-checking stuff
Other:
- sheet output renamed hall & phases
- sheet output1 renamed external
- sheet external: file output.kicad_sch -> second_output.kicad_sch
- sheet external ports: added ERROR_LED, PROCESS_LED; removed none
- sheet voltageregulators ports: added BATTIN, USBVIN; removed none
- note added: "1.0"
- note added: "2024-12-14"
- note added: "PCB_KUBEN"
- note added: "root"
Changed lines of the file:
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@@
+	(wire
+		(pts
+			(xy 104.14 111.76) (xy 104.14 139.7)
+		)
+		(stroke
+			(width 0)
+			(type default)
+		)
+	)
 	(wire
 		(pts
@@
 	(wire
 		(pts
+			(xy 33.02 25.4) (xy 39.37 25.4)
+		)
+		(stroke
+			(width 0)
+			(type default)
+		)
+	)
+	(wire
+		(pts
 			(xy 208.28 68.58) (xy 265.43 68.58)
 		)
@@
 		(pts
 			(xy 205.74 17.78) (xy 205.74 22.86)
+		)
+		(stroke
+			(width 0)
+			(type default)
+		)
+	)
+	(wire
+		(pts
+			(xy 101.6 111.76) (xy 101.6 139.7)
 		)
 		(stroke
@@
 		(fill
 			(type none)
+		)
+	)
+	(text "1.0"
+		(exclude_from_sim no)
+		(at 270.764 193.548 0)
+		(effects
+			(font
+				(size 1.27 1.27)
+			)
 		)
 	)
@@
 		)
 	)
+	(text "root\n"
+		(exclude_from_sim no)
+		(at 191.008 189.992 0)
+		(effects
+			(font
+				(size 1.27 1.27)
+			)
+		)
+	)
+	(text "PCB_KUBEN\n"
+		(exclude_from_sim no)
+		(at 229.108 175.514 0)
+		(effects
+			(font
+				(size 3.81 3.81)
+			)
+		)
+	)
+	(text "2024-12-14"
+		(exclude_from_sim no)
+		(at 212.344 193.548 0)
+		(effects
+			(font
+				(size 1.27 1.27)
+			)
+		)
+	)
 	(text "Motor Stage"
 		(exclude_from_sim no)
@@
 	(sheet
 		(at 72.39 139.7)
-		(size 54.61 20.32)
+		(size 39.37 20.32)
 		(fields_autoplaced yes)
 		(stroke
@@
 			(color 0 0 0 0.0000)
 		)
-		(property "Sheetname" "output1"
+		(property "Sheetname" "external"
 			(at 71.5046 160.02 90)
 			(effects
@@
 			)
 		)
-		(property "Sheetfile" "output.kicad_sch"
-			(at 127.7584 160.02 90)
+		(property "Sheetfile" "second_output.kicad_sch"
+			(at 112.5184 160.02 90)
 			(effects
 				(font
@@
 		(pin "TX" input
 			(at 91.44 139.7 90)
+			(effects
+				(font
+					(size 1.27 1.27)
+				)
+				(justify right)
+			)
+		)
+		(pin "PROCESS_LED" input
+			(at 104.14 139.7 90)
+			(effects
+				(font
+					(size 1.27 1.27)
+				)
+				(justify right)
+			)
+		)
+		(pin "ERROR_LED" input
+			(at 101.6 139.7 90)
 			(effects
 				(font
@@
 	(sheet
 		(at 19.05 20.32)
-		(size 13.97 170.18)
+		(size 13.97 72.39)
 		(fields_autoplaced yes)
 		(stroke
@@
 		)
 		(property "Sheetfile" "input.kicad_sch"
-			(at 19.05 191.2584 0)
+			(at 19.05 93.4684 0)
 			(effects
 				(font
@@
 	)
 	(sheet
-		(at 45.72 17.78)
+		(at 39.37 19.05)
 		(size 44.45 21.59)
 		(fields_autoplaced yes)
@@
 		)
 		(property "Sheetname" "voltageregulators"
-			(at 45.72 16.8946 0)
+			(at 39.37 18.1646 0)
 			(effects
 				(font
@@
 		)
 		(property "Sheetfile" "voltageregulatros.kicad_sch"
-			(at 45.72 40.1284 0)
+			(at 39.37 41.3984 0)
 			(effects
 				(font
@@
 				)
 				(justify left top)
+			)
+		)
+		(pin "BATTIN" input
+			(at 39.37 25.4 180)
+			(effects
+				(font
+					(size 1.27 1.27)
+				)
+				(justify left)
+			)
+		)
+		(pin "USBVIN" input
+			(at 39.37 27.94 180)
+			(effects
+				(font
+					(size 1.27 1.27)
+				)
+				(justify left)
 			)
 		)
@@
 			(color 0 0 0 0.0000)
 		)
-		(property "Sheetname" "output"
+		(property "Sheetname" "hall & phases"
 			(at 267.97 14.3546 0)
 			(effects
@@
 		)
 		(pin "ERR_LED" input
-			(at 100.33 111.76 270)
+			(at 101.6 111.76 270)
 			(effects
 				(font
@@
 		)
 		(pin "PROCESS_LED" input
-			(at 102.87 111.76 270)
-			(effects
-				(font
+			(at 104.14 111.76 270)
+			(effects
+				(font
