File: design/PCBs/MOTORDRIVER/second_output.kicad_sch (KiCad schematic)
At the start: 8 parts, among them J5 1-84952-1, J6 1-84952-1, J7 1-84952-1

Commit message: documentation, values, double-checking stuff
Parts:
- removed J5, J6, J7: 1-84952-1, 1849521, symbol 1-84952-1:1-84952-1
- added D1, D2, D3: LED, symbol Device:LED
- added R4, R5, R6: 1K, symbol Device:R
- gave numbers to parts that had none: 1
- renumbered S2 to S5, S3 to S6, Screen to Screen1
Connections:
- net +3.3V: now also D3.2 (A), R6.1
- net GND: now also D1.1 (K), D2.1 (K), D3.1 (K), R4.2, R5.2, R6.2
- new net ERROR_LED: D2.2 (A), R4.1
- new net PROCESS_LED: D1.2 (A), R5.1
- no-connect marks 6 -> 0
Other:
- note added: "Power"
- note added: "Signal Controlled"
- note added: "externals"
- note removed: "MP1 & MP2 are mounting pins"
- note removed: "Motor Headers"
- note removed: "hall & phases"
- moved on the sheet: S4, S5, S6, Screen1
