File: design/PCBs/MOTORDRIVER/IO.kicad_sch (KiCad schematic)
At the start: 9 parts, among them J1 IMU1, J2 IMU2, J3 Screw_Terminal_01x02, P1 USB_C_Plug_USB2.0

Commit message: cleaned up
Other:
- note added: "FFC (Flat Flexible Connector) to IMU"
- note added: "Microcontroller debug"
- note added: "Should we connect this directly to 5v (essentially bypassing charging and voltage regulation) or not?"
- note removed: "Debug"
- note removed: "FFC to IMU"
Changed lines of the file:
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@@
 	(text "Dont need SAO pin, because \nwe have 2 sep i2c lines"
 		(exclude_from_sim no)
-		(at 147.066 70.358 0)
+		(at 98.044 73.66 0)
 		(effects
 			(font
@@
 		)
 	)
-	(text "FFC to IMU"
+	(text "FFC (Flat Flexible Connector) to IMU"
 		(exclude_from_sim no)
-		(at 97.79 73.406 0)
+		(at 97.536 69.342 0)
 		(effects
 			(font
@@
 		)
 	)
-	(text "Debug"
+	(text "Microcontroller debug"
 		(exclude_from_sim no)
-		(at 190.754 116.586 0)
+		(at 191.77 117.856 0)
 		(effects
 			(font
@@
 			)
 		)
+	)
+	(text "Should we connect this directly\nto 5v (essentially bypassing \ncharging and\nvoltage regulation) \nor not?"
+		(exclude_from_sim no)
+		(at 48.006 70.104 0)
+		(effects
+			(font
+				(size 1.27 1.27)
+			)
+		)
