File: design/PCBs/MOTORDRIVER/IO.kicad_sch (KiCad schematic)
At the start: 9 parts, among them J1 IMU1, J2 IMU2, J3 Screw_Terminal_01x02, P1 USB_C_Plug_USB2.0

Commit message: looked over
Parts:
- removed DB1: Conn_01x02_Pin, Connector_PinHeader_2.54mm:PinHeader_1x02_P2.54mm_Vertical, symbol Connector:Conn_01x02_Pin
- removed Screen1: Conn_01x04, Connector_PinHeader_2.00mm:PinHeader_1x04_P2.00mm_Horizontal, symbol Connector_Generic:Conn_01x04
- added J3: Conn_01x04_Socket, Connector_PinSocket_2.54mm:PinSocket_1x04_P2.54mm_Vertical, symbol Connector:Conn_01x04_Socket
- added TP1: RX, TestPoint:TestPoint_Pad_D1.5mm, symbol Connector:TestPoint
- added TP2: TX, TestPoint:TestPoint_Pad_D1.5mm, symbol Connector:TestPoint
- added TP3: SWCLK, TestPoint:TestPoint_Pad_D1.5mm, symbol Connector:TestPoint
- added TP4: SWDIO, TestPoint:TestPoint_Pad_D1.5mm, symbol Connector:TestPoint
- J1, J2: footprint kuben_footprints:59453052110ECHLF -> kuben-footprints:59453052110ECHLF
- J4: renamed from J3; footprint kuben_footprints:VN02A1500000G -> kuben-footprints:VN02A1500000G
Connections:
- net +3.3V: now also J3.2 (Pin_2)
- net +5V: no longer P1.A4 (VBUS), P1.A9 (VBUS), P1.B4 (VBUS), P1.B9 (VBUS)
- net GND: now also J3.1 (Pin_1)
- net OLED_SCL: now also J3.4 (Pin_4)
- net OLED_SDA: now also J3.3 (Pin_3)
- net RX: now also TP1.1
- net TX: now also TP2.1
- net BAT_12V renamed BATTVIN
- new net SWCLK: TP3.1
- new net SWDIO: TP4.1
- new net USBVIN: P1.A4 (VBUS), P1.A9 (VBUS), P1.B4 (VBUS), P1.B9 (VBUS)
Other:
- note added: "General IO"
- note added: "Initial programming interface"
- note added: "TODO: Find right connector for battery"
- moved on the sheet: J4

Commit message: worked on schematic
Other:
- note added: "Programming interface"
- note added: "TODO: decide on connector for servo"
- note removed: "Initial programming interface"
Changed lines of the file:
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@@
 		)
 	)
-	(text "Initial programming interface"
+	(text "Programming interface"
 		(exclude_from_sim no)
 		(at 240.538 114.3 0)
@@
 		(effects
 			(font
+				(size 1.27 1.27)
+			)
+		)
+	)
+	(text "TODO: decide on connector for servo"
+		(exclude_from_sim no)
+		(at 149.606 77.47 0)
+		(effects
+			(font

Commit message: worked on schemtaic
Parts:
- added TP5, TP6: GND, TestPoint:TestPoint_Pad_D1.5mm, symbol Connector:TestPoint
Connections:
- net GND: now also TP5.1, TP6.1
Other:
- moved on the sheet: J1, J2, J3, J4, P1, TP1, TP2, TP3, TP4

Commit message: worked on schemtaic
Parts:
- J4: footprint kuben-footprints:VN02A1500000G -> TerminalBlock:TerminalBlock_Altech_AK300-2_P5.00mm
- renumbered TP5 to TP3, TP3 to TP4, TP4 to TP5
Other:
- moved on the sheet: J3, J4, TP1, TP2, TP3, TP4, TP5, TP6

Commit message: worked on schemtac
Parts:
- added R113, R115: 5.1kΩ, Resistor_SMD:R_0603_1608Metric, symbol Device:R
- added SW1: SW_DPST_x2, Button_Switch_THT:SW_CK_JS202011AQN_DPDT_Angled, symbol Switch:SW_DPST_x2
- P1: footprint Connector_USB:USB_C_Receptacle_JAE_DX07S024WJ3R400 -> kuben-footprints:USB4110GFA; symbol Connector:USB_C_Plug_USB2.0 -> USB4110-GF-A:USB4110-GF-A; Height (none) -> 3.26; Manufacturer_Name (none) -> GCT (GLOBAL CONNECTOR TECHNOLOGY); Manufacturer_Part_Number (none) -> USB4110-GF-A; Mouser Part Number (none) -> 640-USB4110-GF-A; Mouser Price/Stock (none) -> https://www.mouser.co.uk/ProductDetail/GCT/USB4110-GF-A?qs=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
Connections:
- net BATTVIN: now also SW1.1 (A); no longer J4.1 (Pin_1)
- net D+: now also P1.B6
- net D-: now also P1.B7
- net GND: now also R113.1, R115.2; no longer P1.S1 (SHIELD)
- net at P1.A5: now also R115.1
- net at P1.B5: now also R113.2
- net SERVO_1_SIGNAL renamed BRAKE1
- net SERVO_2_SIGNAL renamed BRAKE2
- net SERVO_3_SIGNAL renamed BRAKE3
- new net: J4.1 (Pin_1), SW1.2 (B)
- no-connect marks 6 -> 10
Other:
- note removed: "Should we connect this directly to 5v (essentially bypassing charging and voltage regulation) or not?"
- moved on the sheet: J1, J2, J4, TP1, TP2, TP3
