File: design/PCBs/MOTORDRIVER/motordriver.kicad_pcb (KiCad board)
At the start: 2 copper layers, 140 x 105 mm, 235 parts, among them IC1 LM5109BSDX_NOPB, IC10 ATSAME53J18A-MF, IC11 LM5109BSDX_NOPB, IC12 LM5109BSDX_NOPB, IC13 LM5109BSDX_NOPB, IC14 INA2181A2IDGSR, IC15 LM5109BSDX_NOPB, IC16 LM5109BSDX_NOPB, IC17 LM5109BSDX_NOPB, IC18 INA2181A2IDGSR, IC2 LM5109BSDX_NOPB, IC3 LM5109BSDX_NOPB, IC4 INA2181A2IDGSR, IC7 BQ24133RGYR, IC9 LM5176PWPR, J1 IMU1, J2 IMU2, J3 Screw_Terminal_01x02, J4 1-84952-1, J5 1-84952-1, J6 1-84952-1, P1 USB_C_Plug_USB2.0, Q1 DMN3042L-7, Q10 DMN3042L-7, Q11 DMN3042L-7, Q12 DMN3042L-7, Q13 DMN3042L-7, Q14 DMN3042L-7, Q15 DMN3042L-7, Q16 DMN3042L-7, Q17 DMN3042L-7, Q18 DMN3042L-7, Q19 DMN3042L-7, Q2 DMN3042L-7, Q20 DMN3042L-7, Q21 DMN3042L-7, Q22 DMN3042L-7, Q23 DMN3042L-7, Q24 DMN3042L-7, Q25 DMN3042L-7, Q3 DMN3042L-7, Q4 DMN3042L-7, Q5 DMN3042L-7, Q6 DMN3042L-7, Q7 DMN3042L-7, Q8 DMN3042L-7, Q9 DMPH6050SK3-13, U1 TMC4671-LA, U2 ATSAMD11D14A-M, U3 TMC4671-LA, U4 TMC4671-LA, U5 LD1117S25TR_SOT223, U6 LD1117S50TR_SOT223, U7 LD1117S33TR_SOT223

Commit message: looked over
Parts:
- removed 100nF1, 100nF10, 100nF11, 100nF12, 100nF13, 100nF14, 100nF15, 100nF16, 100nF17, 100nF18, 100nF19, 100nF2, 100nF20, 100nF21, 100nF3, 100nF4, 100nF5, 100nF6, 100nF7, 100nF8, 100nF9, 15nF1: C, Capacitor_SMD:C_0603_1608Metric
- removed 10ohm1, 133k1, 240k1: R, Resistor_SMD:R_0603_1608Metric
- removed Bootstrap1, Bootstrap2, Bootstrap3: 0.1µF, Capacitor_SMD:C_0603_1608Metric
- removed the C14 at (215.3, 55.0)
- removed the C14 at (94.4, 112.9)
- removed the C16 at (94.4, 117.9)
- removed the C16 at (215.3, 57.5)
- removed the C19 at (98.4, 100.3)
- removed the C19 at (215.3, 60.0)
- removed the C23 at (215.3, 62.5)
- removed the C23 at (98.4, 110.4)
- removed the C7 at (215.3, 50.0)
- removed the C7 at (90.4, 120.4)
- removed the C8 at (215.3, 52.5)
- removed the C8 at (94.4, 97.8)
- removed Charging1: LED, Diode_SMD:D_0603_1608Metric
- removed DBOOT1, DBOOT2, DBOOT3, DBOOT4, DBOOT5, DBOOT6, DBOOT7: D, Diode_SMD:D_0603_1608Metric
- removed IC16, IC17: LM5109BSDX_NOPB, kuben_footprints:SON80P400X400X80-9N
- removed IC18: INA2181A2IDGSR, kuben_footprints:SOP50P490X110-10N
- removed RBOOT1, RBOOT2, RBOOT3, RBOOT4, RBOOT5, RBOOT6, RBOOT7: 2.2Ω, Resistor_SMD:R_0603_1608Metric
- removed Screen1: Conn_01x04, Connector_PinHeader_2.00mm:PinHeader_1x04_P2.00mm_Horizontal
- added C14: 100nF, Capacitor_SMD:C_0603_1608Metric, F.Cu at (33.7, 41.2)
- added C16: 1µF, Capacitor_SMD:C_0603_1608Metric, F.Cu at (33.7, 46.2)
- added C19: 0.047µF, Capacitor_SMD:C_0603_1608Metric, F.Cu at (37.7, 28.6)
- added C23: 0.1µF, Capacitor_SMD:C_0603_1608Metric, F.Cu at (37.7, 38.6)
- added C7: 0.1µF, Capacitor_SMD:C_0603_1608Metric, F.Cu at (33.7, 23.6)
- added C74: 1µF, Capacitor_SMD:C_0603_1608Metric, B.Cu at (132.0, 151.8)
- added C75: 0.1µF, Capacitor_SMD:C_0603_1608Metric, B.Cu at (129.5, 151.8)
- added C76: 1µF, Capacitor_SMD:C_0603_1608Metric, B.Cu at (127.0, 151.8)
- added C77: 0.1µF, Capacitor_SMD:C_0603_1608Metric, F.Cu at (44.3, 141.5)
- added C78: 1µF, Capacitor_SMD:C_0603_1608Metric, F.Cu at (44.3, 144.0)
- added C79: 0.1µF, Capacitor_SMD:C_0603_1608Metric, F.Cu at (44.3, 146.5)
- added C8: 100nF, Capacitor_SMD:C_0603_1608Metric, F.Cu at (33.7, 26.1)
- added D11: LED, Diode_SMD:D_0603_1608Metric, F.Cu at (137.0, 115.3)
- added D12: LED, Diode_SMD:D_0603_1608Metric, F.Cu at (137.0, 117.8)
- added D13: 470mV 500mA, Diode_SMD:D_0603_1608Metric, B.Cu at (237.9, 51.1)
- added D14: 470mV 500mA, Diode_SMD:D_0603_1608Metric, B.Cu at (237.9, 53.7)
- added D15: 470mV 500mA, Diode_SMD:D_0603_1608Metric, B.Cu at (237.9, 56.3)
- added D16: 470mV 500mA, Diode_SMD:D_0603_1608Metric, B.Cu at (124.4, 151.8)
- added D17: 470mV 500mA, Diode_SMD:D_0603_1608Metric, B.Cu at (121.8, 151.8)
- added D18: 470mV 500mA, Diode_SMD:D_0603_1608Metric, B.Cu at (119.3, 151.8)
- added IC5: BQ24133RGYR, kuben-footprints:BQ24133RGYR, F.Cu at (120.8, 34.2)
- added IC6: LM5176PWPR, kuben-footprints:SOP65P640X120-29N, F.Cu at (134.6, 35.4)
- added IC8: LM5109BSDX_NOPB, kuben-footprints:SON80P400X400X80-9N, B.Cu at (258.9, 69.1)
- added J7: Conn_01x04_Socket, Connector_PinSocket_2.54mm:PinSocket_1x04_P2.54mm_Vertical, F.Cu at (100.0, 81.5)
- added R42: 1kΩ, Resistor_SMD:R_0603_1608Metric, F.Cu at (126.7, 109.0)
- added R43: 1kΩ, Resistor_SMD:R_0603_1608Metric, F.Cu at (126.7, 111.5)
- added R44: 10kΩ, Resistor_SMD:R_0603_1608Metric, F.Cu at (97.4, 38.6)
- added R45: 10kΩ, Resistor_SMD:R_0603_1608Metric, F.Cu at (97.4, 41.2)
- added R46: 6Ω, Resistor_SMD:R_0603_1608Metric, B.Cu at (234.0, 36.0)
- added R47: 4.7Ω, Resistor_SMD:R_0603_1608Metric, B.Cu at (234.0, 38.5)
- added R48: 4.7Ω, Resistor_SMD:R_0603_1608Metric, B.Cu at (234.0, 41.0)
- added R49: 6Ω, Resistor_SMD:R_0603_1608Metric, B.Cu at (234.0, 43.5)
- added R50: 4.7Ω, Resistor_SMD:R_0603_1608Metric, B.Cu at (234.0, 46.0)
- added R51: 4.7Ω, Resistor_SMD:R_0603_1608Metric, B.Cu at (234.0, 48.5)
- added R52: 6Ω, Resistor_SMD:R_0603_1608Metric, B.Cu at (230.0, 36.0)
- added R53: 4.7Ω, Resistor_SMD:R_0603_1608Metric, B.Cu at (230.0, 38.5)
- added R54: 4.7Ω, Resistor_SMD:R_0603_1608Metric, B.Cu at (230.0, 41.0)
- added R55: 0.01Ω, Resistor_SMD:R_0603_1608Metric, B.Cu at (230.0, 43.5)
- added R56: 0.01Ω, Resistor_SMD:R_0603_1608Metric, B.Cu at (230.0, 46.0)
- added R57: 10kΩ, Resistor_SMD:R_0603_1608Metric, B.Cu at (158.8, 169.7)
- added R58: 10kΩ, Resistor_SMD:R_0603_1608Metric, B.Cu at (158.8, 172.2)
- added R59: 6Ω, Resistor_SMD:R_0603_1608Metric, B.Cu at (139.5, 147.8)
- added R60: 4.7Ω, Resistor_SMD:R_0603_1608Metric, B.Cu at (137.0, 147.8)
- added R61: 4.7Ω, Resistor_SMD:R_0603_1608Metric, B.Cu at (134.5, 147.8)
- added R62: 6Ω, Resistor_SMD:R_0603_1608Metric, B.Cu at (132.0, 147.8)
- added R63: 4.7Ω, Resistor_SMD:R_0603_1608Metric, B.Cu at (129.5, 147.8)
- added R64: 4.7Ω, Resistor_SMD:R_0603_1608Metric, B.Cu at (127.0, 147.8)
- added R65: 6Ω, Resistor_SMD:R_0603_1608Metric, B.Cu at (139.5, 143.8)
- added R66: 4.7Ω, Resistor_SMD:R_0603_1608Metric, B.Cu at (137.0, 143.8)
- added R67: 4.7Ω, Resistor_SMD:R_0603_1608Metric, B.Cu at (134.5, 143.8)
- added R68: 0.01Ω, Resistor_SMD:R_0603_1608Metric, B.Cu at (132.0, 143.8)
- added R69: 0.01Ω, Resistor_SMD:R_0603_1608Metric, B.Cu at (129.5, 143.8)
- added TP1: TestPoint, TestPoint:TestPoint_Pad_D1.5mm, F.Cu at (180.0, 115.0)
- added TP2: TestPoint, TestPoint:TestPoint_Pad_D1.5mm, F.Cu at (180.0, 109.0)
- added TP3: TestPoint, TestPoint:TestPoint_Pad_D1.5mm, F.Cu at (172.5, 106.5)
- added TP4: TestPoint, TestPoint:TestPoint_Pad_D1.5mm, F.Cu at (167.5, 106.5)
- C1, C3, C34, C35, C36, C37, C39, C60, C67, C73: moved to B.Cu
- C10: value 0.1µF -> ?F
- C11: value 1µF -> 10uF
- C12: value 1µF -> 10µF
- C13: value 0.047µF -> 0.1µF
- C15: value 1µF -> 0.1µF
- C17: value 0.1µF -> 1µF
- C18: value 0.1µF -> 10uF
- C2, C61: value 0.1µF -> 1µF; moved to B.Cu
- C20, C40: value 10µF -> 100nF
- C21: value 10µF -> 1µF
- C22: value 10nF -> 0.1µF
- C24: value 33nF -> 10uF
- C25: value 470pF -> 10µF
- C26: value 15nF -> 10µF
- C27: value 220pF -> 10nF
- C28: value 270µF -> 33nF
- C29: value 100nF -> 470pF
- C30: value 100nF -> 15nF
- C31: value 100nF -> 220pF
- C32: value 100nF -> 270µF
- C38: value 10µF -> 100nF; moved to B.Cu
- C4: value 2.2µF -> 1µF; moved to B.Cu
- C48: value 4.7µF -> 10µF
- C5: value ?F -> 0.1µF; moved to B.Cu
- C50: value 100nF -> 10µF
- C52: value 100nF -> 4.7µF
- C56, C57, C58: value 0.1µF -> 100nF
- C59, C68, C69, C70, C71, C72: value 0.1µF -> 100nF; moved to B.Cu
- C6: value 10µF -> 1µF; moved to B.Cu
- C62, C64, C66: value 100nF -> 0.1µF; moved to B.Cu
- C63, C65: value 100nF -> 1µF; moved to B.Cu
- C9: value 0.1µF -> 2.2µF
- D1: value D -> 470mV 500mA; moved to B.Cu
- D10: value D -> 470mV 500mA
- D2, D3: value BZV55B2V4 -> 470mV 500mA; footprint Diode_SMD:D_MiniMELF -> Diode_SMD:D_0603_1608Metric; moved to B.Cu
- D4: value 470mV 500mA -> BZV55B2V4; footprint Diode_SMD:D_0603_1608Metric -> Diode_SMD:D_MiniMELF
- D5: value LED -> BZV55B2V4; footprint Diode_SMD:D_0603_1608Metric -> Diode_SMD:D_MiniMELF
- D6: value 385mV 500mA -> LED
- D9: value LED -> 385mV 500mA
- IC1, IC12, IC13, IC2, IC3: footprint kuben_footprints:SON80P400X400X80-9N -> kuben-footprints:SON80P400X400X80-9N; moved to B.Cu
- IC10: value ATSAME53J18A-MF -> LM5109BSDX_NOPB; footprint kuben_footprints:QFN50P900X900X100-65N-D -> kuben-footprints:SON80P400X400X80-9N; moved to B.Cu
- IC11, IC15: value LM5109BSDX_NOPB -> INA2181A2IDGSR; footprint kuben_footprints:SON80P400X400X80-9N -> kuben-footprints:SOP50P490X110-10N; moved to B.Cu
- IC14: value INA2181A2IDGSR -> LM5109BSDX_NOPB; footprint kuben_footprints:SOP50P490X110-10N -> kuben-footprints:SON80P400X400X80-9N; moved to B.Cu
- IC4: footprint kuben_footprints:SOP50P490X110-10N -> kuben-footprints:SOP50P490X110-10N; moved to B.Cu
- IC7: value BQ24133RGYR -> ATSAME53J18A-MF; footprint kuben_footprints:BQ24133RGYR -> kuben-footprints:QFN50P900X900X100-65N-D
- IC9: value LM5176PWPR -> LM5109BSDX_NOPB; footprint kuben_footprints:SOP65P640X120-29N -> kuben-footprints:SON80P400X400X80-9N; moved to B.Cu
- J1, J2: footprint kuben_footprints:59453052110ECHLF -> kuben-footprints:59453052110ECHLF; moved to B.Cu
- J3: footprint kuben_footprints:VN02A1500000G -> kuben-footprints:VN02A1500000G
- J4, J5, J6: footprint kuben_footprints:1849521 -> kuben-footprints:1849521; moved to B.Cu
- Q1, Q14, Q15, Q16, Q17, Q18, Q19, Q2, Q20, Q21, Q22, Q23, Q24, Q25, Q3, Q4, Q5, Q6: footprint kuben_footprints:SOT96P240X115-3N -> kuben-footprints:SOT96P240X115-3N; moved to B.Cu
- Q10, Q11, Q12, Q13, Q7, Q8: footprint kuben_footprints:SOT96P240X115-3N -> kuben-footprints:SOT96P240X115-3N
- Q9: footprint kuben_footprints:DMPH6050SK313 -> kuben-footprints:DMPH6050SK313
- R1: value 2.2Ω -> 6Ω; moved to B.Cu
- R10: value 5.23kΩ -> 0.01Ω; moved to B.Cu
- R11: value 30.1kΩ -> 0.01Ω; moved to B.Cu
- R12: value 4.02kΩ -> 10Ω
- R13: value 20mΩ -> 2Ω
- R14: value 232kΩ -> 1MΩ
- R15: value 32.4kΩ -> 100kΩ
- R16: value 100kΩ -> 1.5kΩ
- R17: value 32.4kΩ -> 4.02kΩ
- R18: value 1kΩ -> 5.23kΩ
- R19: value 10MΩ -> 30.1kΩ
- R2, R3: value 0.01Ω -> 4.7Ω; moved to B.Cu
- R20: value 10Ω -> 4.02kΩ
- R21: value 240kΩ -> 20mΩ
- R22: value 133kΩ -> 232kΩ
- R23: value 93.1kΩ -> 32.4kΩ
- R24: value 23.2kΩ -> 100kΩ
- R25: value 280kΩ -> 32.4kΩ
- R26: value 2kΩ -> 1kΩ
- R27: value 20kΩ -> 10MΩ
- R28: value 9.09kΩ -> 10Ω
- R30: value 10kΩ -> 240kΩ
- R31: value 2mΩ -> 133kΩ
- R32: value 10kΩ -> 93.1kΩ
- R33: value 1kΩ -> 23.2kΩ
- R34: value 1kΩ -> 280kΩ
- R35: value 10kΩ -> 2kΩ
- R36: value 0.01Ω -> 20kΩ
- R37: value 0.01Ω -> 9.09kΩ
- R39: value 2.2Ω -> 2mΩ
- R4: value 10Ω -> 6Ω; moved to B.Cu
- R40, R41: value 0.01Ω -> 10kΩ; moved to B.Cu
- R5: value 2Ω -> 4.7Ω; moved to B.Cu
- R6: value 1MΩ -> 4.7Ω; moved to B.Cu
- R7: value 100kΩ -> 6Ω; moved to B.Cu
- R8: value 1.5kΩ -> 4.7Ω; moved to B.Cu
- R9: value 4.02kΩ -> 4.7Ω; moved to B.Cu
- U1: value TMC4671-LA -> LD1117S25TR_SOT223; footprint kuben_footprints:QFN76_10P5X6P5_TRI-L -> Package_TO_SOT_SMD:SOT-223-3_TabPin2
- U2: value ATSAMD11D14A-M -> LD1117S33TR_SOT223; footprint Package_DFN_QFN:QFN-24-1EP_4x4mm_P0.5mm_EP2.6x2.6mm -> Package_TO_SOT_SMD:SOT-223-3_TabPin2
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Connections:
- C1 pad 1: +12V -> Net-(IC1-HS)
- C1 pad 2: GND -> Net-(D1-K)
- C10 pad 1: Net-(IC7-ACP) -> Net-(IC5-AVCC)
- C10 pad 2: Net-(D4-A) -> GND
- C11 pad 1: /voltageregulators/IC4_vref -> +2.5V
- C12 pad 1: Net-(D4-A) -> Net-(D7-A)
- C13 pad 1: Net-(IC7-BTST) -> Net-(IC5-TTC)
- C13 pad 2: Net-(IC7-SW_1) -> GND
- C15 pad 1: Net-(IC7-REGN) -> Net-(IC5-ACP)
- C15 pad 2: GND -> Net-(D7-A)
- C17 pad 1: GND -> Net-(D7-A)
- C17 pad 2: Net-(IC7-SRP) -> GND
- C18 pad 1: Net-(IC7-SRP) -> +3.3V
- C18 pad 2: /voltageregulators/BATTIN -> GND
- C20 pad 1: /voltageregulators/BATTIN -> Net-(U3-VI)
- C21 pad 1: /voltageregulators/BATTIN -> Net-(IC5-REGN)
- C22 pad 1: Net-(IC9-VIN) -> GND
- C22 pad 2: GND -> Net-(IC5-SRP)
- C24 pad 1: GND -> +5V
- C24 pad 2: Net-(C24-Pad2) -> GND
- C25 pad 1: GND -> /voltageregulators/BATTIN
- C25 pad 2: Net-(IC9-COMP) -> GND
- C26 pad 1: GND -> /voltageregulators/BATTIN
- C26 pad 2: Net-(IC9-SS) -> GND
- C27 pad 1: GND -> Net-(IC6-VIN)
- C27 pad 2: Net-(IC9-SLOPE) -> GND
- C28 pad 2: +12V -> Net-(C28-Pad2)
- C29 pad 1: Net-(D7-K) -> GND
- C29 pad 2: /voltageregulators/SW1 -> Net-(IC6-COMP)
- C3 pad 1: +12V -> Net-(IC2-HS)
- C3 pad 2: GND -> Net-(D2-K)
- C30 pad 1: Net-(D6-K) -> GND
- C30 pad 2: /voltageregulators/SW2 -> Net-(IC6-SS)
- C31 pad 2: +3.3V -> Net-(IC6-SLOPE)
- C32 pad 2: +3.3V -> +12V
- C33 pad 1: GND -> Net-(D10-K)
- C33 pad 2: +3.3V -> /voltageregulators/SW1
- C34 pad 1: GND -> Net-(D9-K)
- C34 pad 2: +3.3V -> /voltageregulators/SW2
- C37 pad 1: +3.3V -> GND
- C37 pad 2: GND -> +3.3V
- C38 pad 1: +3.3V -> GND
- C38 pad 2: GND -> +3.3V
- C39 pad 1: +3.3V -> GND
- C39 pad 2: GND -> +3.3V
- C4 pad 1: Net-(C4-Pad1) -> +12V
- C40 pad 1: +3.3V -> GND
- C40 pad 2: GND -> +3.3V
- C47 pad 1: Net-(C47-Pad1) -> +3.3V
- C47 pad 2: Net-(IC10-VDDCORE) -> GND
- C48 pad 1: Net-(C47-Pad1) -> +3.3V
- C48 pad 2: Net-(IC10-VDDCORE) -> GND
- C49 pad 1: GND -> +3.3V
- C49 pad 2: +3.3V -> GND
- C5 pad 1: Net-(IC7-AVCC) -> Net-(IC3-HS)
- C5 pad 2: GND -> Net-(D3-K)
- C50 pad 1: GND -> +3.3V
- C50 pad 2: +3.3V -> GND
- C51 pad 1: GND -> Net-(C51-Pad1)
- C51 pad 2: +3.3V -> Net-(IC7-VDDCORE)
- C52 pad 1: GND -> Net-(C51-Pad1)
- C52 pad 2: +3.3V -> Net-(IC7-VDDCORE)
- C56 pad 1: Net-(IC11-HS) -> GND
- C56 pad 2: Net-(DBOOT3-K) -> +3.3V
- C57 pad 1: +12V -> GND
- C57 pad 2: GND -> +3.3V
- C58 pad 1: Net-(IC12-HS) -> GND
- C58 pad 2: Net-(DBOOT4-K) -> +3.3V
- C59 pad 1: +12V -> GND
- C59 pad 2: GND -> +3.3V
- C6 pad 1: Net-(IC7-ACDRV) -> +12V
- C60 pad 1: Net-(IC13-HS) -> Net-(IC8-HS)
- C60 pad 2: Net-(DBOOT5-K) -> Net-(D13-K)
- C62 pad 1: GND -> Net-(IC9-HS)
- C62 pad 2: +3.3V -> Net-(D14-K)
- C63 pad 1: GND -> +12V
- C63 pad 2: +3.3V -> GND
- C64 pad 1: GND -> Net-(IC10-HS)
- C64 pad 2: +3.3V -> Net-(D15-K)
- C65 pad 1: GND -> +12V
- C65 pad 2: +3.3V -> GND
- C66 pad 2: +3.3V -> +5V
- C68 pad 1: Net-(IC15-HS) -> GND
- C68 pad 2: Net-(D10-K) -> +3.3V
- C69 pad 1: +12V -> GND
- C69 pad 2: GND -> +3.3V
- C70 pad 1: Net-(IC16-HS) -> GND
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Other:
- board size 140 x 105 mm -> 80 x 80 mm
- copper layers 2 -> 4

Commit message: Started on software
State machine structure is laid out.
TMC4671 drivers are taken from official software.
IMU drivers are taken from portalspace/drivers, but are
not fully configured for our purposes yet.
Compact Quaternion library has also been added.
Parts:
- removed the C14 at (33.7, 41.2)
- removed the C16 at (33.7, 46.2)
- removed the C19 at (37.7, 28.6)
- removed the C23 at (37.7, 38.6)
- removed the C7 at (33.7, 23.6)
- removed C74, C76, C78: 1µF, Capacitor_SMD:C_0603_1608Metric
- removed C75, C77, C79: 0.1µF, Capacitor_SMD:C_0603_1608Metric
- removed the C8 at (33.7, 26.1)
- removed D11, D12: LED, Diode_SMD:D_0603_1608Metric
- removed D13, D14, D15, D16, D17, D18: 470mV 500mA, Diode_SMD:D_0603_1608Metric
- removed IC5: BQ24133RGYR, kuben-footprints:BQ24133RGYR
- removed IC6: LM5176PWPR, kuben-footprints:SOP65P640X120-29N
- removed IC8: LM5109BSDX_NOPB, kuben-footprints:SON80P400X400X80-9N
- removed J7: Conn_01x04_Socket, Connector_PinSocket_2.54mm:PinSocket_1x04_P2.54mm_Vertical
- removed R42, R43: 1kΩ, Resistor_SMD:R_0603_1608Metric
- removed R44, R45, R57, R58: 10kΩ, Resistor_SMD:R_0603_1608Metric
- removed R46, R49, R52, R59, R62, R65: 6Ω, Resistor_SMD:R_0603_1608Metric
- removed R47, R48, R50, R51, R53, R54, R60, R61, R63, R64, R66, R67: 4.7Ω, Resistor_SMD:R_0603_1608Metric
- removed R55, R56, R68, R69: 0.01Ω, Resistor_SMD:R_0603_1608Metric
- removed TP1, TP2, TP3, TP4: TestPoint, TestPoint:TestPoint_Pad_D1.5mm
- added 100nF1: C, Capacitor_SMD:C_0603_1608Metric, F.Cu at (90.4, 97.8)
- added 100nF10: C, Capacitor_SMD:C_0603_1608Metric, F.Cu at (112.5, 124.9)
- added 100nF11: C, Capacitor_SMD:C_0603_1608Metric, F.Cu at (112.5, 127.4)
- added 100nF12: C, Capacitor_SMD:C_0603_1608Metric, F.Cu at (112.5, 129.9)
- added 100nF13: C, Capacitor_SMD:C_0603_1608Metric, F.Cu at (112.5, 132.5)
- added 100nF14: C, Capacitor_SMD:C_0603_1608Metric, F.Cu at (112.5, 135.0)
- added 100nF15: C, Capacitor_SMD:C_0603_1608Metric, F.Cu at (112.5, 137.5)
- added 100nF16: C, Capacitor_SMD:C_0603_1608Metric, F.Cu at (106.5, 124.9)
- added 100nF17: C, Capacitor_SMD:C_0603_1608Metric, F.Cu at (106.5, 127.4)
- added 100nF18: C, Capacitor_SMD:C_0603_1608Metric, F.Cu at (106.5, 129.9)
- added 100nF19: C, Capacitor_SMD:C_0603_1608Metric, F.Cu at (106.5, 132.5)
- added 100nF2: C, Capacitor_SMD:C_0603_1608Metric, F.Cu at (90.4, 100.3)
- added 100nF20: C, Capacitor_SMD:C_0603_1608Metric, F.Cu at (106.5, 135.0)
- added 100nF21: C, Capacitor_SMD:C_0603_1608Metric, F.Cu at (106.5, 137.5)
- added 100nF3: C, Capacitor_SMD:C_0603_1608Metric, F.Cu at (100.5, 124.9)
- added 100nF4: C, Capacitor_SMD:C_0603_1608Metric, F.Cu at (100.5, 127.4)
- added 100nF5: C, Capacitor_SMD:C_0603_1608Metric, F.Cu at (100.5, 129.9)
- added 100nF6: C, Capacitor_SMD:C_0603_1608Metric, F.Cu at (100.5, 132.5)
- added 100nF7: C, Capacitor_SMD:C_0603_1608Metric, F.Cu at (100.5, 135.0)
- added 100nF8: C, Capacitor_SMD:C_0603_1608Metric, F.Cu at (100.5, 137.5)
- added 100nF9: C, Capacitor_SMD:C_0603_1608Metric, F.Cu at (118.5, 134.0)
- added 10ohm1: R, Resistor_SMD:R_0603_1608Metric, F.Cu at (90.4, 102.8)
- added 133k1: R, Resistor_SMD:R_0603_1608Metric, F.Cu at (90.4, 105.4)
- added 15nF1: C, Capacitor_SMD:C_0603_1608Metric, F.Cu at (90.4, 107.9)
- added 240k1: R, Resistor_SMD:R_0603_1608Metric, F.Cu at (90.4, 110.4)
- added Bootstrap1: 0.1µF, Capacitor_SMD:C_0603_1608Metric, F.Cu at (130.6, 97.8)
- added Bootstrap2: 0.1µF, Capacitor_SMD:C_0603_1608Metric, F.Cu at (130.6, 100.3)
- added Bootstrap3: 0.1µF, Capacitor_SMD:C_0603_1608Metric, F.Cu at (130.6, 102.8)
- added C14: 100nF, Capacitor_SMD:C_0603_1608Metric, F.Cu at (215.3, 55.0)
- added C14: 100nF, Capacitor_SMD:C_0603_1608Metric, F.Cu at (94.4, 112.9)
- added C16: 100nF, Capacitor_SMD:C_0603_1608Metric, F.Cu at (94.4, 117.9)
- added C16: 10uF, Capacitor_SMD:C_0603_1608Metric, F.Cu at (215.3, 57.5)
- added C19: 100nF, Capacitor_SMD:C_0603_1608Metric, F.Cu at (98.4, 100.3)
- added C19: 100nF, Capacitor_SMD:C_0603_1608Metric, F.Cu at (215.3, 60.0)
- added C23: 10uF, Capacitor_SMD:C_0603_1608Metric, F.Cu at (215.3, 62.5)
- added C23: 10µF, Capacitor_SMD:C_0603_1608Metric, F.Cu at (98.4, 110.4)
- added C7: 100nF, Capacitor_SMD:C_0603_1608Metric, F.Cu at (215.3, 50.0)
- added C7: 100nF, Capacitor_SMD:C_0603_1608Metric, F.Cu at (90.4, 120.4)
- added C8: 10uF, Capacitor_SMD:C_0603_1608Metric, F.Cu at (215.3, 52.5)
- added C8: 100nF, Capacitor_SMD:C_0603_1608Metric, F.Cu at (94.4, 97.8)
- added Charging1: LED, Diode_SMD:D_0603_1608Metric, F.Cu at (114.5, 97.9)
- added DBOOT1: D, Diode_SMD:D_0603_1608Metric, F.Cu at (134.6, 100.5)
- added DBOOT2: D, Diode_SMD:D_0603_1608Metric, F.Cu at (134.6, 103.0)
- added DBOOT3: D, Diode_SMD:D_0603_1608Metric, F.Cu at (94.5, 125.0)
- added DBOOT4: D, Diode_SMD:D_0603_1608Metric, F.Cu at (94.5, 127.6)
- added DBOOT5: D, Diode_SMD:D_0603_1608Metric, F.Cu at (94.5, 130.2)
- added DBOOT6: D, Diode_SMD:D_0603_1608Metric, F.Cu at (124.6, 100.5)
- added DBOOT7: D, Diode_SMD:D_0603_1608Metric, F.Cu at (124.6, 103.0)
- added IC16: LM5109BSDX_NOPB, kuben_footprints:SON80P400X400X80-9N, F.Cu at (196.5, 79.8)
- added IC17: LM5109BSDX_NOPB, kuben_footprints:SON80P400X400X80-9N, F.Cu at (196.5, 85.5)
- added IC18: INA2181A2IDGSR, kuben_footprints:SOP50P490X110-10N, F.Cu at (197.1, 90.6)
- added RBOOT1: 2.2Ω, Resistor_SMD:R_0603_1608Metric, F.Cu at (151.8, 68.5)
- added RBOOT2: 2.2Ω, Resistor_SMD:R_0603_1608Metric, F.Cu at (151.8, 71.0)
- added RBOOT3: 2.2Ω, Resistor_SMD:R_0603_1608Metric, F.Cu at (90.4, 145.0)
- added RBOOT4: 2.2Ω, Resistor_SMD:R_0603_1608Metric, F.Cu at (129.7, 71.5)
- added RBOOT5: 2.2Ω, Resistor_SMD:R_0603_1608Metric, F.Cu at (129.7, 74.0)
- added RBOOT6: 2.2Ω, Resistor_SMD:R_0603_1608Metric, F.Cu at (145.8, 64.0)
- added RBOOT7: 2.2Ω, Resistor_SMD:R_0603_1608Metric, F.Cu at (145.8, 66.5)
- added Screen1: Conn_01x04, Connector_PinHeader_2.00mm:PinHeader_1x04_P2.00mm_Horizontal, F.Cu at (174.5, 49.1)
- C1, C3, C34, C35, C36, C37, C39, C60, C67, C73: moved to F.Cu
- C10: value ?F -> 0.1µF
- C11: value 10uF -> 1µF
- C12: value 10µF -> 1µF
- C13: value 0.1µF -> 0.047µF
- C15: value 0.1µF -> 1µF
- C17: value 1µF -> 0.1µF
- C18: value 10uF -> 0.1µF
- C2, C61: value 1µF -> 0.1µF; moved to F.Cu
- C20, C40: value 100nF -> 10µF
- C21: value 1µF -> 10µF
- C22: value 0.1µF -> 10nF
- C24: value 10uF -> 33nF
- C25: value 10µF -> 470pF
- C26: value 10µF -> 15nF
- C27: value 10nF -> 220pF
- C28: value 33nF -> 270µF
- C29: value 470pF -> 100nF
- C30: value 15nF -> 100nF
- C31: value 220pF -> 100nF
- C32: value 270µF -> 100nF
- C38: value 100nF -> 10µF; moved to F.Cu
- C4: value 1µF -> 2.2µF; moved to F.Cu
- C48: value 10µF -> 4.7µF
- C5: value 0.1µF -> ?F; moved to F.Cu
- C50: value 10µF -> 100nF
- C52: value 4.7µF -> 100nF
- C56, C57, C58: value 100nF -> 0.1µF
- C59, C68, C69, C70, C71, C72: value 100nF -> 0.1µF; moved to F.Cu
- C6: value 1µF -> 10µF; moved to F.Cu
- C62, C64, C66: value 0.1µF -> 100nF; moved to F.Cu
- C63, C65: value 1µF -> 100nF; moved to F.Cu
- C9: value 2.2µF -> 0.1µF
- D1: value 470mV 500mA -> D; moved to F.Cu
- D10: value 470mV 500mA -> D
- D2, D3: value 470mV 500mA -> BZV55B2V4; footprint Diode_SMD:D_0603_1608Metric -> Diode_SMD:D_MiniMELF; moved to F.Cu
- D4: value BZV55B2V4 -> 470mV 500mA; footprint Diode_SMD:D_MiniMELF -> Diode_SMD:D_0603_1608Metric
- D5: value BZV55B2V4 -> LED; footprint Diode_SMD:D_MiniMELF -> Diode_SMD:D_0603_1608Metric
- D6: value LED -> 385mV 500mA
- D9: value 385mV 500mA -> LED
- IC1, IC12, IC13, IC2, IC3: footprint kuben-footprints:SON80P400X400X80-9N -> kuben_footprints:SON80P400X400X80-9N; moved to F.Cu
- IC10: value LM5109BSDX_NOPB -> ATSAME53J18A-MF; footprint kuben-footprints:SON80P400X400X80-9N -> kuben_footprints:QFN50P900X900X100-65N-D; moved to F.Cu
- IC11, IC15: value INA2181A2IDGSR -> LM5109BSDX_NOPB; footprint kuben-footprints:SOP50P490X110-10N -> kuben_footprints:SON80P400X400X80-9N; moved to F.Cu
- IC14: value LM5109BSDX_NOPB -> INA2181A2IDGSR; footprint kuben-footprints:SON80P400X400X80-9N -> kuben_footprints:SOP50P490X110-10N; moved to F.Cu
- IC4: footprint kuben-footprints:SOP50P490X110-10N -> kuben_footprints:SOP50P490X110-10N; moved to F.Cu
- IC7: value ATSAME53J18A-MF -> BQ24133RGYR; footprint kuben-footprints:QFN50P900X900X100-65N-D -> kuben_footprints:BQ24133RGYR
- IC9: value LM5109BSDX_NOPB -> LM5176PWPR; footprint kuben-footprints:SON80P400X400X80-9N -> kuben_footprints:SOP65P640X120-29N; moved to F.Cu
- J1, J2: footprint kuben-footprints:59453052110ECHLF -> kuben_footprints:59453052110ECHLF; moved to F.Cu
- J3: footprint kuben-footprints:VN02A1500000G -> kuben_footprints:VN02A1500000G
- J4, J5, J6: footprint kuben-footprints:1849521 -> kuben_footprints:1849521; moved to F.Cu
- Q1, Q14, Q15, Q16, Q17, Q18, Q19, Q2, Q20, Q21, Q22, Q23, Q24, Q25, Q3, Q4, Q5, Q6: footprint kuben-footprints:SOT96P240X115-3N -> kuben_footprints:SOT96P240X115-3N; moved to F.Cu
- Q10, Q11, Q12, Q13, Q7, Q8: footprint kuben-footprints:SOT96P240X115-3N -> kuben_footprints:SOT96P240X115-3N
- Q9: footprint kuben-footprints:DMPH6050SK313 -> kuben_footprints:DMPH6050SK313
- R1: value 6Ω -> 2.2Ω; moved to F.Cu
- R10: value 0.01Ω -> 5.23kΩ; moved to F.Cu
- R11: value 0.01Ω -> 30.1kΩ; moved to F.Cu
- R12: value 10Ω -> 4.02kΩ
- R13: value 2Ω -> 20mΩ
- R14: value 1MΩ -> 232kΩ
- R15: value 100kΩ -> 32.4kΩ
- R16: value 1.5kΩ -> 100kΩ
- R17: value 4.02kΩ -> 32.4kΩ
- R18: value 5.23kΩ -> 1kΩ
- R19: value 30.1kΩ -> 10MΩ
- R2, R3: value 4.7Ω -> 0.01Ω; moved to F.Cu
- R20: value 4.02kΩ -> 10Ω
- R21: value 20mΩ -> 240kΩ
- R22: value 232kΩ -> 133kΩ
- R23: value 32.4kΩ -> 93.1kΩ
- R24: value 100kΩ -> 23.2kΩ
- R25: value 32.4kΩ -> 280kΩ
- R26: value 1kΩ -> 2kΩ
- R27: value 10MΩ -> 20kΩ
- R28: value 10Ω -> 9.09kΩ
- R30: value 240kΩ -> 10kΩ
- R31: value 133kΩ -> 2mΩ
- R32: value 93.1kΩ -> 10kΩ
- R33: value 23.2kΩ -> 1kΩ
- R34: value 280kΩ -> 1kΩ
- R35: value 2kΩ -> 10kΩ
- R36: value 20kΩ -> 0.01Ω
- R37: value 9.09kΩ -> 0.01Ω
- R39: value 2mΩ -> 2.2Ω
- R4: value 6Ω -> 10Ω; moved to F.Cu
- R40, R41: value 10kΩ -> 0.01Ω; moved to F.Cu
- R5: value 4.7Ω -> 2Ω; moved to F.Cu
- R6: value 4.7Ω -> 1MΩ; moved to F.Cu
- R7: value 6Ω -> 100kΩ; moved to F.Cu
- R8: value 4.7Ω -> 1.5kΩ; moved to F.Cu
- R9: value 4.7Ω -> 4.02kΩ; moved to F.Cu
- U1: value LD1117S25TR_SOT223 -> TMC4671-LA; footprint Package_TO_SOT_SMD:SOT-223-3_TabPin2 -> kuben_footprints:QFN76_10P5X6P5_TRI-L
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Connections:
- C1 pad 1: Net-(IC1-HS) -> +12V
- C1 pad 2: Net-(D1-K) -> GND
- C10 pad 1: Net-(IC5-AVCC) -> Net-(IC7-ACP)
- C10 pad 2: GND -> Net-(D4-A)
- C11 pad 1: +2.5V -> /voltageregulators/IC4_vref
- C12 pad 1: Net-(D7-A) -> Net-(D4-A)
- C13 pad 1: Net-(IC5-TTC) -> Net-(IC7-BTST)
- C13 pad 2: GND -> Net-(IC7-SW_1)
- C15 pad 1: Net-(IC5-ACP) -> Net-(IC7-REGN)
- C15 pad 2: Net-(D7-A) -> GND
- C17 pad 1: Net-(D7-A) -> GND
- C17 pad 2: GND -> Net-(IC7-SRP)
- C18 pad 1: +3.3V -> Net-(IC7-SRP)
- C18 pad 2: GND -> /voltageregulators/BATTIN
- C20 pad 1: Net-(U3-VI) -> /voltageregulators/BATTIN
- C21 pad 1: Net-(IC5-REGN) -> /voltageregulators/BATTIN
- C22 pad 1: GND -> Net-(IC9-VIN)
- C22 pad 2: Net-(IC5-SRP) -> GND
- C24 pad 1: +5V -> GND
- C24 pad 2: GND -> Net-(C24-Pad2)
- C25 pad 1: /voltageregulators/BATTIN -> GND
- C25 pad 2: GND -> Net-(IC9-COMP)
- C26 pad 1: /voltageregulators/BATTIN -> GND
- C26 pad 2: GND -> Net-(IC9-SS)
- C27 pad 1: Net-(IC6-VIN) -> GND
- C27 pad 2: GND -> Net-(IC9-SLOPE)
- C28 pad 2: Net-(C28-Pad2) -> +12V
- C29 pad 1: GND -> Net-(D7-K)
- C29 pad 2: Net-(IC6-COMP) -> /voltageregulators/SW1
- C3 pad 1: Net-(IC2-HS) -> +12V
- C3 pad 2: Net-(D2-K) -> GND
- C30 pad 1: GND -> Net-(D6-K)
- C30 pad 2: Net-(IC6-SS) -> /voltageregulators/SW2
- C31 pad 2: Net-(IC6-SLOPE) -> +3.3V
- C32 pad 2: +12V -> +3.3V
- C33 pad 1: Net-(D10-K) -> GND
- C33 pad 2: /voltageregulators/SW1 -> +3.3V
- C34 pad 1: Net-(D9-K) -> GND
- C34 pad 2: /voltageregulators/SW2 -> +3.3V
- C37 pad 1: GND -> +3.3V
- C37 pad 2: +3.3V -> GND
- C38 pad 1: GND -> +3.3V
- C38 pad 2: +3.3V -> GND
- C39 pad 1: GND -> +3.3V
- C39 pad 2: +3.3V -> GND
- C4 pad 1: +12V -> Net-(C4-Pad1)
- C40 pad 1: GND -> +3.3V
- C40 pad 2: +3.3V -> GND
- C47 pad 1: +3.3V -> Net-(C47-Pad1)
- C47 pad 2: GND -> Net-(IC10-VDDCORE)
- C48 pad 1: +3.3V -> Net-(C47-Pad1)
- C48 pad 2: GND -> Net-(IC10-VDDCORE)
- C49 pad 1: +3.3V -> GND
- C49 pad 2: GND -> +3.3V
- C5 pad 1: Net-(IC3-HS) -> Net-(IC7-AVCC)
- C5 pad 2: Net-(D3-K) -> GND
- C50 pad 1: +3.3V -> GND
- C50 pad 2: GND -> +3.3V
- C51 pad 1: Net-(C51-Pad1) -> GND
- C51 pad 2: Net-(IC7-VDDCORE) -> +3.3V
- C52 pad 1: Net-(C51-Pad1) -> GND
- C52 pad 2: Net-(IC7-VDDCORE) -> +3.3V
- C56 pad 1: GND -> Net-(IC11-HS)
- C56 pad 2: +3.3V -> Net-(DBOOT3-K)
- C57 pad 1: GND -> +12V
- C57 pad 2: +3.3V -> GND
- C58 pad 1: GND -> Net-(IC12-HS)
- C58 pad 2: +3.3V -> Net-(DBOOT4-K)
- C59 pad 1: GND -> +12V
- C59 pad 2: +3.3V -> GND
- C6 pad 1: +12V -> Net-(IC7-ACDRV)
- C60 pad 1: Net-(IC8-HS) -> Net-(IC13-HS)
- C60 pad 2: Net-(D13-K) -> Net-(DBOOT5-K)
- C62 pad 1: Net-(IC9-HS) -> GND
- C62 pad 2: Net-(D14-K) -> +3.3V
- C63 pad 1: +12V -> GND
- C63 pad 2: GND -> +3.3V
- C64 pad 1: Net-(IC10-HS) -> GND
- C64 pad 2: Net-(D15-K) -> +3.3V
- C65 pad 1: +12V -> GND
- C65 pad 2: GND -> +3.3V
- C66 pad 2: +5V -> +3.3V
- C68 pad 1: GND -> Net-(IC15-HS)
- C68 pad 2: +3.3V -> Net-(D10-K)
- C69 pad 1: GND -> +12V
- C69 pad 2: +3.3V -> GND
- C70 pad 1: GND -> Net-(IC16-HS)
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Other:
- board size 80 x 80 mm -> 140 x 105 mm
- copper layers 4 -> 2

Commit message: worked on schemtaic
Parts:
- removed 100nF1, 100nF10, 100nF11, 100nF12, 100nF13, 100nF14, 100nF15, 100nF16, 100nF17, 100nF18, 100nF19, 100nF2, 100nF20, 100nF21, 100nF3, 100nF4, 100nF5, 100nF6, 100nF7, 100nF8, 100nF9, 15nF1: C, Capacitor_SMD:C_0603_1608Metric
- removed 10ohm1, 133k1, 240k1: R, Resistor_SMD:R_0603_1608Metric
- removed Bootstrap1, Bootstrap2, Bootstrap3: 0.1µF, Capacitor_SMD:C_0603_1608Metric
- removed the C14 at (215.3, 55.0)
- removed the C14 at (94.4, 112.9)
- removed the C16 at (94.4, 117.9)
- removed the C16 at (215.3, 57.5)
- removed the C19 at (98.4, 100.3)
- removed the C19 at (215.3, 60.0)
- removed the C23 at (215.3, 62.5)
- removed the C23 at (98.4, 110.4)
- removed the C7 at (215.3, 50.0)
- removed the C7 at (90.4, 120.4)
- removed the C8 at (215.3, 52.5)
- removed the C8 at (94.4, 97.8)
- removed Charging1: LED, Diode_SMD:D_0603_1608Metric
- removed DB1: Conn_01x02_Pin, Connector_PinHeader_2.54mm:PinHeader_1x02_P2.54mm_Vertical
- removed DBOOT1, DBOOT2, DBOOT3, DBOOT4, DBOOT5, DBOOT6, DBOOT7: D, Diode_SMD:D_0603_1608Metric
- removed L3: ?H, Inductor_SMD:L_0603_1608Metric
- removed RBOOT1, RBOOT2, RBOOT3, RBOOT4, RBOOT5, RBOOT6, RBOOT7: 2.2Ω, Resistor_SMD:R_0603_1608Metric
- removed Screen1: Conn_01x04, Connector_PinHeader_2.00mm:PinHeader_1x04_P2.00mm_Horizontal
- added C100: 1µF, Capacitor_SMD:C_0603_1608Metric, F.Cu at (90.2, 48.9)
- added C101: 0.1µF, Capacitor_SMD:C_0603_1608Metric, F.Cu at (90.2, 51.4)
- added C102: 1µF, Capacitor_SMD:C_0603_1608Metric, F.Cu at (90.2, 53.9)
- added C103: 0.1µF, Capacitor_SMD:C_0603_1608Metric, F.Cu at (90.2, 56.4)
- added C104: 1µF, Capacitor_SMD:C_0603_1608Metric, F.Cu at (90.2, 58.9)
- added C105: 220µF 35V, kuben-footprints:CAPAE1050X1050N, F.Cu at (108.1, 48.9)
- added C106: 0.1µF, Capacitor_SMD:C_0603_1608Metric, F.Cu at (94.2, 43.8)
- added C14: 10µF, Capacitor_SMD:C_0603_1608Metric, F.Cu at (93.8, 130.6)
- added C16: 100nF, Capacitor_SMD:C_0603_1608Metric, F.Cu at (93.8, 135.6)
- added C19: 1µF, Capacitor_SMD:C_0603_1608Metric, F.Cu at (97.8, 120.5)
- added C23: 1µF, Capacitor_SMD:C_0603_1608Metric, F.Cu at (97.8, 130.6)
- added C7: 1µF, Capacitor_SMD:C_0603_1608Metric, F.Cu at (159.7, 58.9)
- added C74: 100nF, Capacitor_SMD:C_0603_1608Metric, F.Cu at (169.6, 140.3)
- added C75: 10nF, Capacitor_SMD:C_0603_1608Metric, F.Cu at (169.6, 142.8)
- added C76: 0.1µF, Capacitor_SMD:C_0603_1608Metric, F.Cu at (90.2, 82.2)
- added C77: 1µF, Capacitor_SMD:C_0603_1608Metric, F.Cu at (90.2, 84.7)
- added C78: 1µF, Capacitor_SMD:C_0603_1608Metric, F.Cu at (90.2, 87.2)
- added C79: 0.1µF, Capacitor_SMD:C_0603_1608Metric, F.Cu at (90.2, 89.7)
- added C8: 220µF 35V, kuben-footprints:CAPAE1050X1050N, F.Cu at (177.6, 48.9)
- added C80: 1µF, Capacitor_SMD:C_0603_1608Metric, F.Cu at (90.2, 92.2)
- added C81: 0.1µF, Capacitor_SMD:C_0603_1608Metric, F.Cu at (90.2, 94.7)
- added C82: 1µF, Capacitor_SMD:C_0603_1608Metric, F.Cu at (90.2, 97.2)
- added C83: 220µF 35V, kuben-footprints:CAPAE1050X1050N, F.Cu at (108.1, 87.2)
- added C84: 0.1µF, Capacitor_SMD:C_0603_1608Metric, F.Cu at (94.2, 82.2)
- added C85: 100pF, Capacitor_SMD:C_0603_1608Metric, F.Cu at (165.6, 101.9)
- added C86: 100pF, Capacitor_SMD:C_0603_1608Metric, F.Cu at (165.6, 104.4)
- added C87: 100pF, Capacitor_SMD:C_0603_1608Metric, F.Cu at (165.6, 107.0)
- added C88: 100nF, Capacitor_SMD:C_0603_1608Metric, F.Cu at (165.6, 109.5)
- added C89: 100nF, Capacitor_SMD:C_0603_1608Metric, F.Cu at (165.6, 112.0)
- added C90: 100nF, Capacitor_SMD:C_0603_1608Metric, F.Cu at (165.6, 114.5)
- added C91: 100nF, Capacitor_SMD:C_0603_1608Metric, F.Cu at (165.6, 117.0)
- added C92: 100nF, Capacitor_SMD:C_0603_1608Metric, F.Cu at (169.6, 101.9)
- added C93: 100nF, Capacitor_SMD:C_0603_1608Metric, F.Cu at (169.6, 104.4)
- added C94: 100nF, Capacitor_SMD:C_0603_1608Metric, F.Cu at (169.6, 107.0)
- added C95: 100nF, Capacitor_SMD:C_0603_1608Metric, F.Cu at (169.6, 109.5)
- added C96: 100nF, Capacitor_SMD:C_0603_1608Metric, F.Cu at (169.6, 112.0)
- added C97: 10nF, Capacitor_SMD:C_0603_1608Metric, F.Cu at (169.6, 114.5)
- added C98: 0.1µF, Capacitor_SMD:C_0603_1608Metric, F.Cu at (90.2, 43.8)
- added C99: 1µF, Capacitor_SMD:C_0603_1608Metric, F.Cu at (90.2, 46.3)
- added D11: 470mV 500mA, Diode_SMD:D_0603_1608Metric, F.Cu at (117.9, 136.1)
- added D12: 470mV 500mA, Diode_SMD:D_0603_1608Metric, F.Cu at (177.5, 68.5)
- added D13: 470mV 500mA, Diode_SMD:D_0603_1608Metric, F.Cu at (177.5, 71.1)
- added D14: 470mV 500mA, Diode_SMD:D_0603_1608Metric, F.Cu at (177.5, 73.7)
- added D15: 470mV 500mA, Diode_SMD:D_0603_1608Metric, F.Cu at (177.5, 76.2)
- added D16: 470mV 500mA, Diode_SMD:D_0603_1608Metric, F.Cu at (177.5, 78.8)
- added D17: 470mV 500mA, Diode_SMD:D_0603_1608Metric, F.Cu at (177.5, 81.4)
- added D18: 470mV 500mA, Diode_SMD:D_0603_1608Metric, F.Cu at (177.5, 84.0)
- added D19: 470mV 500mA, Diode_SMD:D_0603_1608Metric, F.Cu at (181.5, 68.5)
- added D20: 470mV 500mA, Diode_SMD:D_0603_1608Metric, F.Cu at (181.5, 71.1)
- added D21: 470mV 500mA, Diode_SMD:D_0603_1608Metric, F.Cu at (181.5, 73.7)
- added D22: 470mV 500mA, Diode_SMD:D_0603_1608Metric, F.Cu at (181.5, 76.2)
- added D23: 470mV 500mA, Diode_SMD:D_0603_1608Metric, F.Cu at (181.5, 78.8)
- added D24: 470mV 500mA, Diode_SMD:D_0603_1608Metric, F.Cu at (181.5, 81.4)
- added D25: 470mV 500mA, Diode_SMD:D_0603_1608Metric, F.Cu at (181.5, 84.0)
- added D26: LED, Diode_SMD:D_0603_1608Metric, F.Cu at (185.6, 68.5)
- added D27: LED, Diode_SMD:D_0603_1608Metric, F.Cu at (185.6, 71.1)
- added D28: LED, Diode_SMD:D_0603_1608Metric, F.Cu at (185.6, 73.7)
- added D29: 470mV 500mA, Diode_SMD:D_0603_1608Metric, F.Cu at (185.6, 76.2)
- added D30: 470mV 500mA, Diode_SMD:D_0603_1608Metric, F.Cu at (185.6, 78.8)
- added D31: LED, Diode_SMD:D_0603_1608Metric, F.Cu at (202.0, 143.0)
- added D32: LED, Diode_SMD:D_0603_1608Metric, F.Cu at (202.0, 145.6)
- added D33: 470mV 500mA, Diode_SMD:D_0603_1608Metric, F.Cu at (153.4, 130.3)
- added D34: 470mV 500mA, Diode_SMD:D_0603_1608Metric, F.Cu at (153.4, 132.9)
- added D35: 470mV 500mA, Diode_SMD:D_0603_1608Metric, F.Cu at (153.4, 135.5)
- added D36: 470mV 500mA, Diode_SMD:D_0603_1608Metric, F.Cu at (153.4, 138.1)
- added D37: 470mV 500mA, Diode_SMD:D_0603_1608Metric, F.Cu at (153.4, 140.7)
- added D38: 470mV 500mA, Diode_SMD:D_0603_1608Metric, F.Cu at (153.4, 143.3)
- added D39: 470mV 500mA, Diode_SMD:D_0603_1608Metric, F.Cu at (153.4, 145.9)
- added D40: 470mV 500mA, Diode_SMD:D_0603_1608Metric, F.Cu at (157.5, 130.3)
- added D41: 470mV 500mA, Diode_SMD:D_0603_1608Metric, F.Cu at (157.5, 132.9)
- added D42: 470mV 500mA, Diode_SMD:D_0603_1608Metric, F.Cu at (157.5, 135.5)
- added D43: 470mV 500mA, Diode_SMD:D_0603_1608Metric, F.Cu at (157.5, 138.1)
- added D44: 470mV 500mA, Diode_SMD:D_0603_1608Metric, F.Cu at (157.5, 140.7)
- added D45: 470mV 500mA, Diode_SMD:D_0603_1608Metric, F.Cu at (157.5, 143.3)
- added D46: 470mV 500mA, Diode_SMD:D_0603_1608Metric, F.Cu at (157.5, 145.9)
- added D47: LED, Diode_SMD:D_0603_1608Metric, F.Cu at (161.5, 130.3)
- added D48: LED, Diode_SMD:D_0603_1608Metric, F.Cu at (161.5, 132.9)
- added D49: LED, Diode_SMD:D_0603_1608Metric, F.Cu at (161.5, 135.5)
- added D50: 470mV 500mA, Diode_SMD:D_0603_1608Metric, F.Cu at (161.5, 138.1)
- added D51: 470mV 500mA, Diode_SMD:D_0603_1608Metric, F.Cu at (161.5, 140.7)
- added D52: 20Vr 5A, Diode_SMD:D_0603_1608Metric, F.Cu at (118.0, 82.2)
- added D53: 20Vr 5A, Diode_SMD:D_0603_1608Metric, F.Cu at (118.0, 84.8)
- added D54: 20Vr 5A, Diode_SMD:D_0603_1608Metric, F.Cu at (118.0, 87.4)
- added D55: 20Vr 5A, Diode_SMD:D_0603_1608Metric, F.Cu at (118.0, 90.0)
- added D56: 470mV 500mA, Diode_SMD:D_0603_1608Metric, F.Cu at (153.4, 102.0)
- added D57: 470mV 500mA, Diode_SMD:D_0603_1608Metric, F.Cu at (153.4, 104.6)
- added D58: 470mV 500mA, Diode_SMD:D_0603_1608Metric, F.Cu at (153.4, 107.2)
- added D59: 470mV 500mA, Diode_SMD:D_0603_1608Metric, F.Cu at (153.4, 109.7)
- added D60: 470mV 500mA, Diode_SMD:D_0603_1608Metric, F.Cu at (153.4, 112.3)
- added D61: 470mV 500mA, Diode_SMD:D_0603_1608Metric, F.Cu at (153.4, 114.9)
- added D62: 470mV 500mA, Diode_SMD:D_0603_1608Metric, F.Cu at (153.4, 117.5)
- added D63: 470mV 500mA, Diode_SMD:D_0603_1608Metric, F.Cu at (157.5, 102.0)
- added D64: 470mV 500mA, Diode_SMD:D_0603_1608Metric, F.Cu at (157.5, 104.6)
- added D65: 470mV 500mA, Diode_SMD:D_0603_1608Metric, F.Cu at (157.5, 107.2)
- added D66: 470mV 500mA, Diode_SMD:D_0603_1608Metric, F.Cu at (157.5, 109.7)
- added D67: 470mV 500mA, Diode_SMD:D_0603_1608Metric, F.Cu at (157.5, 112.3)
- added D68: 470mV 500mA, Diode_SMD:D_0603_1608Metric, F.Cu at (157.5, 114.9)
- added D69: 470mV 500mA, Diode_SMD:D_0603_1608Metric, F.Cu at (157.5, 117.5)
- added D70: LED, Diode_SMD:D_0603_1608Metric, F.Cu at (161.5, 102.0)
- added D71: LED, Diode_SMD:D_0603_1608Metric, F.Cu at (161.5, 104.6)
- added D72: LED, Diode_SMD:D_0603_1608Metric, F.Cu at (161.5, 107.2)
- added D73: 470mV 500mA, Diode_SMD:D_0603_1608Metric, F.Cu at (161.5, 109.7)
- added D74: 470mV 500mA, Diode_SMD:D_0603_1608Metric, F.Cu at (161.5, 112.3)
- added D75: 20Vr 5A, Diode_SMD:D_0603_1608Metric, F.Cu at (118.0, 43.9)
- added D76: 20Vr 5A, Diode_SMD:D_0603_1608Metric, F.Cu at (118.0, 46.5)
- added D77: 20Vr 5A, Diode_SMD:D_0603_1608Metric, F.Cu at (118.0, 49.0)
- added D78: 20Vr 5A, Diode_SMD:D_0603_1608Metric, F.Cu at (118.0, 51.6)
- added IC5: INA2181A2IDGSR, kuben-footprints:SOP50P490X110-10N, F.Cu at (193.2, 44.9)
- added IC6: BQ24133RGYR, kuben-footprints:BQ24133RGYR, F.Cu at (125.3, 149.8)
- added IC8: ATSAME53J18A-MF, kuben-footprints:QFN50P900X900X100-65N-D, F.Cu at (199.2, 136.1)
- added J7: 1-84952-1, kuben-footprints:1849521, F.Cu at (162.4, 94.4)
- added Q26: 30V 71A, kuben-footprints:IPD047N03LF2SATMA1, F.Cu at (125.3, 35.7)
- added Q27: 30V 71A, kuben-footprints:IPD047N03LF2SATMA1, F.Cu at (134.9, 35.7)
- added Q28: 30V 71A, kuben-footprints:IPD047N03LF2SATMA1, F.Cu at (144.6, 35.7)
- added R100: 5Ω, Resistor_SMD:R_0603_1608Metric, F.Cu at (94.2, 53.9)
- added R101: 4.7Ω, Resistor_SMD:R_0603_1608Metric, F.Cu at (94.2, 56.4)
- added R102: 4.7Ω, Resistor_SMD:R_0603_1608Metric, F.Cu at (94.2, 58.9)
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Connections:
- net Net-(IC14-IN-1) renamed /drivergates2/PWM_W_H
- net Net-(IC4-IN-1) renamed /drivergates/PWM_U_H
- C1 pad 1: +12V -> Net-(IC1-HS)
- C1 pad 2: GND -> Net-(D1-K)
- C10 pad 1: Net-(IC7-ACP) -> Net-(U1-VI)
- C10 pad 2: Net-(D4-A) -> GND
- C11 pad 1: /voltageregulators/IC4_vref -> Net-(C11-Pad1)
- C12 pad 1: Net-(D4-A) -> Net-(IC6-AVCC)
- C13 pad 1: Net-(IC7-BTST) -> +2.5V
- C13 pad 2: Net-(IC7-SW_1) -> GND
- C15 pad 1: Net-(IC7-REGN) -> Net-(IC6-TTC)
- C17 pad 1: GND -> Net-(IC6-ACP)
- C17 pad 2: Net-(IC7-SRP) -> Net-(D8-A)
- C18 pad 1: Net-(IC7-SRP) -> /voltageregulators/IC5_VREF
- C18 pad 2: /voltageregulators/BATTIN -> GND
- C20 pad 1: /voltageregulators/BATTIN -> +3.3V
- C21 pad 1: /voltageregulators/BATTIN -> Net-(IC6-BTST)
- C21 pad 2: GND -> Net-(IC6-SW_1)
- C22 pad 1: Net-(IC9-VIN) -> Net-(U3-VI)
- C24 pad 2: Net-(C24-Pad2) -> Net-(IC6-SRP)
- C25 pad 1: GND -> Net-(IC6-SRP)
- C25 pad 2: Net-(IC9-COMP) -> /IO/BATTVIN
- C26 pad 1: GND -> +5V
- C26 pad 2: Net-(IC9-SS) -> GND
- C27 pad 1: GND -> /IO/BATTVIN
- C27 pad 2: Net-(IC9-SLOPE) -> GND
- C28 pad 1: GND -> /IO/BATTVIN
- C28 pad 2: +12V -> GND
- C29 pad 1: Net-(D7-K) -> Net-(IC7-VIN)
- C29 pad 2: /voltageregulators/SW1 -> GND
- C30 pad 1: Net-(D6-K) -> GND
- C30 pad 2: /voltageregulators/SW2 -> Net-(C30-Pad2)
- C31 pad 2: +3.3V -> Net-(IC7-COMP)
- C32 pad 2: +3.3V -> Net-(IC7-SS)
- C33 pad 2: +3.3V -> Net-(IC7-SLOPE)
- C34 pad 1: GND -> Net-(D11-K)
- C34 pad 2: +3.3V -> /voltageregulators/SW1
- C35 pad 1: GND -> Net-(D10-K)
- C35 pad 2: +3.3V -> /voltageregulators/SW2
- C36 pad 1: GND -> +12V
- C36 pad 2: +3.3V -> GND
- C37 pad 1: +3.3V -> GND
- C37 pad 2: GND -> /driverIC/HALL_U
- C38 pad 1: +3.3V -> GND
- C38 pad 2: GND -> /driverIC/HALL_V
- C39 pad 1: +3.3V -> GND
- C39 pad 2: GND -> /driverIC/HALL_W
- C4 pad 1: Net-(C4-Pad1) -> Net-(IC2-HS)
- C4 pad 2: GND -> Net-(D2-K)
- C40 pad 1: +3.3V -> GND
- C40 pad 2: GND -> +3.3V
- C41 pad 1: +3.3V -> GND
- C41 pad 2: GND -> +3.3V
- C42 pad 1: +3.3V -> GND
- C42 pad 2: GND -> Net-(U4-VCCCORE3)
- C43 pad 1: +3.3V -> GND
- C43 pad 2: GND -> +3.3V
- C44 pad 1: +3.3V -> GND
- C44 pad 2: GND -> +3.3V
- C45 pad 1: +3.3V -> GND
- C45 pad 2: GND -> Net-(U4-VCCCORE2)
- C46 pad 1: +3.3V -> GND
- C46 pad 2: GND -> +3.3V
- C47 pad 1: Net-(C47-Pad1) -> GND
- C47 pad 2: Net-(IC10-VDDCORE) -> +3.3V
- C48 pad 1: Net-(C47-Pad1) -> GND
- C48 pad 2: Net-(IC10-VDDCORE) -> Net-(U4-VCCCORE1)
- C49 pad 2: +3.3V -> Net-(D29-A)
- C5 pad 1: Net-(IC7-AVCC) -> +12V
- C50 pad 1: GND -> +3.3V
- C50 pad 2: +3.3V -> GND
- C51 pad 1: GND -> +3.3V
- C51 pad 2: +3.3V -> GND
- C52 pad 1: GND -> +3.3V
- C52 pad 2: +3.3V -> GND
- C53 pad 1: GND -> +3.3V
- C53 pad 2: +3.3V -> GND
- C54 pad 1: GND -> +3.3V
- C54 pad 2: +3.3V -> GND
- C55 pad 1: GND -> +3.3V
- C55 pad 2: +3.3V -> GND
- C56 pad 1: Net-(IC11-HS) -> +3.3V
- C56 pad 2: Net-(DBOOT3-K) -> GND
- C57 pad 1: +12V -> +3.3V
- C58 pad 1: Net-(IC12-HS) -> +3.3V
- C58 pad 2: Net-(DBOOT4-K) -> GND
- C59 pad 1: +12V -> +3.3V
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Other:
- board outline removed
- copper layers 2 -> 4
