File: design/PCBs/MOTORDRIVER/motordriver.kicad_pcb (KiCad board)
At the start: 4 copper layers, 365 parts, among them IC1 LM5109BSDX_NOPB, IC10 LM5109BSDX_NOPB, IC11 LM5109BSDX_NOPB, IC12 LM5109BSDX_NOPB, IC13 INA2181A2IDGSR, IC14 LM5109BSDX_NOPB, IC15 LM5109BSDX_NOPB, IC16 LM5109BSDX_NOPB, IC17 LM5109BSDX_NOPB, IC18 INA2181A2IDGSR, IC2 LM5109BSDX_NOPB, IC3 LM5109BSDX_NOPB, IC4 LM5109BSDX_NOPB, IC5 INA2181A2IDGSR, IC6 BQ24133RGYR, IC7 LM5176PWPR, IC8 ATSAME53J18A-MF, IC9 LM5109BSDX_NOPB, J1 IMU1, J2 IMU2, J3 Conn_01x04_Socket, J4 Screw_Terminal_01x02, J5 1-84952-1, J6 1-84952-1, J7 1-84952-1, P1 USB_C_Plug_USB2.0, Q1 30V 71A, Q10 40V 70A, Q11 30V 71A, Q12 30V 71A, Q13 30V 71A, Q14 30V 71A, Q15 30V 71A, Q16 30V 71A, Q17 30V 71A, Q18 30V 71A, Q19 30V 71A, Q2 30V 71A, Q20 30V 71A, Q21 30V 71A, Q22 30V 71A, Q23 30V 71A, Q24 30V 71A, Q25 30V 71A, Q26 30V 71A, Q27 30V 71A, Q28 30V 71A, Q3 30V 71A, Q4 30V 71A, Q5 30V 71A, Q6 30V 71A, Q7 30V 71A, Q8 30V 71A, Q9 30V 71A, U1 LD1117S25TR_SOT223, U2 LD1117S33TR_SOT223, U3 LD1117S50TR_SOT223, U4 TMC4671-LA, U5 ATSAMD11D14A-M, U6 TMC4671-LA, U7 TMC4671-LA

Commit message: worked on schemtac
Parts:
- added D79: 20Vr 5A, Diode_SMD:D_0603_1608Metric, F.Cu at (215.2, 124.0)
- added D80: 20Vr 5A, Diode_SMD:D_0603_1608Metric, F.Cu at (215.2, 126.6)
- added D81: 20Vr 5A, Diode_SMD:D_0603_1608Metric, F.Cu at (215.2, 129.2)
- added R110: 4.7Ω, Resistor_SMD:R_0603_1608Metric, F.Cu at (219.2, 124.0)
- added R111: 0.01Ω, Resistor_SMD:R_0603_1608Metric, F.Cu at (219.2, 126.5)
- added R112: 0.01Ω, Resistor_SMD:R_0603_1608Metric, F.Cu at (219.2, 129.0)
- D29, D51: value 470mV 500mA -> STATUS
- D31, D47, D70, D71: value LED -> 470mV 500mA
- D33, D50, D73, D74: value 470mV 500mA -> LED
- D52, D53, D76, D77: value 20Vr 5A -> 470mV 500mA
- D56, D57: value 470mV 500mA -> 20Vr 5A
- D75: value 20Vr 5A -> STATUS
- P1: footprint Connector_USB:USB_C_Receptacle_JAE_DX07S024WJ3R400 -> kuben-footprints:USB4110GFA
- R106, R73, R76, R79: value 4.7Ω -> 5Ω
- R108, R109, R82, R83: value 0.01Ω -> 4.7Ω
- R52, R57, R64, R68, R90, R94: value 10kΩ -> 1kΩ
- R53: value 100kΩ -> 10kΩ
- R54: value 1.5kΩ -> 100kΩ
- R55: value 1kΩ -> 1.5kΩ
- R58: value 4.7kΩ -> 10kΩ
- R61, R87, R88: value 1kΩ -> 4.7kΩ
- R65, R92: value 1kΩ -> 10kΩ
- R69, R95: value 100kΩ -> 1kΩ
- R70: value 1.5kΩ -> 10kΩ
- R71: value 5Ω -> 100kΩ
- R72, R99: value 4.7Ω -> 1.5kΩ
- R74, R77: value 5Ω -> 4.7Ω
- R84, R85: value 4.7kΩ -> 0.01Ω
- R96: value 1.5kΩ -> 1kΩ
- R97: value 5Ω -> 10kΩ
- R98: value 4.7Ω -> 100kΩ
- moved P1 20.8 mm to (220.9, 115.5)
Connections:
- net /IO/SERVO_1_SIGNAL renamed /IO/BRAKE1
- net /IO/SERVO_2_SIGNAL renamed /IO/BRAKE2
- net /IO/SERVO_3_SIGNAL renamed /IO/BRAKE3
- net /driverIC/TMC_CS renamed /driverIC/SPI_CS
- net /driverIC/TMC_RX renamed /driverIC/UART_RX
- net /driverIC/TMC_TX renamed /driverIC/UART_TX
- net /driverIC1/TMC_CS renamed /driverIC1/SPI_CS
- net /driverIC1/TMC_RX renamed /driverIC1/UART_RX
- net /driverIC1/TMC_TX renamed /driverIC1/UART_TX
- net /driverIC2/TMC_CS renamed /driverIC2/SPI_CS
- net /driverIC2/TMC_RX renamed /driverIC2/UART_RX
- net /driverIC2/TMC_TX renamed /driverIC2/UART_TX
- C101 pad 2: Net-(D76-K) -> Net-(D79-K)
- C103 pad 2: Net-(D77-K) -> Net-(D80-K)
- C49 pad 2: Net-(D29-A) -> Net-(D30-A)
- C75 pad 2: Net-(D50-A) -> Net-(D52-A)
- C76 pad 2: Net-(D52-K) -> Net-(D54-K)
- C79 pad 2: Net-(D53-K) -> Net-(D55-K)
- C81 pad 2: Net-(D54-K) -> Net-(D56-K)
- C97 pad 2: Net-(D73-A) -> Net-(D76-A)
- C98 pad 2: Net-(D75-K) -> Net-(D78-K)
- D29 pad 1: +5V -> GND
- D30 pad 1: Net-(D29-A) -> +5V
- D30 pad 2: GND -> Net-(D30-A)
- D31 pad 1: GND -> Net-(D30-A)
- D31 pad 2: Net-(D31-A) -> GND
- D33 pad 1: +5V -> GND
- D33 pad 2: /driverIC1/ADC_I0_POS -> Net-(D33-A)
- D34 pad 1: /driverIC1/ADC_I0_POS -> +5V
- D34 pad 2: GND -> /driverIC1/ADC_I0_POS
- D35 pad 1: +5V -> /driverIC1/ADC_I0_POS
- D35 pad 2: /driverIC1/ADC_I1_POS -> GND
- D36 pad 1: /driverIC1/ADC_I1_POS -> +5V
- D36 pad 2: GND -> /driverIC1/ADC_I1_POS
- D37 pad 1: +5V -> /driverIC1/ADC_I1_POS
- D37 pad 2: +2.5V -> GND
- D38 pad 1: +2.5V -> +5V
- D38 pad 2: GND -> +2.5V
- D39 pad 1: +5V -> +2.5V
- D39 pad 2: +2.5V -> GND
- D40 pad 1: +2.5V -> +5V
- D40 pad 2: GND -> +2.5V
- D41 pad 1: +5V -> +2.5V
- D41 pad 2: /driverIC1/HALL_W -> GND
- D42 pad 1: /driverIC1/HALL_W -> +5V
- D42 pad 2: GND -> /driverIC1/HALL_W
- D43 pad 1: +5V -> /driverIC1/HALL_W
- D43 pad 2: /driverIC1/HALL_V -> GND
- D44 pad 1: /driverIC1/HALL_V -> +5V
- D44 pad 2: GND -> /driverIC1/HALL_V
- D45 pad 1: +5V -> /driverIC1/HALL_V
- D45 pad 2: /driverIC1/HALL_U -> GND
- D46 pad 1: /driverIC1/HALL_U -> +5V
- D46 pad 2: GND -> /driverIC1/HALL_U
- D47 pad 1: GND -> /driverIC1/HALL_U
- D47 pad 2: Net-(D47-A) -> GND
- D50 pad 1: +5V -> GND
- D51 pad 1: Net-(D50-A) -> GND
- D51 pad 2: GND -> Net-(D51-A)
- D52 pad 1: Net-(D52-K) -> +5V
- D53 pad 1: Net-(D53-K) -> Net-(D52-A)
- D53 pad 2: Net-(D53-A) -> GND
- D55 pad 1: +12V -> Net-(D55-K)
- D56 pad 1: +5V -> Net-(D56-K)
- D56 pad 2: /driverIC2/ADC_I0_POS -> Net-(D56-A)
- D57 pad 1: /driverIC2/ADC_I0_POS -> +12V
- D57 pad 2: GND -> Net-(D57-A)
- D58 pad 2: /driverIC2/ADC_I1_POS -> /driverIC2/ADC_I0_POS
- D59 pad 1: /driverIC2/ADC_I1_POS -> /driverIC2/ADC_I0_POS
- D60 pad 2: +2.5V -> /driverIC2/ADC_I1_POS
- D61 pad 1: +2.5V -> /driverIC2/ADC_I1_POS
- D64 pad 2: /driverIC2/HALL_W -> +2.5V
- D65 pad 1: /driverIC2/HALL_W -> +2.5V
- D66 pad 2: /driverIC2/HALL_V -> /driverIC2/HALL_W
- D67 pad 1: /driverIC2/HALL_V -> /driverIC2/HALL_W
- D68 pad 2: /driverIC2/HALL_U -> /driverIC2/HALL_V
- D69 pad 1: /driverIC2/HALL_U -> /driverIC2/HALL_V
- D70 pad 1: GND -> +5V
- D70 pad 2: Net-(D70-A) -> /driverIC2/HALL_U
- D71 pad 1: GND -> /driverIC2/HALL_U
- D71 pad 2: Net-(D71-A) -> GND
- D73 pad 1: +5V -> GND
- D74 pad 1: Net-(D73-A) -> GND
- D74 pad 2: GND -> Net-(D74-A)
- D75 pad 1: Net-(D75-K) -> GND
- D76 pad 1: Net-(D76-K) -> +5V
- D77 pad 1: Net-(D77-K) -> Net-(D76-A)
- D77 pad 2: Net-(D77-A) -> GND
- D78 pad 1: +12V -> Net-(D78-K)
- IC10 pad 8: Net-(D53-K) -> Net-(D55-K)
- IC12 pad 8: Net-(D54-K) -> Net-(D56-K)
- IC14 pad 8: Net-(D75-K) -> Net-(D78-K)
- IC15 pad 8: Net-(D76-K) -> Net-(D79-K)
- IC17 pad 8: Net-(D77-K) -> Net-(D80-K)
- IC9 pad 8: Net-(D52-K) -> Net-(D54-K)
- P1 pad A1: GND -> unconnected-(P1-PadA1)
- P1 pad A12: GND -> unconnected-(P1-PadA12)
- P1 pad A4: /IO/USBVIN -> unconnected-(P1-PadA4)
- P1 pad A6: /IO/D+ -> unconnected-(P1-PadA6)
- P1 pad A7: /IO/D- -> unconnected-(P1-PadA7)
- P1 pad A8: (no net) -> unconnected-(P1-PadA8)
- P1 pad A9: /IO/USBVIN -> unconnected-(P1-PadA9)
- P1 pad B1: GND -> unconnected-(P1-PadB1)
- P1 pad B12: GND -> unconnected-(P1-PadB12)
- P1 pad B4: /IO/USBVIN -> unconnected-(P1-PadB4)
- P1 pad B6: (no net) -> unconnected-(P1-PadB6)
- P1 pad B7: (no net) -> unconnected-(P1-PadB7)
- P1 pad B8: (no net) -> unconnected-(P1-PadB8)
- P1 pad B9: /IO/USBVIN -> unconnected-(P1-PadB9)
- Q15 pad 2: Net-(D55-A) -> Net-(D57-A)
- Q22 pad 2: Net-(D78-A) -> Net-(D81-A)
- R100 pad 2: Net-(D76-A) -> Net-(D78-A)
- R101 pad 1: Net-(IC15-HO) -> Net-(IC14-HO)
- R101 pad 2: Net-(Q25-G) -> Net-(Q27-G)
- R102 pad 1: Net-(Q26-G) -> Net-(Q28-G)
- R102 pad 2: Net-(IC15-LO) -> Net-(IC14-LO)
- R103 pad 2: Net-(D77-A) -> Net-(D79-A)
- R104 pad 1: Net-(IC17-HO) -> Net-(IC15-HO)
- R104 pad 2: Net-(Q23-G) -> Net-(Q25-G)
- R105 pad 1: Net-(Q22-G) -> Net-(Q26-G)
- R105 pad 2: Net-(IC16-LO) -> Net-(IC15-LO)
- R106 pad 1: Net-(Q24-G) -> +12V
- R106 pad 2: Net-(IC17-LO) -> Net-(D80-A)
- R107 pad 1: +12V -> Net-(IC17-HO)
- R107 pad 2: Net-(D78-A) -> Net-(Q23-G)
- R108 pad 1: Net-(Q23-S) -> Net-(Q22-G)
- R108 pad 2: Net-(IC18-IN+1) -> Net-(IC16-LO)
- R109 pad 1: Net-(Q25-S) -> Net-(Q24-G)
- R109 pad 2: Net-(IC18-IN+2) -> Net-(IC17-LO)
- R52 pad 1: Net-(U4-NRST) -> Net-(D29-A)
- R52 pad 2: +3.3V -> Net-(U4-STATUS)
- R53 pad 1: +12V -> Net-(U4-NRST)
- R53 pad 2: Net-(D29-A) -> +3.3V
- R54 pad 1: Net-(D29-A) -> +12V
- R54 pad 2: GND -> Net-(D30-A)
- R55 pad 1: Net-(D31-A) -> Net-(D30-A)
- R55 pad 2: /microcontrollers/ERRLED -> GND
- R56 pad 2: /microcontrollers/PROCLED -> /microcontrollers/ERRLED
- R57 pad 1: Net-(U5-PA28/~{RESET}) -> Net-(D33-A)
- R57 pad 2: +3.3V -> /microcontrollers/PROCLED
- R58 pad 1: +5V -> Net-(U5-PA28/~{RESET})
- R58 pad 2: /driverIC1/HALL_U -> +3.3V
- R59 pad 2: /driverIC1/HALL_V -> /driverIC1/HALL_U
- R60 pad 2: /driverIC1/HALL_W -> /driverIC1/HALL_V
- R61 pad 1: /driverIC1/HALL_W -> +5V
- R62 pad 1: /driverIC1/HALL_V -> /driverIC1/HALL_W
- R62 pad 2: /driverIC1/HALL_V -> /driverIC1/HALL_W
- R63 pad 1: /driverIC1/HALL_U -> /driverIC1/HALL_V
- R63 pad 2: /driverIC1/HALL_U -> /driverIC1/HALL_V
- R64 pad 1: /driverIC1/ENI -> /driverIC1/HALL_U
- R64 pad 2: GND -> /driverIC1/HALL_U
- R65 pad 1: Net-(D47-A) -> /driverIC1/ENI
- R65 pad 2: Net-(U6-GPIO5_/_AENC_UX_MCD_/_DBGSPI_MOSI) -> GND
- R66 pad 2: Net-(U6-GPIO6_/_AENC_VN_MCD_/_DBGSPI_MISO) -> Net-(U6-GPIO5_/_AENC_UX_MCD_/_DBGSPI_MOSI)
- R67 pad 2: Net-(U6-GPIO7_/_AENC_WY_MCD_/_DBGSPI_TRG) -> Net-(U6-GPIO6_/_AENC_VN_MCD_/_DBGSPI_MISO)
- R68 pad 1: Net-(U6-NRST) -> Net-(D50-A)
- R68 pad 2: +3.3V -> Net-(U6-GPIO7_/_AENC_WY_MCD_/_DBGSPI_TRG)
- R69 pad 1: +12V -> Net-(D51-A)
- R69 pad 2: Net-(D50-A) -> Net-(U6-STATUS)
- R70 pad 1: Net-(D50-A) -> Net-(U6-NRST)
- R70 pad 2: GND -> +3.3V
- R72 pad 1: Net-(IC9-HO) -> Net-(D52-A)
- R72 pad 2: Net-(Q20-G) -> GND
- R73 pad 1: Net-(Q21-G) -> +12V
- R73 pad 2: Net-(IC9-LO) -> Net-(D54-A)
- R74 pad 1: +12V -> Net-(IC9-HO)
- R74 pad 2: Net-(D53-A) -> Net-(Q20-G)
- R75 pad 1: Net-(IC10-HO) -> Net-(Q21-G)
- R75 pad 2: Net-(Q18-G) -> Net-(IC9-LO)
- R76 pad 1: Net-(Q19-G) -> +12V
- R76 pad 2: Net-(IC10-LO) -> Net-(D55-A)
- R77 pad 1: +12V -> Net-(IC10-HO)
- R77 pad 2: Net-(D54-A) -> Net-(Q18-G)
- R78 pad 1: Net-(IC12-HO) -> Net-(Q19-G)
- R78 pad 2: Net-(Q16-G) -> Net-(IC10-LO)
- R79 pad 1: Net-(Q15-G) -> +12V
- R79 pad 2: Net-(IC11-LO) -> Net-(D56-A)
- R80 pad 1: Net-(Q17-G) -> Net-(IC12-HO)
- R80 pad 2: Net-(IC12-LO) -> Net-(Q16-G)
- R81 pad 1: +12V -> Net-(Q15-G)
- R81 pad 2: Net-(D55-A) -> Net-(IC11-LO)
- R82 pad 1: Net-(Q16-S) -> Net-(Q17-G)
- R82 pad 2: Net-(IC13-IN+1) -> Net-(IC12-LO)
- R83 pad 1: Net-(Q18-S) -> +12V
- R83 pad 2: Net-(IC13-IN+2) -> Net-(D57-A)
- R84 pad 1: +5V -> Net-(Q16-S)
- R84 pad 2: /driverIC2/HALL_U -> Net-(IC13-IN+1)
- R85 pad 1: +5V -> Net-(Q18-S)
- R85 pad 2: /driverIC2/HALL_V -> Net-(IC13-IN+2)
- R86 pad 2: /driverIC2/HALL_W -> /driverIC2/HALL_U
- R87 pad 1: /driverIC2/HALL_W -> +5V
- R87 pad 2: /driverIC2/HALL_W -> /driverIC2/HALL_V
- R88 pad 1: /driverIC2/HALL_V -> +5V
- R88 pad 2: /driverIC2/HALL_V -> /driverIC2/HALL_W
- R89 pad 1: /driverIC2/HALL_U -> /driverIC2/HALL_W
- R89 pad 2: /driverIC2/HALL_U -> /driverIC2/HALL_W
- R90 pad 1: /driverIC2/ENI -> /driverIC2/HALL_V
- R90 pad 2: GND -> /driverIC2/HALL_V
- R91 pad 1: Net-(D70-A) -> /driverIC2/HALL_U
- R91 pad 2: Net-(U7-GPIO5_/_AENC_UX_MCD_/_DBGSPI_MOSI) -> /driverIC2/HALL_U
- R92 pad 1: Net-(D71-A) -> /driverIC2/ENI
- R92 pad 2: Net-(U7-GPIO6_/_AENC_VN_MCD_/_DBGSPI_MISO) -> GND
- R93 pad 2: Net-(U7-GPIO7_/_AENC_WY_MCD_/_DBGSPI_TRG) -> Net-(U7-GPIO5_/_AENC_UX_MCD_/_DBGSPI_MOSI)
- R94 pad 1: Net-(U7-NRST) -> Net-(D73-A)
- R94 pad 2: +3.3V -> Net-(U7-GPIO6_/_AENC_VN_MCD_/_DBGSPI_MISO)
- R95 pad 1: +12V -> Net-(D74-A)
- R95 pad 2: Net-(D73-A) -> Net-(U7-GPIO7_/_AENC_WY_MCD_/_DBGSPI_TRG)
- R96 pad 1: Net-(D73-A) -> Net-(D75-A)
- R96 pad 2: GND -> Net-(U7-STATUS)
- R97 pad 1: +12V -> Net-(U7-NRST)
- R97 pad 2: Net-(D75-A) -> +3.3V
- R98 pad 1: Net-(IC14-HO) -> +12V
- R98 pad 2: Net-(Q27-G) -> Net-(D76-A)
- R99 pad 1: Net-(Q28-G) -> Net-(D76-A)
- R99 pad 2: Net-(IC14-LO) -> GND
- U4 pad 12: /driverIC/STATUS -> Net-(U4-STATUS)
- U4 pad 20: Net-(D29-A) -> Net-(D30-A)
- U6 pad 12: /driverIC1/STATUS -> Net-(U6-STATUS)
- U6 pad 20: Net-(D50-A) -> Net-(D52-A)
- U7 pad 12: /driverIC2/STATUS -> Net-(U7-STATUS)
- U7 pad 20: Net-(D73-A) -> Net-(D76-A)
