File: designfiles/electronics/MOTORDRIVER/IO.kicad_sch (KiCad schematic)
At the start: 22 parts, among them J1 Conn_01x04_Socket, J3 IMU1, J4 IMU2, J6 XT60-M, P1 USB_C_Plug_USB2.0, SW1 PUSH

Commit message: worked on pcb
Parts:
- renumbered J3 to J1, J4 to J2, J1 to J3, J6 to J4, R73 to R43, R72 to R44, R5 to R45, TP3 to TP2, TP4 to TP3, TP6 to TP4, TP2 to TP6
Changed lines of the file:
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@@
 		(on_board yes)
 		(dnp no)
-		(property "Reference" "TP2"
+		(property "Reference" "TP6"
 			(at 226.06 123.444 90)
 			(effects
@@
 			(project "motordriver"
 				(path "/c7634e88-16d1-45ec-9aac-9c841e03cf6d/38bc72d2-c2f6-4538-9c33-e1ab2a8ac987"
-					(reference "TP2")
+					(reference "TP6")
 					(unit 1)
 				)
@@
 		(on_board yes)
 		(dnp no)
-		(property "Reference" "TP4"
+		(property "Reference" "TP3"
 			(at 180.594 122.174 90)
 			(effects
@@
 			(project "motordriver"
 				(path "/c7634e88-16d1-45ec-9aac-9c841e03cf6d/38bc72d2-c2f6-4538-9c33-e1ab2a8ac987"
-					(reference "TP4")
+					(reference "TP3")
 					(unit 1)
 				)
@@
 		(dnp no)
 		(fields_autoplaced yes)
-		(property "Reference" "J4"
+		(property "Reference" "J2"
 			(at 102.87 101.6 0)
 			(effects
@@
 			(project "motordriver"
 				(path "/c7634e88-16d1-45ec-9aac-9c841e03cf6d/38bc72d2-c2f6-4538-9c33-e1ab2a8ac987"
-					(reference "J4")
+					(reference "J2")
 					(unit 1)
 				)
@@
 		(dnp no)
 		(fields_autoplaced yes)
-		(property "Reference" "R5"
+		(property "Reference" "R45"
 			(at 191.77 40.6399 0)
 			(effects
@@
 			(project ""
 				(path "/c7634e88-16d1-45ec-9aac-9c841e03cf6d/38bc72d2-c2f6-4538-9c33-e1ab2a8ac987"
-					(reference "R5")
+					(reference "R45")
 					(unit 1)
 				)
@@
 		(dnp no)
 		(fields_autoplaced yes)
-		(property "Reference" "R72"
+		(property "Reference" "R44"
 			(at 76.2 83.82 90)
 			(effects
@@
 			(project "motordriver"
 				(path "/c7634e88-16d1-45ec-9aac-9c841e03cf6d/38bc72d2-c2f6-4538-9c33-e1ab2a8ac987"
-					(reference "R72")
+					(reference "R44")
 					(unit 1)
 				)
@@
 		(on_board yes)
 		(dnp no)
-		(property "Reference" "TP6"
+		(property "Reference" "TP4"
 			(at 225.806 117.856 90)
 			(effects
@@
 			(project "motordriver"
 				(path "/c7634e88-16d1-45ec-9aac-9c841e03cf6d/38bc72d2-c2f6-4538-9c33-e1ab2a8ac987"
-					(reference "TP6")
+					(reference "TP4")
 					(unit 1)
 				)
@@
 		(dnp no)
 		(fields_autoplaced yes)
-		(property "Reference" "J3"
+		(property "Reference" "J1"
 			(at 102.87 74.93 0)
 			(effects
@@
 			(project "motordriver"
 				(path "/c7634e88-16d1-45ec-9aac-9c841e03cf6d/38bc72d2-c2f6-4538-9c33-e1ab2a8ac987"
-					(reference "J3")
+					(reference "J1")
 					(unit 1)
 				)
@@
 		(on_board yes)
 		(dnp no)
-		(property "Reference" "TP3"
+		(property "Reference" "TP2"
 			(at 180.594 119.38 90)
 			(effects
@@
 			(project "motordriver"
 				(path "/c7634e88-16d1-45ec-9aac-9c841e03cf6d/38bc72d2-c2f6-4538-9c33-e1ab2a8ac987"
-					(reference "TP3")
+					(reference "TP2")
 					(unit 1)
 				)
@@
 		(dnp no)
 		(fields_autoplaced yes)
-		(property "Reference" "R73"
+		(property "Reference" "R43"
 			(at 27.94 88.9 90)
 			(effects
@@
 			(project "motordriver"
 				(path "/c7634e88-16d1-45ec-9aac-9c841e03cf6d/38bc72d2-c2f6-4538-9c33-e1ab2a8ac987"
-					(reference "R73")
+					(reference "R43")
 					(unit 1)
 				)
@@
 		(dnp no)
 		(fields_autoplaced yes)
-		(property "Reference" "J6"
+		(property "Reference" "J4"
 			(at 246.38 87.6299 0)
 			(effects
@@
 			(project ""
 				(path "/c7634e88-16d1-45ec-9aac-9c841e03cf6d/38bc72d2-c2f6-4538-9c33-e1ab2a8ac987"
-					(reference "J6")
+					(reference "J4")
 					(unit 1)
 				)
@@
 		(on_board yes)
 		(dnp no)
-		(property "Reference" "J1"
+		(property "Reference" "J3"
 			(at 196.85 90.1701 0)
 			(effects
@@
 			(project ""
 				(path "/c7634e88-16d1-45ec-9aac-9c841e03cf6d/38bc72d2-c2f6-4538-9c33-e1ab2a8ac987"
-					(reference "J1")
+					(reference "J3")
 					(unit 1)
 				)

Commit message: worked on pcb
Connections:
- net GND: now also P1.MP1, P1.MP2, P1.MP3, P1.MP4
- no-connect marks 10 -> 6
