File: designfiles/electronics/MOTORDRIVER/microcontrollers.kicad_sch (KiCad schematic)
At the start: 27 parts, among them IC8 ATSAME53J18A-MF, U5 ATSAMD11D14A-M

Commit message: added inductors
Parts:
- removed C65, C67: 100nF, Capacitor_SMD:C_0603_1608Metric, symbol Device:C
- removed C75: 4.7µF, Capacitor_SMD:C_0603_1608Metric, symbol Device:C
- added C76: 10µF, Capacitor_SMD:C_0603_1608Metric, symbol Device:C
- added C77, C79, C80: 100nF, Capacitor_SMD:C_0603_1608Metric, symbol Device:C
- added C78: 4.7µF, Capacitor_SMD:C_0603_1608Metric, symbol Device:C
- IC8: footprint kuben-footprints:QFN50P900X900X100-65N-D -> QFN50P900X900X100-65N-D
- U5: footprint kuben-footprints:QFN50P400X400X90-25N-D -> QFN50P400X400X90-25N-D
- renumbered C69 to C65, C68 to C67, C71 to C68, C70 to C69, C73 to C70, C72 to C71, C76 to C72, C74 to C73, C77 to C74, C78 to C75, D31 to D30, D32 to D31, D33 to D32, D34 to D33, D35 to D34
Connections:
- net +3.3V: now also C76.1, C80.1
- net GND: now also C76.2, C77.1, C78.1, C79.2, C80.2
- net RESETN: now also C79.1
- net at IC8.53 (VDDCORE): now also C77.2, C78.2
Other:
- note added: "Decoupling capacitors, place them close to VDD on ICs"
- note removed: "Decoupling capacitors, place them close to IC"
- moved on the sheet: C65, C66, C68, C70, C72, C74, C75

Commit message: double checked SERCOM again, as well as PWM and interrupt pin capabilities
Connections:
- net BRAKE1: now also IC8.39 (PB16); no longer IC8.28 (PB15)
- net BRAKE2: now also IC8.40 (PB17); no longer IC8.29 (PA12)
- net OLED_SCL: now also IC8.30 (PA13); no longer IC8.44 (PA23)
- net OLED_SDA: now also IC8.29 (PA12); no longer IC8.43 (PA22)
- net RX: now also IC8.37 (PA18); no longer IC8.30 (PA13)
- net SERVO1_PWM_I: now also IC8.41 (PA20); no longer IC8.25 (PB12)
- net SERVO2_PWM_I: now also IC8.42 (PA21); no longer IC8.26 (PB13)
- net SERVO3_PWM_I: now also IC8.43 (PA22); no longer IC8.27 (PB14)
- net SPI_SCK: now also IC8.44 (PA23); no longer IC8.42 (PA21)
- net TMC_DB_MISO: now also IC8.25 (PB12); no longer IC8.39 (PB16)
- net TMC_DB_MOSI: now also IC8.26 (PB13); no longer IC8.40 (PB17)
- net TMC_DB_SCK: now also IC8.27 (PB14); no longer IC8.41 (PA20)
- net TX: now also IC8.38 (PA19); no longer IC8.31 (PA14)
- no-connect marks 19 -> 26
Other:
- note removed: "25MHz CLK for servocontroller"
- note removed: "Enable servocontrollers"
Changed lines of the file:
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@@
 	)
 	(no_connect
+		(at 118.11 120.65)
+	)
+	(no_connect
 		(at 265.43 102.87)
 	)
@@
 	)
 	(no_connect
+		(at 118.11 125.73)
+	)
+	(no_connect
 		(at 151.13 69.85)
 	)
@@
 	)
 	(no_connect
+		(at 118.11 95.25)
+	)
+	(no_connect
+		(at 118.11 128.27)
+	)
+	(no_connect
 		(at 224.79 102.87)
 	)
@@
 	)
 	(no_connect
+		(at 118.11 118.11)
+	)
+	(no_connect
 		(at 224.79 100.33)
 	)
 	(no_connect
+		(at 118.11 115.57)
+	)
+	(no_connect
 		(at 224.79 92.71)
 	)
 	(no_connect
+		(at 118.11 123.19)
+	)
+	(no_connect
 		(at 237.49 118.11)
 	)
@@
 	(text_box "SERCOM4"
 		(exclude_from_sim no)
-		(at 157.48 157.48 90)
-		(size 5.08 10.16)
+		(at 144.78 160.02 90)
+		(size 7.62 10.16)
 		(stroke
 			(width 0)
@@
 		)
 	)
-	(text_box "SERCOM3"
+	(text_box "SERCOM5"
 		(exclude_from_sim no)
 		(at 189.23 93.98 0)
-		(size 10.16 5.08)
+		(size 10.16 7.62)
 		(stroke
 			(width 0)
@@
 		)
 	)
-	(text_box "SERCOM2"
+	(text_box "SERCOM2\n"
 		(exclude_from_sim no)
-		(at 189.23 99.06 0)
-		(size 10.16 5.08)
-		(stroke
-			(width 0)
-			(type default)
-		)
-		(fill
-			(type none)
-		)
-		(effects
-			(font
-				(size 1.27 1.27)
-			)
-			(justify left top)
-		)
-	)
-	(text_box "SERCOM5"
-		(exclude_from_sim no)
-		(at 189.23 109.22 0)
-		(size 10.16 5.08)
+		(at 154.94 156.21 90)
+		(size 5.08 10.16)
 		(stroke
 			(width 0)
@@
 		)
 	)
-	(text_box "SERCOM3"
+	(text_box "SERCOM3\n"
 		(exclude_from_sim no)
-		(at 189.23 104.14 0)
-		(size 10.16 2.54)
+		(at 189.23 114.935 0)
+		(size 10.16 4.445)
 		(stroke
 			(width 0)
@@
 		)
 	)
-	(text "Enable\nservocontrollers"
-		(exclude_from_sim no)
-		(at 141.732 163.83 0)
-		(effects
-			(font
-				(size 1.27 1.27)
-			)
-		)
-	)
-	(text "25MHz CLK\nfor servocontroller"
-		(exclude_from_sim no)
-		(at 141.732 168.91 0)
-		(effects
-			(font
-				(size 1.27 1.27)
-			)
-		)
-	)
 	(text "Programmer"
 		(exclude_from_sim no)
@@
 	(global_label "SPI_SCK"
 		(shape input)
-		(at 173.99 105.41 0)
+		(at 173.99 100.33 0)
 		(fields_autoplaced yes)
 		(effects
@@
 		)
 		(property "Intersheetrefs" "${INTERSHEET_REFS}"
-			(at 184.2221 105.41 0)
+			(at 184.2221 100.33 0)
 			(effects
 				(font
@@
 	(global_label "TMC_DB_SCK"
 		(shape input)
-		(at 173.99 107.95 0)
+		(at 151.13 146.05 270)
 		(fields_autoplaced yes)
 		(effects
@@
 				(size 1.27 1.27)
 			)
-			(justify left)
+			(justify right)
 		)
 		(property "Intersheetrefs" "${INTERSHEET_REFS}"
-			(at 187.4232 107.95 0)
+			(at 151.13 159.4832 90)
 			(effects
 				(font
 					(size 1.27 1.27)
 				)
-				(justify left)
+				(justify right)
 				(hide yes)
 			)
@@
 	(global_label "TMC_DB_MISO"
 		(shape input)
-		(at 173.99 113.03 0)
+		(at 146.05 146.05 270)
 		(fields_autoplaced yes)
 		(effects
@@
 				(size 1.27 1.27)
 			)
-			(justify left)
+			(justify right)
 		)
 		(property "Intersheetrefs" "${INTERSHEET_REFS}"
-			(at 188.4903 113.03 0)
+			(at 146.05 160.5503 90)
 			(effects
 				(font
 					(size 1.27 1.27)
 				)
-				(justify left)
+				(justify right)
 				(hide yes)
 			)
@@
 	(global_label "TMC_DB_MOSI"
 		(shape input)
-		(at 173.99 110.49 0)
+		(at 148.59 146.05 270)
 		(fields_autoplaced yes)
 		(effects
@@
 				(size 1.27 1.27)
 			)
-			(justify left)
+			(justify right)
 		)
 		(property "Intersheetrefs" "${INTERSHEET_REFS}"
-			(at 188.4903 110.49 0)
+			(at 148.59 160.5503 90)
 			(effects
 				(font
 					(size 1.27 1.27)
 				)
-				(justify left)
+				(justify right)
 				(hide yes)
 			)
@@
 	(hierarchical_label "BRAKE2"
 		(shape input)
-		(at 156.21 146.05 270)
+		(at 173.99 110.49 0)
 		(fields_autoplaced yes)
 		(effects
@@
 				(size 1.27 1.27)
 			)
-			(justify right)
+			(justify left)
 		)
 	)
@@
 	(hierarchical_label "RX"
 		(shape input)
-		(at 158.75 146.05 270)
+		(at 173.99 118.11 0)
 		(fields_autoplaced yes)
 		(effects
@@
 				(size 1.27 1.27)
 			)
-			(justify right)
+			(justify left)
 		)
 	)
 	(hierarchical_label "TX"
 		(shape input)
-		(at 161.29 146.05 270)
+		(at 173.99 115.57 0)
 		(fields_autoplaced yes)
 		(effects
@@
 				(size 1.27 1.27)
 			)
-			(justify right)
+			(justify left)
 		)
 	)
@@
 	(hierarchical_label "BRAKE1"
 		(shape input)
-		(at 153.67 146.05 270)
+		(at 173.99 113.03 0)
 		(fields_autoplaced yes)
 		(effects
@@
 				(size 1.27 1.27)
 			)
-			(justify right)
+			(justify left)
 		)
 	)
@@
 	(hierarchical_label "SERVO2_PWM_I"
 		(shape input)
-		(at 148.59 146.05 270)
+		(at 173.99 105.41 0)
 		(fields_autoplaced yes)
 		(effects
@@
 				(size 1.27 1.27)
 			)
-			(justify right)
+			(justify left)
 		)
 	)
@@
 	(hierarchical_label "OLED_SCL"
 		(shape input)
-		(at 173.99 100.33 0)
+		(at 158.75 146.05 270)
 		(fields_autoplaced yes)
 		(effects
@@
 				(size 1.27 1.27)
 			)
-			(justify left)
+			(justify right)
 		)
 	)
@@
 	(hierarchical_label "SERVO1_PWM_I"
 		(shape input)
-		(at 146.05 146.05 270)
+		(at 173.99 107.95 0)
 		(fields_autoplaced yes)
 		(effects
@@
 				(size 1.27 1.27)
 			)
-			(justify right)
+			(justify left)
 		)
 	)
 	(hierarchical_label "SERVO3_PWM_I"
 		(shape input)
-		(at 151.13 146.05 270)
+		(at 173.99 102.87 0)
 		(fields_autoplaced yes)
 		(effects
@@
 				(size 1.27 1.27)
 			)
-			(justify right)
+			(justify left)
 		)
 	)
 	(hierarchical_label "OLED_SDA"
 		(shape input)
-		(at 173.99 102.87 0)
+		(at 156.21 146.05 270)
 		(fields_autoplaced yes)
 		(effects
@@
 				(size 1.27 1.27)
 			)
-			(justify left)
+			(justify right)
 		)
 	)
@@
 		(dnp no)
 		(property "Reference" "U5"
-			(at 260.604 70.866 0)
+			(at 260.096 64.77 0)
 			(effects
 				(font
@@
 		)
 		(property "Value" "ATSAMD11D14A-M"
-			(at 261.112 73.406 0)
+			(at 260.858 67.31 0)
 			(effects
 				(font

Commit message: minor tweaks on schematic and started on the pcb layout, made good work
Parts:
- IC8: footprint QFN50P900X900X100-65N-D -> kuben-footprints:QFN50P900X900X100-65N-D
- U5: footprint QFN50P400X400X90-25N-D -> kuben-footprints:QFN50P400X400X90-25N-D
Changed lines of the file:
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@@
 	(text_box "SERCOM0"
 		(exclude_from_sim no)
-		(at 124.46 157.48 90)
+		(at 124.46 160.02 90)
 		(size 5.08 10.16)
 		(stroke
@@
 	(text_box "SERCOM2\n"
 		(exclude_from_sim no)
-		(at 154.94 156.21 90)
+		(at 154.94 160.02 90)
 		(size 5.08 10.16)
 		(stroke
@@
 			)
 		)
-		(property "Footprint" "QFN50P400X400X90-25N-D"
+		(property "Footprint" "kuben-footprints:QFN50P400X400X90-25N-D"
 			(at 261.62 174.93 0)
 			(effects
@@
 			)
 		)
-		(property "Footprint" "QFN50P900X900X100-65N-D"
+		(property "Footprint" "kuben-footprints:QFN50P900X900X100-65N-D"
 			(at 170.18 172.39 0)
 			(effects

Commit message: worked on PCB
Connections:
- net INT_IMU3: now reaches IC8.11 (PB08)
- net INT1_IMU1 renamed INT_IMU2
- net INT1_IMU2 renamed INT_IMU1
- no-connect marks 26 -> 25
Changed lines of the file:
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@@
-	)
-	(no_connect
-		(at 118.11 115.57)
 	)
 	(no_connect
@@
 		)
 	)
+	(hierarchical_label "SDA_IMU3"
+		(shape input)
+		(at 114.3 147.32 270)
+		(fields_autoplaced yes)
+		(effects
+			(font
+				(size 1.27 1.27)
+			)
+			(justify right)
+		)
+	)
 	(hierarchical_label "SDA_IMU2"
 		(shape input)
@@
 		)
 	)
+	(hierarchical_label "INT_IMU3"
+		(shape input)
+		(at 118.11 115.57 180)
+		(fields_autoplaced yes)
+		(effects
+			(font
+				(size 1.27 1.27)
+			)
+			(justify right)
+		)
+	)
 	(hierarchical_label "SWDIO"
 		(shape input)
@@
 		)
 	)
-	(hierarchical_label "INT1_IMU2"
+	(hierarchical_label "INT_IMU2"
+		(shape input)
+		(at 118.11 113.03 180)
+		(fields_autoplaced yes)
+		(effects
+			(font
+				(size 1.27 1.27)
+			)
+			(justify right)
+		)
+	)
+	(hierarchical_label "OLED_SCL"
+		(shape input)
+		(at 158.75 146.05 270)
+		(fields_autoplaced yes)
+		(effects
+			(font
+				(size 1.27 1.27)
+			)
+			(justify right)
+		)
+	)
+	(hierarchical_label "SERVO1_CS"
+		(shape input)
+		(at 128.27 69.85 90)
+		(fields_autoplaced yes)
+		(effects
+			(font
+				(size 1.27 1.27)
+			)
+			(justify left)
+		)
+	)
+	(hierarchical_label "SCL_IMU3"
+		(shape input)
+		(at 116.84 147.32 270)
+		(fields_autoplaced yes)
+		(effects
+			(font
+				(size 1.27 1.27)
+			)
+			(justify right)
+		)
+	)
+	(hierarchical_label "SERVO1_PWM_I"
+		(shape input)
+		(at 173.99 107.95 0)
+		(fields_autoplaced yes)
+		(effects
+			(font
+				(size 1.27 1.27)
+			)
+			(justify left)
+		)
+	)
+	(hierarchical_label "SERVO3_PWM_I"
+		(shape input)
+		(at 173.99 102.87 0)
+		(fields_autoplaced yes)
+		(effects
+			(font
+				(size 1.27 1.27)
+			)
+			(justify left)
+		)
+	)
+	(hierarchical_label "OLED_SDA"
+		(shape input)
+		(at 156.21 146.05 270)
+		(fields_autoplaced yes)
+		(effects
+			(font
+				(size 1.27 1.27)
+			)
+			(justify right)
+		)
+	)
+	(hierarchical_label "INT_IMU1"
 		(shape input)
 		(at 118.11 110.49 180)
 		(fields_autoplaced yes)
 		(effects
-			(font
-				(size 1.27 1.27)
-			)
-			(justify right)
-		)
-	)
-	(hierarchical_label "OLED_SCL"
-		(shape input)
-		(at 158.75 146.05 270)
-		(fields_autoplaced yes)
-		(effects
-			(font
-				(size 1.27 1.27)
-			)
-			(justify right)
-		)
-	)
-	(hierarchical_label "SERVO1_CS"
-		(shape input)
-		(at 128.27 69.85 90)
-		(fields_autoplaced yes)
-		(effects
-			(font
-				(size 1.27 1.27)
-			)
-			(justify left)
-		)
-	)
-	(hierarchical_label "SERVO1_PWM_I"
-		(shape input)
-		(at 173.99 107.95 0)
-		(fields_autoplaced yes)
-		(effects
-			(font
-				(size 1.27 1.27)
-			)
-			(justify left)
-		)
-	)
-	(hierarchical_label "SERVO3_PWM_I"
-		(shape input)
-		(at 173.99 102.87 0)
-		(fields_autoplaced yes)
-		(effects
-			(font
-				(size 1.27 1.27)
-			)
-			(justify left)
-		)
-	)
-	(hierarchical_label "OLED_SDA"
-		(shape input)
-		(at 156.21 146.05 270)
-		(fields_autoplaced yes)
-		(effects
-			(font
-				(size 1.27 1.27)
-			)
-			(justify right)
-		)
-	)
-	(hierarchical_label "INT1_IMU1"
-		(shape input)
-		(at 118.11 113.03 180)
-		(fields_autoplaced yes)
-		(effects

Commit message: worked on PCB
Parts:
- renumbered C74 to C109, C70 to C110, C73 to C111, C80 to C112, C65 to C113, C66 to C114, C71 to C115, C77 to C116, C72 to C117, C69 to C118, C79 to C119, C78 to C120, C75 to C125, C76 to C126, C68 to C71, C67 to C74, D32 to D45, D33 to D49, D31 to D52, D30 to D53, D34 to D55, IC8 to IC3, R60 to R59, R59 to R62, R61 to R63, R62 to R64, R63 to R65, R58 to R66, U5 to U7

Commit message: worked on pcb
Parts:
- renumbered C113 to C65, C114 to C66, C74 to C67, C71 to C68, C118 to C69, C110 to C70, C115 to C71, C117 to C72, C111 to C73, C109 to C74, C125 to C75, C126 to C76, C116 to C77, C120 to C78, C119 to C79, C112 to C80, D53 to D30, D52 to D31, D45 to D32, D49 to D33, D55 to D34, IC3 to IC8, R66 to R58, R62 to R59, R59 to R60, R63 to R61, R64 to R62, R65 to R63, U7 to U5
Connections:
- net INT_IMU3: no longer names the net of IC8.11 (PB08)
- no-connect marks 25 -> 30
