File: designfiles/electronics/MOTORDRIVER/motorIO.kicad_sch (KiCad schematic)
At the start: 3 parts, among them J5 1-84952-1, J6 1-84952-1, J7 1-84952-1

Commit message: added inductors
Parts:
- J5, J6, J7: footprint kuben-footprints:1849521 -> 1849521
Changed lines of the file:
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@@
 		(dnp no)
 		(fields_autoplaced yes)
-		(property "Reference" "#PWR0312"
+		(property "Reference" "#PWR0317"
 			(at 255.27 113.03 0)
 			(effects
@@
 			(project "motordriver"
 				(path "/c7634e88-16d1-45ec-9aac-9c841e03cf6d/5d8f5153-26a2-4903-a925-dc0c63f77bf7"
-					(reference "#PWR0312")
+					(reference "#PWR0317")
 					(unit 1)
 				)
@@
 			)
 		)
-		(property "Footprint" "kuben-footprints:1849521"
+		(property "Footprint" "1849521"
 			(at 154.94 186.36 0)
 			(effects
@@
 		(dnp no)
 		(fields_autoplaced yes)
-		(property "Reference" "#PWR0307"
+		(property "Reference" "#PWR0312"
 			(at 97.79 123.19 0)
 			(effects
@@
 			(project "motordriver"
 				(path "/c7634e88-16d1-45ec-9aac-9c841e03cf6d/5d8f5153-26a2-4903-a925-dc0c63f77bf7"
-					(reference "#PWR0307")
+					(reference "#PWR0312")
 					(unit 1)
 				)
@@
 			)
 		)
-		(property "Footprint" "kuben-footprints:1849521"
+		(property "Footprint" "1849521"
 			(at 231.14 186.36 0)
 			(effects
@@
 		(dnp no)
 		(fields_autoplaced yes)
-		(property "Reference" "#PWR0308"
+		(property "Reference" "#PWR0313"
 			(at 104.14 115.57 0)
 			(effects
@@
 			(project "motordriver"
 				(path "/c7634e88-16d1-45ec-9aac-9c841e03cf6d/5d8f5153-26a2-4903-a925-dc0c63f77bf7"
-					(reference "#PWR0308")
+					(reference "#PWR0313")
 					(unit 1)
 				)
@@
 		(dnp no)
 		(fields_autoplaced yes)
-		(property "Reference" "#PWR0311"
+		(property "Reference" "#PWR0316"
 			(at 248.92 120.65 0)
 			(effects
@@
 			(project "motordriver"
 				(path "/c7634e88-16d1-45ec-9aac-9c841e03cf6d/5d8f5153-26a2-4903-a925-dc0c63f77bf7"
-					(reference "#PWR0311")
+					(reference "#PWR0316")
 					(unit 1)
 				)
@@
 		(dnp no)
 		(fields_autoplaced yes)
-		(property "Reference" "#PWR0310"
+		(property "Reference" "#PWR0315"
 			(at 179.07 113.03 0)
 			(effects
@@
 			(project "motordriver"
 				(path "/c7634e88-16d1-45ec-9aac-9c841e03cf6d/5d8f5153-26a2-4903-a925-dc0c63f77bf7"
-					(reference "#PWR0310")
+					(reference "#PWR0315")
 					(unit 1)
 				)
@@
 			)
 		)
-		(property "Footprint" "kuben-footprints:1849521"
+		(property "Footprint" "1849521"
 			(at 80.01 188.9 0)
 			(effects
@@
 		(dnp no)
 		(fields_autoplaced yes)
-		(property "Reference" "#PWR0309"
+		(property "Reference" "#PWR0314"
 			(at 172.72 120.65 0)
 			(effects
@@
 			(project "motordriver"
 				(path "/c7634e88-16d1-45ec-9aac-9c841e03cf6d/5d8f5153-26a2-4903-a925-dc0c63f77bf7"
-					(reference "#PWR0309")
-					(unit 1)
-				)
+					(reference "#PWR0314")
+					(unit 1)
+				)

Commit message: minor tweaks on schematic and started on the pcb layout, made good work
Parts:
- J5, J6, J7: footprint 1849521 -> kuben-footprints:1849521
Changed lines of the file:
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@@
 			)
 		)
-		(property "Footprint" "1849521"
+		(property "Footprint" "kuben-footprints:1849521"
 			(at 154.94 186.36 0)
 			(effects
@@
 			)
 		)
-		(property "Footprint" "1849521"
+		(property "Footprint" "kuben-footprints:1849521"
 			(at 231.14 186.36 0)
 			(effects
@@
 			)
 		)
-		(property "Footprint" "1849521"
+		(property "Footprint" "kuben-footprints:1849521"
 			(at 80.01 188.9 0)
 			(effects

Commit message: worked on PCB
Parts:
- renumbered J7 to J2, J6 to J7
Changed lines of the file:
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@@
 		(dnp no)
 		(fields_autoplaced yes)
-		(property "Reference" "#PWR0317"
+		(property "Reference" "#PWR0318"
 			(at 255.27 113.03 0)
 			(effects
@@
 			(project "motordriver"
 				(path "/c7634e88-16d1-45ec-9aac-9c841e03cf6d/5d8f5153-26a2-4903-a925-dc0c63f77bf7"
-					(reference "#PWR0317")
+					(reference "#PWR0318")
 					(unit 1)
 				)
@@
 		(dnp no)
 		(fields_autoplaced yes)
-		(property "Reference" "J6"
+		(property "Reference" "J7"
 			(at 146.05 83.82 0)
 			(effects
@@
 			(project "motordriver"
 				(path "/c7634e88-16d1-45ec-9aac-9c841e03cf6d/5d8f5153-26a2-4903-a925-dc0c63f77bf7"
-					(reference "J6")
+					(reference "J7")
 					(unit 1)
 				)
@@
 		(dnp no)
 		(fields_autoplaced yes)
-		(property "Reference" "#PWR0312"
+		(property "Reference" "#PWR0313"
 			(at 97.79 123.19 0)
 			(effects
@@
 			(project "motordriver"
 				(path "/c7634e88-16d1-45ec-9aac-9c841e03cf6d/5d8f5153-26a2-4903-a925-dc0c63f77bf7"
-					(reference "#PWR0312")
+					(reference "#PWR0313")
 					(unit 1)
 				)
@@
 		(dnp no)
 		(fields_autoplaced yes)
-		(property "Reference" "J7"
+		(property "Reference" "J2"
 			(at 222.25 83.82 0)
 			(effects
@@
 			(project "motordriver"
 				(path "/c7634e88-16d1-45ec-9aac-9c841e03cf6d/5d8f5153-26a2-4903-a925-dc0c63f77bf7"
-					(reference "J7")
+					(reference "J2")
 					(unit 1)
 				)
@@
 		(dnp no)
 		(fields_autoplaced yes)
-		(property "Reference" "#PWR0313"
+		(property "Reference" "#PWR0314"
 			(at 104.14 115.57 0)
 			(effects
@@
 			(project "motordriver"
 				(path "/c7634e88-16d1-45ec-9aac-9c841e03cf6d/5d8f5153-26a2-4903-a925-dc0c63f77bf7"
-					(reference "#PWR0313")
+					(reference "#PWR0314")
 					(unit 1)
 				)
@@
 		(dnp no)
 		(fields_autoplaced yes)
-		(property "Reference" "#PWR0316"
+		(property "Reference" "#PWR0317"
 			(at 248.92 120.65 0)
 			(effects
@@
 			(project "motordriver"
 				(path "/c7634e88-16d1-45ec-9aac-9c841e03cf6d/5d8f5153-26a2-4903-a925-dc0c63f77bf7"
-					(reference "#PWR0316")
+					(reference "#PWR0317")
 					(unit 1)
 				)
@@
 		(dnp no)
 		(fields_autoplaced yes)
-		(property "Reference" "#PWR0315"
+		(property "Reference" "#PWR0316"
 			(at 179.07 113.03 0)
 			(effects
@@
 			(project "motordriver"
 				(path "/c7634e88-16d1-45ec-9aac-9c841e03cf6d/5d8f5153-26a2-4903-a925-dc0c63f77bf7"
-					(reference "#PWR0315")
+					(reference "#PWR0316")
 					(unit 1)
 				)
@@
 		(dnp no)
 		(fields_autoplaced yes)
-		(property "Reference" "#PWR0314"
+		(property "Reference" "#PWR0315"
 			(at 172.72 120.65 0)
 			(effects
@@
 			(project "motordriver"
 				(path "/c7634e88-16d1-45ec-9aac-9c841e03cf6d/5d8f5153-26a2-4903-a925-dc0c63f77bf7"
-					(reference "#PWR0314")
-					(unit 1)
-				)
+					(reference "#PWR0315")
+					(unit 1)
+				)

Commit message: worked on pcb
Parts:
- removed J2: 1-84952-1, kuben-footprints:1849521, symbol 1-84952-1:1-84952-1
- added J7: 1-84952-1, kuben-footprints:1849521, symbol 1-84952-1:1-84952-1
- renumbered J7 to J6
Connections:
- net +12V: now also J5.1, J6.1, J7.1; no longer J5.11, J6.11
- net GND: now also J5.5, J6.5, J7.5; no longer J5.7, J6.7
- net HALL_A1: now also J5.3; no longer J5.9
- net HALL_A2: now also J6.3; no longer J6.9
- net HALL_A3: now also J7.3
- net HALL_B1: now also J5.4; no longer J5.8
- net HALL_B2: now also J6.4; no longer J6.8
- net HALL_B3: now also J7.4
- net HALL_C1: now also J5.2; no longer J5.10
- net HALL_C2: now also J6.2; no longer J6.10
- net HALL_C3: now also J7.2
- net PHASE_U1: now also J5.10, J5.11; no longer J5.1, J5.2
- net PHASE_U2: now also J6.10, J6.11; no longer J6.1, J6.2
- net PHASE_U3: now also J7.10, J7.11
- net PHASE_V1: now also J5.8, J5.9; no longer J5.3, J5.4
- net PHASE_V2: now also J6.8, J6.9; no longer J6.3, J6.4
- net PHASE_V3: now also J7.8, J7.9
- net PHASE_W1: now also J5.7; no longer J5.5
- net PHASE_W2: now also J6.7; no longer J6.5
- net PHASE_W3: now also J7.6, J7.7
Other:
- moved on the sheet: J6
