File: designfiles/electronics/MOTORDRIVER/servocontroller.kicad_sch (KiCad schematic)
At the start: 59 parts, among them U4 TMC4671-LA

Commit message: small tweaks
Parts:
- removed C37, C38, C39: 100nF, Capacitor_SMD:C_0603_1608Metric, symbol Device:C
- added C43, C55, C58, C64: 100nF, Capacitor_SMD:C_0603_1608Metric, symbol Device:C
- added C62: 4.7µF, Capacitor_SMD:C_0603_1608Metric, symbol Device:C
- renumbered C40 to C37, C41 to C38, C42 to C39, C43 to C40, C44 to C41, C45 to C42, C46 to C44, C47 to C45, C48 to C46, C49 to C47, C50 to C48, C51 to C49, C52 to C50, C53 to C51, C54 to C52, C55 to C53, C56 to C54, C57 to C56, C58 to C57, C62 to C63
Connections:
- net +3.3V: now also U4.13 (VCCIO2), U4.2 (VCCIO1), U4.43 (VCCIO3), U4.52 (VCCIO4), U4.61 (VCCIO5), U4.72 (VCCIO6)
- net +5V: now also C62.2, C64.2
- net GND: now also C43.1, C55.1, C58.1, C62.1, C64.1
- net at U4.15 (VCCCORE1): now also C58.2
- net at U4.45 (VCCCORE2): now also C55.2
- net at U4.63 (VCCCORE3): now also C43.2

Commit message: tmc gpio pins fixed, spi db fixed, all mcu digital pins fixed, decoupled resetn
Parts:
- removed D27: LED, Diode_SMD:D_0603_1608Metric, symbol Device:LED
- removed R53: 1kΩ, Resistor_SMD:R_0603_1608Metric, symbol Device:R
Connections:
- net GPIO2 is gone; now on an unnamed net: U4.74 (GPIO2_/_ADC_VM_MCD)
- net at R52.2: no longer U4.1 (GPIO5_/_AENC_UX_MCD_/_DBGSPI_MOSI)
- net TMC_DB_MISO: now reaches U4.4 (GPIO6_/_AENC_VN_MCD_/_DBGSPI_MISO)
- net TMC_DB_CS: now reaches U4.75 (GPIO3_/_AGPI_A_MCD_/_DBGSPI_NSCS)
- net TMC_DB_SCK: now reaches U4.76 (GPIO4_/_AGPI_B_MCD_/_DBGSPI_SCK)
- net GPIO0: no longer names the net of U4.70 (GPIO0_/_ADC_I0_MCD)
- net GPIO1: no longer names the net of U4.71 (GPIO1_/_ADC_I1_MCD)
- net UART_RX: no longer names the net of U4.10 (UART_RXD)
- net UART_TX: no longer names the net of U4.11 (UART_TXD)
- new net TMC_DB_MOSI: U4.1 (GPIO5_/_AENC_UX_MCD_/_DBGSPI_MOSI)
Other:
- moved on the sheet: D26, R52

Commit message: added inductors
Parts:
- removed C61: 4.7µF, Capacitor_SMD:C_0603_1608Metric, symbol Device:C
- added C50: 100nF, Capacitor_SMD:C_0603_1608Metric, symbol Device:C
- U4: footprint kuben-footprints:QFN40P1050X650X90-77N -> QFN40P1050X650X90-77N
- renumbered C50 to C51, C51 to C52, C52 to C53, C53 to C54, C54 to C55, C55 to C56, C56 to C57, C57 to C58, C58 to C59, C59 to C60, C60 to C61, D26 to D24, D24 to D25, D25 to D26, D28 to D27, D29 to D28, D30 to D29, R45 to R46, R46 to R47, R47 to R48, R48 to R49, R49 to R50, R50 to R51, R51 to R52, R52 to R53
Connections:
- net GND: now also C50.2
- net at R54.1, U4.50 (NRST): now also C50.1
Other:
- moved on the sheet: D24, R53, R54

Commit message: minor tweaks on schematic and started on the pcb layout, made good work
Parts:
- U4: footprint QFN40P1050X650X90-77N -> kuben-footprints:QFN40P1050X650X90-77N
Changed lines of the file:
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@@
 			)
 		)
-		(property "Footprint" "QFN40P1050X650X90-77N"
+		(property "Footprint" "kuben-footprints:QFN40P1050X650X90-77N"
 			(at 221.92 54.61 0)
 			(effects

Commit message: worked on PCB
Parts:
- renumbered C58 to C13, C59 to C14, C53 to C15, C55 to C16, C61 to C17, C60 to C18, C62 to C19, C54 to C20, C57 to C21, C40 to C22, C46 to C23, C42 to C24, C47 to C25, C43 to C26, C64 to C27, C51 to C28, C48 to C29, C37 to C30, C38 to C31, C52 to C32, C50 to C33, C39 to C34, C49 to C35, C56 to C37, C63 to C50, C41 to C61, C45 to C66, C44 to C69, D28 to D11, D17 to D12, D29 to D13, D15 to D14, D16 to D15, D12 to D16, D19 to D17, D13 to D19, D23 to D21, D20 to D23, D21 to D24, D18 to D3, D14 to D4, D24 to D5, D27 to D6, D26 to D7, D25 to D8, R55 to R11, R48 to R12, R53 to R13, R47 to R14, R54 to R16, R52 to R17, R46 to R18, R57 to R25, R56 to R27, R49 to R28, R50 to R29, R51 to R35
Connections:
- net HALL_U: no longer C61.2, D7.1 (K), D8.2 (A), R35.2, U4.38 (HALL_UX)
- net HALL_V: no longer C69.2, D21.1 (K), D22.2 (A), R29.2, U4.37 (HALL_V)
- net HALL_W: no longer C66.2, D23.2 (A), D24.1 (K), R28.2, U4.36 (HALL_WY)
- new net HALL_U_FILT: C61.2, D7.1 (K), D8.2 (A), R35.2, U4.38 (HALL_UX)
- new net HALL_V_FILT: C69.2, D21.1 (K), D22.2 (A), R29.2, U4.37 (HALL_V)
- new net HALL_W_FILT: C66.2, D23.2 (A), D24.1 (K), R28.2, U4.36 (HALL_WY)

Commit message: worked on pcb
Parts:
- renumbered C30 to C37, C31 to C38, C34 to C39, C22 to C40, C61 to C41, C24 to C42, C26 to C43, C69 to C44, C66 to C45, C23 to C46, C25 to C47, C29 to C48, C35 to C49, C33 to C50, C28 to C51, C32 to C52, C15 to C53, C20 to C54, C16 to C55, C37 to C56, C21 to C57, C13 to C58, C14 to C59, C18 to C60, C17 to C61, C19 to C62, C50 to C63, C27 to C64, D16 to D12, D19 to D13, D4 to D14, D14 to D15, D15 to D16, D12 to D17, D3 to D18, D17 to D19, D23 to D20, D24 to D21, D21 to D23, D5 to D24, D8 to D25, D7 to D26, D6 to D27, D11 to D28, D13 to D29, R18 to R46, R14 to R47, R12 to R48, R28 to R49, R29 to R50, R35 to R51, R17 to R52, R13 to R53, R16 to R54, R11 to R55, R27 to R56, R25 to R57

Commit message: added design rules from pcbway, we need to redo some work to fit the design rules
Connections:
- no-connect marks 26 -> 28

Commit message: worked on pcb
Parts:
- renumbered C37 to C39, C38 to C40, C39 to C41, C40 to C42, C41 to C43, C42 to C44, C43 to C45, C44 to C46, C45 to C47, C46 to C48, C47 to C49, C48 to C50, C49 to C51, C50 to C52, C51 to C53, C52 to C54, C53 to C55, C54 to C56, C55 to C57, C56 to C58, C57 to C59, C58 to C60, C59 to C61, C60 to C62, C61 to C63, C62 to C64, C63 to C65, C64 to C66, U4 to U5
Connections:
- net +5V renamed +5VA
