File: designfiles/electronics/MOTORDRIVER/voltageregulatros.kicad_sch (KiCad schematic)
At the start: 76 parts, among them IC6 BQ24133RGYR, IC7 LM5176PWPR, Q10 40V 70A, Q11 30V 71A, Q12 30V 71A, Q13 30V 71A, Q14 30V 71A, Q8 30V 71A, Q9 30V 71A, U1 LD1117S25TR_SOT223, U2 LD1117S33TR_SOT223, U3 LD1117S50TR_SOT223

Commit message: removed backup files and found components for special resistors and diodes
Parts:
- renumbered R14 to R15, R15 to R16, R16 to R17, R17 to R18, R18 to R19, R19 to R20, R20 to R21, R21 to R22, R22 to R23, R23 to R24, R24 to R25, R25 to R26, R26 to R27, R27 to R28, R28 to R29, R29 to R30, R30 to R31, R31 to R32, R32 to R33, R33 to R34, R34 to R35, R35 to R36, R36 to R37, R37 to R38, R38 to R39, R39 to R40, R40 to R41, R41 to R42
Changed lines of the file:
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@@
 		(on_board yes)
 		(dnp no)
-		(property "Reference" "R25"
+		(property "Reference" "R26"
 			(at 88.9 114.046 0)
 			(effects
@@
 			(project "motordriver"
 				(path "/c7634e88-16d1-45ec-9aac-9c841e03cf6d/40fe2217-7020-4fd5-b361-1423767f0697"
-					(reference "R25")
+					(reference "R26")
 					(unit 1)
 				)
@@
 		(on_board yes)
 		(dnp no)
-		(property "Reference" "R21"
+		(property "Reference" "R22"
 			(at 47.244 111.76 0)
 			(effects
@@
 			(project "motordriver"
 				(path "/c7634e88-16d1-45ec-9aac-9c841e03cf6d/40fe2217-7020-4fd5-b361-1423767f0697"
-					(reference "R21")
+					(reference "R22")
 					(unit 1)
 				)
@@
 		(on_board yes)
 		(dnp no)
-		(property "Reference" "R14"
+		(property "Reference" "R15"
 			(at 18.034 72.898 0)
 			(effects
@@
 			(project "motordriver"
 				(path "/c7634e88-16d1-45ec-9aac-9c841e03cf6d/40fe2217-7020-4fd5-b361-1423767f0697"
-					(reference "R14")
+					(reference "R15")
 					(unit 1)
 				)
@@
 		(dnp no)
 		(fields_autoplaced yes)
-		(property "Reference" "R23"
+		(property "Reference" "R24"
 			(at 72.39 36.83 90)
 			(effects
@@
 			(project "motordriver"
 				(path "/c7634e88-16d1-45ec-9aac-9c841e03cf6d/40fe2217-7020-4fd5-b361-1423767f0697"
-					(reference "R23")
+					(reference "R24")
 					(unit 1)
 				)
@@
 		(on_board yes)
 		(dnp no)
-		(property "Reference" "R24"
+		(property "Reference" "R25"
 			(at 79.756 107.95 90)
 			(effects
@@
 			(project "motordriver"
 				(path "/c7634e88-16d1-45ec-9aac-9c841e03cf6d/40fe2217-7020-4fd5-b361-1423767f0697"
-					(reference "R24")
+					(reference "R25")
 					(unit 1)
 				)
@@
 		(dnp no)
 		(fields_autoplaced yes)
-		(property "Reference" "R31"
+		(property "Reference" "R32"
 			(at 162.56 137.16 90)
 			(effects
@@
 			(project "motordriver"
 				(path "/c7634e88-16d1-45ec-9aac-9c841e03cf6d/40fe2217-7020-4fd5-b361-1423767f0697"
-					(reference "R31")
+					(reference "R32")
 					(unit 1)
 				)
@@
 		(on_board yes)
 		(dnp no)
-		(property "Reference" "R19"
+		(property "Reference" "R20"
 			(at 49.784 53.086 0)
 			(effects
@@
 			(project "motordriver"
 				(path "/c7634e88-16d1-45ec-9aac-9c841e03cf6d/40fe2217-7020-4fd5-b361-1423767f0697"
-					(reference "R19")
+					(reference "R20")
 					(unit 1)
 				)
@@
 		(on_board yes)
 		(dnp no)
-		(property "Reference" "R37"
+		(property "Reference" "R38"
 			(at 172.212 36.068 0)
 			(effects
@@
 			(project "motordriver"
 				(path "/c7634e88-16d1-45ec-9aac-9c841e03cf6d/40fe2217-7020-4fd5-b361-1423767f0697"
-					(reference "R37")
+					(reference "R38")
 					(unit 1)
 				)
@@
 		(dnp no)
 		(fields_autoplaced yes)
-		(property "Reference" "R17"
+		(property "Reference" "R18"
 			(at 34.29 132.0799 0)
 			(effects
@@
 			(project "motordriver"
 				(path "/c7634e88-16d1-45ec-9aac-9c841e03cf6d/40fe2217-7020-4fd5-b361-1423767f0697"
-					(reference "R17")
+					(reference "R18")
 					(unit 1)
 				)
@@
 		(on_board yes)
 		(dnp no)
-		(property "Reference" "R30"
+		(property "Reference" "R31"
 			(at 151.638 38.354 90)
 			(effects
@@
 			(project "motordriver"
 				(path "/c7634e88-16d1-45ec-9aac-9c841e03cf6d/40fe2217-7020-4fd5-b361-1423767f0697"
-					(reference "R30")
+					(reference "R31")
 					(unit 1)
 				)
@@
 		(on_board yes)
 		(dnp no)
-		(property "Reference" "R18"
+		(property "Reference" "R19"
 			(at 38.608 94.234 90)
 			(effects
@@
 			(project ""
 				(path "/c7634e88-16d1-45ec-9aac-9c841e03cf6d/40fe2217-7020-4fd5-b361-1423767f0697"
-					(reference "R18")
+					(reference "R19")
 					(unit 1)
 				)
@@
 		(on_board yes)
 		(dnp no)
-		(property "Reference" "R20"
+		(property "Reference" "R21"
 			(at 46.736 104.394 0)
 			(effects
@@
 			(project "motordriver"
 				(path "/c7634e88-16d1-45ec-9aac-9c841e03cf6d/40fe2217-7020-4fd5-b361-1423767f0697"
-					(reference "R20")
+					(reference "R21")
 					(unit 1)
 				)
@@
 		(on_board yes)
 		(dnp no)
-		(property "Reference" "R32"
+		(property "Reference" "R33"
 			(at 163.576 23.876 90)
 			(effects
@@
 			(project "motordriver"
 				(path "/c7634e88-16d1-45ec-9aac-9c841e03cf6d/40fe2217-7020-4fd5-b361-1423767f0697"
-					(reference "R32")
+					(reference "R33")
 					(unit 1)
 				)
@@
 		(on_board yes)
 		(dnp no)
-		(property "Reference" "R33"
+		(property "Reference" "R34"
 			(at 163.576 31.75 90)
 			(effects
@@
 			(project "motordriver"
 				(path "/c7634e88-16d1-45ec-9aac-9c841e03cf6d/40fe2217-7020-4fd5-b361-1423767f0697"
-					(reference "R33")
+					(reference "R34")
 					(unit 1)
 				)
@@
 		(dnp no)
 		(fields_autoplaced yes)
-		(property "Reference" "R41"
+		(property "Reference" "R42"
 			(at 252.73 76.1999 0)
 			(effects
@@
 			(project "motordriver"
 				(path "/c7634e88-16d1-45ec-9aac-9c841e03cf6d/40fe2217-7020-4fd5-b361-1423767f0697"
-					(reference "R41")
+					(reference "R42")
 					(unit 1)
 				)
@@
 		(on_board yes)
 		(dnp no)
-		(property "Reference" "R40"
+		(property "Reference" "R41"
 			(at 213.106 84.836 0)
 			(effects
@@
 			(project "motordriver"
 				(path "/c7634e88-16d1-45ec-9aac-9c841e03cf6d/40fe2217-7020-4fd5-b361-1423767f0697"
-					(reference "R40")
+					(reference "R41")
 					(unit 1)
 				)
@@
 		(on_board yes)
 		(dnp no)
-		(property "Reference" "R22"
+		(property "Reference" "R23"
 			(at 62.484 50.038 0)
 			(effects
@@
 			(project "motordriver"
 				(path "/c7634e88-16d1-45ec-9aac-9c841e03cf6d/40fe2217-7020-4fd5-b361-1423767f0697"
-					(reference "R22")
+					(reference "R23")
 					(unit 1)
 				)
@@
 		(dnp no)
 		(fields_autoplaced yes)
-		(property "Reference" "R16"
+		(property "Reference" "R17"
 			(at 34.29 121.9199 0)
 			(effects
@@
 			(project "motordriver"
 				(path "/c7634e88-16d1-45ec-9aac-9c841e03cf6d/40fe2217-7020-4fd5-b361-1423767f0697"
-					(reference "R16")
+					(reference "R17")
 					(unit 1)
 				)
@@
 		(dnp no)
 		(fields_autoplaced yes)
-		(property "Reference" "R28"
+		(property "Reference" "R29"
 			(at 113.03 46.99 90)
 			(effects
@@
 			(project "motordriver"
 				(path "/c7634e88-16d1-45ec-9aac-9c841e03cf6d/40fe2217-7020-4fd5-b361-1423767f0697"
-					(reference "R28")
+					(reference "R29")
 					(unit 1)
 				)
@@
 		(on_board yes)
 		(dnp no)
-		(property "Reference" "R35"
+		(property "Reference" "R36"
 			(at 169.672 55.626 90)
 			(effects
@@
 			(project "motordriver"
 				(path "/c7634e88-16d1-45ec-9aac-9c841e03cf6d/40fe2217-7020-4fd5-b361-1423767f0697"
-					(reference "R35")
+					(reference "R36")
 					(unit 1)
 				)
@@
 		(on_board yes)
 		(dnp no)
-		(property "Reference" "R15"
+		(property "Reference" "R16"
 			(at 23.876 45.466 0)
 			(effects
@@
 			(project "motordriver"
 				(path "/c7634e88-16d1-45ec-9aac-9c841e03cf6d/40fe2217-7020-4fd5-b361-1423767f0697"
-					(reference "R15")
+					(reference "R16")
 					(unit 1)
 				)
@@
 		(on_board yes)
 		(dnp no)
-		(property "Reference" "R39"
+		(property "Reference" "R40"
 			(at 184.912 102.362 0)
 			(effects
@@
 			(project "motordriver"
 				(path "/c7634e88-16d1-45ec-9aac-9c841e03cf6d/40fe2217-7020-4fd5-b361-1423767f0697"
-					(reference "R39")
+					(reference "R40")
 					(unit 1)
 				)
@@
 		(dnp no)
 		(fields_autoplaced yes)
-		(property "Reference" "R29"
+		(property "Reference" "R30"
 			(at 129.54 57.15 90)
 			(effects
@@
 			(project "motordriver"
 				(path "/c7634e88-16d1-45ec-9aac-9c841e03cf6d/40fe2217-7020-4fd5-b361-1423767f0697"
-					(reference "R29")
+					(reference "R30")
 					(unit 1)
 				)
@@
 		(on_board yes)
 		(dnp no)
-		(property "Reference" "R36"
+		(property "Reference" "R37"
 			(at 170.434 113.03 0)
 			(effects
@@
 			(project "motordriver"
 				(path "/c7634e88-16d1-45ec-9aac-9c841e03cf6d/40fe2217-7020-4fd5-b361-1423767f0697"
-					(reference "R36")
+					(reference "R37")
 					(unit 1)
 				)
@@
 		(on_board yes)
 		(dnp no)
-		(property "Reference" "R27"
+		(property "Reference" "R28"
 			(at 113.03 116.8399 0)
 			(effects
@@
 			(project "motordriver"
 				(path "/c7634e88-16d1-45ec-9aac-9c841e03cf6d/40fe2217-7020-4fd5-b361-1423767f0697"
-					(reference "R27")
+					(reference "R28")
 					(unit 1)
 				)
@@
 		(on_board yes)
 		(dnp no)
-		(property "Reference" "R34"
+		(property "Reference" "R35"
 			(at 169.926 44.45 90)
 			(effects
@@
 			(project "motordriver"
 				(path "/c7634e88-16d1-45ec-9aac-9c841e03cf6d/40fe2217-7020-4fd5-b361-1423767f0697"
-					(reference "R34")
+					(reference "R35")
 					(unit 1)
 				)
@@
 		(dnp no)
 		(fields_autoplaced yes)
-		(property "Reference" "R26"
+		(property "Reference" "R27"
 			(at 113.03 106.6799 0)
 			(effects
@@
 			(project "motordriver"
 				(path "/c7634e88-16d1-45ec-9aac-9c841e03cf6d/40fe2217-7020-4fd5-b361-1423767f0697"
-					(reference "R26")
+					(reference "R27")
 					(unit 1)
 				)
@@
 		(on_board yes)
 		(dnp no)
-		(property "Reference" "R38"
+		(property "Reference" "R39"
 			(at 175.006 105.41 90)
 			(effects
@@
 			(project "motordriver"
 				(path "/c7634e88-16d1-45ec-9aac-9c841e03cf6d/40fe2217-7020-4fd5-b361-1423767f0697"
-					(reference "R38")
+					(reference "R39")
 					(unit 1)
 				)

Commit message: added diodes
Parts:
- D10: value 385mVf 500mA -> 4.7Vf 0.5A; footprint Diode_SMD:D_0603_1608Metric -> kuben-footprints:DIOC1709X85N; Height (none) -> 0.85; Manufacturer_Name (none) -> Comchip Technology; Manufacturer_Part_Number (none) -> CDBU0520; Mouser Part Number (none) -> 750-CDBU0520; Mouser Price/Stock (none) -> https://www.mouser.co.uk/ProductDetail/Comchip-Technology/C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
- D11, D5, D6, D8: value 470mVf 500mA -> 4.7Vf 0.5A; footprint Diode_SMD:D_0603_1608Metric -> kuben-footprints:DIOC1709X85N; Height (none) -> 0.85; Manufacturer_Name (none) -> Comchip Technology; Manufacturer_Part_Number (none) -> CDBU0520; Mouser Part Number (none) -> 750-CDBU0520; Mouser Price/Stock (none) -> https://www.mouser.co.uk/ProductDetail/Comchip-Technology/C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

Commit message: added inductors
Parts:
- C36: footprint kuben-footprints:CAPAE1050X1050N -> CAPAE1050X1050N
- IC6: footprint kuben-footprints:BQ24133RGYR -> BQ24133RGYR
- IC7: footprint kuben-footprints:SOP65P640X120-29N -> SOP65P640X120-29N
- L1: footprint Inductor_SMD:L_10.4x10.4_H4.8 -> kuben-footprints:INDPM6965X300N; Height (none) -> 3; Manufacturer_Name (none) -> Vishay; Manufacturer_Part_Number (none) -> IHLP2525CZER3R3M01; Mouser Part Number (none) -> 70-IHLP2525CZER3R3M0; Mouser Price/Stock (none) -> https://www.mouser.co.uk/ProductDetail/Vishay-Dale/IHLP2525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
- L2: value 1µH 420µΩ -> 1µH 22A; footprint Inductor_SMD:L_12x12mm_H8mm -> kuben-footprints:INDPM6965X300N; Height (none) -> 3; Manufacturer_Name (none) -> Vishay; Manufacturer_Part_Number (none) -> IHLP2525CZER1R0M06; Mouser Part Number (none) -> 70-IHLP2525CZR1R0M06; Mouser Price/Stock (none) -> https://www.mouser.co.uk/ProductDetail/Vishay-Dale/IHLP2525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
- Q10: footprint kuben-footprints:IPD70P04P4L08ATMA2 -> IPD70P04P4L08ATMA2
- Q11, Q12, Q13, Q14, Q8, Q9: footprint kuben-footprints:IPD047N03LF2SATMA1 -> IPD047N03LF2SATMA1
Changed lines of the file:
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@@
 	)
 	(symbol
-		(lib_id "Device:L")
-		(at 250.19 50.8 90)
-		(unit 1)
-		(exclude_from_sim no)
-		(in_bom yes)
-		(on_board yes)
-		(dnp no)
-		(fields_autoplaced yes)
-		(property "Reference" "L2"
-			(at 250.19 45.72 90)
-			(effects
-				(font
-					(size 1.27 1.27)
-				)
-			)
-		)
-		(property "Value" "1µH 420µΩ"
-			(at 250.19 48.26 90)
-			(effects
-				(font
-					(size 1.27 1.27)
-				)
-			)
-		)
-		(property "Footprint" "Inductor_SMD:L_12x12mm_H8mm"
-			(at 250.19 50.8 0)
-			(effects
-				(font
-					(size 1.27 1.27)
-				)
-				(hide yes)
-			)
-		)
-		(property "Datasheet" "~"
-			(at 250.19 50.8 0)
-			(effects
-				(font
-					(size 1.27 1.27)
-				)
-				(hide yes)
-			)
-		)
-		(property "Description" "Inductor"
-			(at 250.19 50.8 0)
-			(effects
-				(font
-					(size 1.27 1.27)
-				)
-				(hide yes)
-			)
-		)
-		(pin "2"
-		)
-		(pin "1"
-		)
-		(instances
-			(project "motordriver"
-				(path "/c7634e88-16d1-45ec-9aac-9c841e03cf6d/40fe2217-7020-4fd5-b361-1423767f0697"
-					(reference "L2")
-					(unit 1)
-				)
-			)
-		)
-	)
-	(symbol
 		(lib_id "Device:R")
 		(at 52.07 111.76 180)
@@
 			)
 		)
-		(property "Footprint" "kuben-footprints:IPD047N03LF2SATMA1"
+		(property "Footprint" "IPD047N03LF2SATMA1"
 			(at 57.15 39.37 0)
 			(effects
@@
 			)
 		)
-		(property "Footprint" "kuben-footprints:IPD047N03LF2SATMA1"
+		(property "Footprint" "IPD047N03LF2SATMA1"
 			(at 245.11 44.45 0)
 			(effects
@@
 			)
 		)
-		(property "Footprint" "kuben-footprints:CAPAE1050X1050N"
+		(property "Footprint" "CAPAE1050X1050N"
 			(at 174.32 29.21 0)
 			(effects
@@
 	)
 	(symbol
+		(lib_id "Device:L")
+		(at 250.19 50.8 90)
+		(unit 1)
+		(exclude_from_sim no)
+		(in_bom yes)
+		(on_board yes)
+		(dnp no)
+		(fields_autoplaced yes)
+		(property "Reference" "L2"
+			(at 250.19 45.72 90)
+			(effects
+				(font
+					(size 1.27 1.27)
+				)
+			)
+		)
+		(property "Value" "1µH 22A"
+			(at 250.19 48.26 90)
+			(effects
+				(font
+					(size 1.27 1.27)
+				)
+			)
+		)
+		(property "Footprint" "kuben-footprints:INDPM6965X300N"
+			(at 250.19 50.8 0)
+			(effects
+				(font
+					(size 1.27 1.27)
+				)
+				(hide yes)
+			)
+		)
+		(property "Datasheet" "~"
+			(at 250.19 50.8 0)
+			(effects
+				(font
+					(size 1.27 1.27)
+				)
+				(hide yes)
+			)
+		)
+		(property "Description" "Inductor"
+			(at 250.19 50.8 0)
+			(effects
+				(font
+					(size 1.27 1.27)
+				)
+				(hide yes)
+			)
+		)
+		(property "Height" "3"
+			(at 646.38 34.29 0)
+			(effects
+				(font
+					(size 1.27 1.27)
+				)
+				(justify left top)
+				(hide yes)
+			)
+		)
+		(property "Mouser Part Number" "70-IHLP2525CZR1R0M06"
+			(at 746.38 34.29 0)
+			(effects
+				(font
+					(size 1.27 1.27)
+				)
+				(justify left top)
+				(hide yes)
+			)
+		)
+		(property "Mouser Price/Stock" "https://www.mouser.co.uk/ProductDetail/Vishay-Dale/IHLP2525CZER1R0M06?qs=gMuw6kkpPFiOvUjVH4k3sQ%3D%3D"
+			(at 846.38 34.29 0)
+			(effects
+				(font
+					(size 1.27 1.27)
+				)
+				(justify left top)
+				(hide yes)
+			)
+		)
+		(property "Manufacturer_Name" "Vishay"
+			(at 946.38 34.29 0)
+			(effects
+				(font
+					(size 1.27 1.27)
+				)
+				(justify left top)
+				(hide yes)
+			)
+		)
+		(property "Manufacturer_Part_Number" "IHLP2525CZER1R0M06"
+			(at 1046.38 34.29 0)
+			(effects
+				(font
+					(size 1.27 1.27)
+				)
+				(justify left top)
+				(hide yes)
+			)
+		)
+		(pin "2"
+		)
+		(pin "1"
+		)
+		(instances
+			(project ""
+				(path "/c7634e88-16d1-45ec-9aac-9c841e03cf6d/40fe2217-7020-4fd5-b361-1423767f0697"
+					(reference "L2")
+					(unit 1)
+				)
+			)
+		)
+	)
+	(symbol
 		(lib_id "power:GND")
 		(at 77.47 120.65 0)
@@
 			)
 		)
-		(property "Footprint" "kuben-footprints:BQ24133RGYR"
+		(property "Footprint" "BQ24133RGYR"
 			(at 0.33 102.87 0)
 			(effects
@@
 			)
 		)
-		(property "Footprint" "kuben-footprints:IPD047N03LF2SATMA1"
+		(property "Footprint" "IPD047N03LF2SATMA1"
 			(at 255.27 62.23 0)
 			(effects
@@
 			)
 		)
-		(property "Footprint" "kuben-footprints:IPD047N03LF2SATMA1"
+		(property "Footprint" "IPD047N03LF2SATMA1"
 			(at 255.27 44.45 0)
 			(effects
@@
 			)
 		)
-		(property "Footprint" "kuben-footprints:SOP65P640X120-29N"
+		(property "Footprint" "SOP65P640X120-29N"
 			(at 209.55 135.56 0)
 			(effects
@@
 	)
 	(symbol
+		(lib_id "Device:L")
+		(at 114.3 63.5 90)
+		(unit 1)
+		(exclude_from_sim no)
+		(in_bom yes)
+		(on_board yes)
+		(dnp no)
+		(fields_autoplaced yes)
+		(property "Reference" "L1"
+			(at 114.3 58.42 90)
+			(effects
+				(font
+					(size 1.27 1.27)
+				)
+			)
+		)
+		(property "Value" "3.3µH"
+			(at 114.3 60.96 90)
+			(effects
+				(font
+					(size 1.27 1.27)
+				)
+			)
+		)
+		(property "Footprint" "kuben-footprints:INDPM6965X300N"
+			(at 114.3 63.5 0)
+			(effects
+				(font
+					(size 1.27 1.27)
+				)
+				(hide yes)
+			)
+		)
+		(property "Datasheet" "~"
+			(at 114.3 63.5 0)
+			(effects
+				(font
+					(size 1.27 1.27)
+				)
+				(hide yes)
+			)
+		)
+		(property "Description" "Inductor"
+			(at 114.3 63.5 0)
+			(effects
+				(font
+					(size 1.27 1.27)
+				)
+				(hide yes)
+			)
+		)
+		(property "Height" "3"
+			(at 510.49 46.99 0)
+			(effects
+				(font
+					(size 1.27 1.27)
+				)
+				(justify left top)
+				(hide yes)
+			)
+		)
+		(property "Mouser Part Number" "70-IHLP2525CZER3R3M0"
+			(at 610.49 46.99 0)
+			(effects
+				(font
+					(size 1.27 1.27)
+				)
+				(justify left top)
+				(hide yes)
+			)
+		)
+		(property "Mouser Price/Stock" "https://www.mouser.co.uk/ProductDetail/Vishay-Dale/IHLP2525CZER3R3M01?qs=PA%252BPfIdQ8xlEO%252B8WW0W2Xw%3D%3D"
+			(at 710.49 46.99 0)
+			(effects
+				(font
+					(size 1.27 1.27)
+				)
+				(justify left top)
+				(hide yes)
+			)
+		)
+		(property "Manufacturer_Name" "Vishay"
+			(at 810.49 46.99 0)
+			(effects
+				(font
+					(size 1.27 1.27)
+				)
+				(justify left top)
+				(hide yes)
+			)
+		)
+		(property "Manufacturer_Part_Number" "IHLP2525CZER3R3M01"
+			(at 910.49 46.99 0)
+			(effects
+				(font
+					(size 1.27 1.27)
+				)
+				(justify left top)
+				(hide yes)
+			)
+		)
+		(pin "2"
+		)
+		(pin "1"
+		)
+		(instances
+			(project ""
+				(path "/c7634e88-16d1-45ec-9aac-9c841e03cf6d/40fe2217-7020-4fd5-b361-1423767f0697"
+					(reference "L1")
+					(unit 1)
+				)
+			)
+		)
+	)
+	(symbol
 		(lib_id "Device:C")
 		(at 27.94 167.64 0)
@@
 			)
 		)
-		(property "Footprint" "kuben-footprints:IPD047N03LF2SATMA1"
+		(property "Footprint" "IPD047N03LF2SATMA1"
 			(at 245.11 62.23 0)
 			(effects
@@
 			)
 		)
-		(property "Footprint" "kuben-footprints:IPD70P04P4L08ATMA2"
+		(property "Footprint" "IPD70P04P4L08ATMA2"
 			(at 138.43 46.99 0)
 			(effects
@@
 		(dnp no)
 		(property "Reference" "D5"
-			(at 12.7 67.6276 0)
+			(at 14.224 64.262 0)
 			(effects
 				(font
@@
 	)
 	(symbol
-		(lib_id "Device:L")
-		(at 114.3 63.5 90)
-		(unit 1)
-		(exclude_from_sim no)
-		(in_bom yes)
-		(on_board yes)
-		(dnp no)
-		(fields_autoplaced yes)
-		(property "Reference" "L1"
-			(at 114.3 58.42 90)
-			(effects
-				(font
-					(size 1.27 1.27)
-				)
-			)
-		)
-		(property "Value" "3.3µH"
-			(at 114.3 60.96 90)
-			(effects
-				(font
-					(size 1.27 1.27)
-				)
-			)
-		)
-		(property "Footprint" "Inductor_SMD:L_10.4x10.4_H4.8"
-			(at 114.3 63.5 0)
-			(effects
-				(font
-					(size 1.27 1.27)
-				)
-				(hide yes)
-			)
-		)
-		(property "Datasheet" "~"
-			(at 114.3 63.5 0)
-			(effects
-				(font
-					(size 1.27 1.27)
-				)
-				(hide yes)
-			)
-		)
-		(property "Description" "Inductor"
-			(at 114.3 63.5 0)
-			(effects
-				(font
-					(size 1.27 1.27)
-				)
-				(hide yes)
-			)
-		)
-		(pin "2"
-		)
-		(pin "1"
-		)
-		(instances
-			(project ""
-				(path "/c7634e88-16d1-45ec-9aac-9c841e03cf6d/40fe2217-7020-4fd5-b361-1423767f0697"
-					(reference "L1")
-					(unit 1)
-				)
-			)
-		)
-	)
-	(symbol
 		(lib_id "Device:R")
 		(at 187.96 104.14 180)
@@
 			)
 		)
-		(property "Footprint" "kuben-footprints:IPD047N03LF2SATMA1"
+		(property "Footprint" "IPD047N03LF2SATMA1"
 			(at 139.37 39.37 0)
 			(effects

Commit message: minor tweaks on schematic and started on the pcb layout, made good work
Parts:
- C36: footprint CAPAE1050X1050N -> kuben-footprints:CAPAE1050X1050N
- IC6: footprint BQ24133RGYR -> kuben-footprints:BQ24133RGYR
- IC7: footprint SOP65P640X120-29N -> kuben-footprints:SOP65P640X120-29N
- Q10: footprint IPD70P04P4L08ATMA2 -> kuben-footprints:IPD70P04P4L08ATMA2
- Q11, Q12, Q13, Q14, Q8, Q9: footprint IPD047N03LF2SATMA1 -> kuben-footprints:IPD047N03LF2SATMA1
Changed lines of the file:
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@@
 			)
 		)
-		(property "Footprint" "IPD047N03LF2SATMA1"
+		(property "Footprint" "kuben-footprints:IPD047N03LF2SATMA1"
 			(at 57.15 39.37 0)
 			(effects
@@
 			)
 		)
-		(property "Footprint" "IPD047N03LF2SATMA1"
+		(property "Footprint" "kuben-footprints:IPD047N03LF2SATMA1"
 			(at 245.11 44.45 0)
 			(effects
@@
 			)
 		)
-		(property "Footprint" "CAPAE1050X1050N"
+		(property "Footprint" "kuben-footprints:CAPAE1050X1050N"
 			(at 174.32 29.21 0)
 			(effects
@@
 			)
 		)
-		(property "Footprint" "BQ24133RGYR"
+		(property "Footprint" "kuben-footprints:BQ24133RGYR"
 			(at 0.33 102.87 0)
 			(effects
@@
 			)
 		)
-		(property "Footprint" "IPD047N03LF2SATMA1"
+		(property "Footprint" "kuben-footprints:IPD047N03LF2SATMA1"
 			(at 255.27 62.23 0)
 			(effects
@@
 			)
 		)
-		(property "Footprint" "IPD047N03LF2SATMA1"
+		(property "Footprint" "kuben-footprints:IPD047N03LF2SATMA1"
 			(at 255.27 44.45 0)
 			(effects
@@
 			)
 		)
-		(property "Footprint" "SOP65P640X120-29N"
+		(property "Footprint" "kuben-footprints:SOP65P640X120-29N"
 			(at 209.55 135.56 0)
 			(effects
@@
 			)
 		)
-		(property "Footprint" "IPD047N03LF2SATMA1"
+		(property "Footprint" "kuben-footprints:IPD047N03LF2SATMA1"
 			(at 245.11 62.23 0)
 			(effects
@@
 			)
 		)
-		(property "Footprint" "IPD70P04P4L08ATMA2"
+		(property "Footprint" "kuben-footprints:IPD70P04P4L08ATMA2"
 			(at 138.43 46.99 0)
 			(effects
@@
 			)
 		)
-		(property "Footprint" "IPD047N03LF2SATMA1"
+		(property "Footprint" "kuben-footprints:IPD047N03LF2SATMA1"
 			(at 139.37 39.37 0)
 			(effects

Commit message: worked on PCB
Parts:
- renumbered C20 to C1, C16 to C10, C26 to C11, C27 to C12, C36 to C140, C28 to C2, C10 to C3, C12 to C36, C18 to C38, C14 to C39, C24 to C4, C15 to C40, C17 to C41, C19 to C42, C11 to C43, C23 to C5, C29 to C56, C32 to C59, C22 to C6, C33 to C63, C31 to C65, C30 to C67, C13 to C7, C35 to C72, C34 to C73, C21 to C8, C25 to C9, D9 to D1, D7 to D10, D5 to D2, D8 to D25, D11 to D26, D10 to D28, D6 to D9, IC6 to IC1, IC7 to IC2, Q10 to Q1, Q11 to Q2, Q12 to Q3, Q14 to Q4, Q13 to Q5, Q9 to Q6, Q8 to Q7, R32 to R1, R30 to R10, R26 to R19, R18 to R2, R16 to R22, R22 to R23, R28 to R3, R33 to R31, R31 to R32, R40 to R33, R36 to R37, R39 to R38, R35 to R39, R25 to R4, R42 to R40, R37 to R42, R38 to R43, R24 to R46, R23 to R47, R19 to R6, R29 to R7, R17 to R8, R27 to R9, U2 to U1, U1 to U2

Commit message: worked on pcb
Parts:
- renumbered C3 to C10, C43 to C11, C36 to C12, C7 to C13, C39 to C14, C40 to C15, C10 to C16, C41 to C17, C38 to C18, C42 to C19, C1 to C20, C8 to C21, C6 to C22, C5 to C23, C4 to C24, C9 to C25, C11 to C26, C12 to C27, C2 to C28, C56 to C29, C67 to C30, C65 to C31, C59 to C32, C63 to C33, C73 to C34, C72 to C35, C140 to C36, D28 to D10, D26 to D11, D2 to D5, D9 to D6, D10 to D7, D25 to D8, D1 to D9, IC1 to IC6, IC2 to IC7, Q1 to Q10, Q2 to Q11, Q3 to Q12, Q5 to Q13, Q4 to Q14, Q7 to Q8, Q6 to Q9, R22 to R16, R8 to R17, R2 to R18, R6 to R19, R23 to R22, R47 to R23, R46 to R24, R4 to R25, R19 to R26, R9 to R27, R3 to R28, R7 to R29, R10 to R30, R32 to R31, R1 to R32, R31 to R33, R39 to R35, R37 to R36, R42 to R37, R43 to R38, R38 to R39, R33 to R40, R40 to R42, U2 to U1, U1 to U2
Connections:
- no-connect marks 0 -> 1

Commit message: added design rules from pcbway, we need to redo some work to fit the design rules
Parts:
- removed R42: 2mΩ, Resistor_SMD:R_0603_1608Metric, symbol Device:R_Shunt
- added R42: 2mΩ, Resistor_SMD:R_0603_1608Metric, symbol Device:R
Connections:
- net +12V: now also C10.1, C16.1, C22.1, U1.3 (VI), U2.3 (VI), U3.3 (VI)
- net GND: now also IC7.15 (CSG), R42.1
- net at Q12.3 (S), Q14.3 (S): now also IC7.16 (CS), R42.2

Commit message: worked on pcb
Parts:
- added C28: 100nF, Capacitor_SMD:C_0603_1608Metric, symbol Device:C
- added C31: 10uF, Capacitor_SMD:C_0603_1608Metric, symbol Device:C
- added U4: LD1117S50TR_SOT223, Package_TO_SOT_SMD:SOT-223-3_TabPin2, symbol Regulator_Linear:LD1117S50TR_SOT223
- renumbered C28 to C29, C29 to C30, C30 to C32, C31 to C33, C32 to C34, C33 to C35, C34 to C36, C35 to C37, C36 to C38
Connections:
- net +12V: now also C28.1, U4.3 (VI)
- net GND: now also C28.2, C31.2, U4.1 (GND)
- new net +5VA: C31.1, U4.2 (VO)
