File: hardware/electronics/MOTORDRIVER/IO.kicad_sch (KiCad schematic)
At the start: 22 parts, among them J1 IMU1, J2 IMU2, J3 Conn_01x04_Socket, J4 XT60-M, P1 USB_C_Plug_USB2.0, SW1 PUSH

Commit message: worked on pcb
Parts:
- R45: value 10K -> 10kΩ
Changed lines of the file:
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@@
 			)
 		)
-		(property "Value" "10K"
+		(property "Value" "10kΩ"
 			(at 191.77 43.1799 0)
 			(effects
