File: hardware/electronics/MOTORDRIVER/motordriver.kicad_pcb (KiCad board)
At the start: 4 copper layers, 122 x 122 mm, 433 parts, among them IC1 LM5109BSDX_NOPB, IC10 LM5109BSDX_NOPB, IC11 LM5109BSDX_NOPB, IC12 LM5109BSDX_NOPB, IC13 INA2181A2IDGSR, IC14 LM5109BSDX_NOPB, IC15 LM5109BSDX_NOPB, IC16 LM5109BSDX_NOPB, IC17 LM5109BSDX_NOPB, IC18 INA2181A2IDGSR, IC2 LM5109BSDX_NOPB, IC3 LM5109BSDX_NOPB, IC4 LM5109BSDX_NOPB, IC5 INA2181A2IDGSR, IC6 BQ24133RGYR, IC7 LM5176PWPR, IC8 ATSAME53J18A-MF, IC9 LM5109BSDX_NOPB, J1 IMU1, J2 IMU2, J3 Conn_01x04_Socket, J4 XT60-M, J5 1-84952-1, J6 1-84952-1, J7 1-84952-1, P1 USB_C_Plug_USB2.0, Q1 30V 71A, Q10 40V 70A, Q11 30V 71A, Q12 30V 71A, Q13 30V 71A, Q14 30V 71A, Q15 30V 71A, Q16 30V 71A, Q17 30V 71A, Q18 30V 71A, Q19 30V 71A, Q2 30V 71A, Q20 30V 71A, Q21 30V 71A, Q22 30V 71A, Q23 30V 71A, Q24 30V 71A, Q25 30V 71A, Q26 30V 71A, Q27 30V 71A, Q28 30V 71A, Q3 30V 71A, Q4 30V 71A, Q5 30V 71A, Q6 30V 71A, Q7 30V 71A, Q8 30V 71A, Q9 30V 71A, SW1 PUSH, U1 LD1117S25TR_SOT223, U2 LD1117S33TR_SOT223, U3 LD1117S50TR_SOT223, U4 LD1117S50TR_SOT223, U5 TMC4671-LA, U6 ATSAMD11D14A-M, U7 TMC4671-LA, U8 TMC4671-LA, Y1 DSC6001CI2B-025.0000T

Commit message: worked on pcb
Parts:
- moved IC5 7.16 mm to (176.5, 60.4)
- moved C9 5.94 mm to (119.6, 69.7), turned to -90 degrees
- moved C157 5.62 mm to (174.3, 57.8), turned to 180 degrees
- moved IC13 4.00 mm to (121.8, 73.0), turned to 180 degrees
Routing:
- net +5VA: track 339.2 -> 513.2 mm, vias 6 -> 20
- net +2.5V: track 325.6 -> 476.5 mm, vias 6 -> 10
- net Net-(IC18-IN+1): track 12.9 -> 115.7 mm, vias 0 -> 2
- net /drivergates2/PHASE_V: track 12.7 -> 54.6 mm, vias 0 -> 2
- net SERVO_ENI: track 141.7 -> 180.0 mm, vias 4 -> 6
- net Net-(IC18-IN+2): track 16.0 -> 48.9 mm, vias 1 -> 2
- net Net-(IC13-IN+2): track 12.8 -> 43.7 mm, vias 0 -> 2
- net /drivergates1/PHASE_V: track 23.0 -> 41.9 mm, vias 0 -> 2
- net Net-(IC5-IN+2): track 8.76 -> 25.8 mm, vias 0 -> 2
- net Net-(IC5-IN+1): track 7.15 -> 24.0 mm, vias 0 -> 2
- net /drivergates2/PHASE_U: track 19.5 -> 33.9 mm
- net Net-(IC13-IN+1): track 12.5 -> 26.4 mm
- net /drivergates1/PHASE_U: track 29.0 -> 40.6 mm, vias 0 -> 2
- net /servo2/ADC_I1_POS: track 18.4 -> 28.4 mm, vias 0 -> 1
- net /servo1/ADC_I0_POS: track 18.6 -> 27.1 mm, vias 0 -> 1
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
Commit message: - worked on pcb
Routing:
- net +12V: track 47.4 -> 86.2 mm, vias 25 -> 29
- net /servo1/ADC_I0_POS: track 27.1 -> 60.7 mm, vias 1 -> 3
- net /servo1/ADC_I1_POS: track 23.7 -> 54.2 mm, vias 1 -> 5
- net +5VA: track 513.2 -> 516.3 mm
