File: hardware/electronics/main-pcb/servocontroller.kicad_sch (KiCad schematic)
At the start: 59 parts, among them U5 TMC4671-LA

Commit message: added new brake chopper logic, the previous was sketchy, still we might need to find better brake resistors than the one I added
Parts:
- renumbered C39 to C38, C40 to C39, C41 to C40, C42 to C41, C43 to C42, C44 to C43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
