File: hardware/electronics/main-pcb/servocontroller.kicad_sch (KiCad schematic)
At the start: 59 parts, among them U5 TMC4671-LA

Commit message: saved here
Parts:
- renumbered C38 to C39, C39 to C40, C40 to C41, C41 to C42, C42 to C43, C43 to C44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
