File: hardware/electronics/main-pcb/brake.kicad_sch (KiCad schematic)
At the start: 6 parts, among them IC12 LM5109BSDX_NOPB, Q20 30V 71A

Commit message: saved here
Parts:
- removed R88: 10Ω 20W, PWR263S2010R0F, symbol PWR263S-20-10R0F:PWR263S-20-10R0F
- added R88: 20Ω 50W, symbol Device:R
Connections:
- net +12V: now also R88.1
- net GND: now also D57.2 (A), Q20.2 (D), R88.2
Other:
- moved on the sheet: D57
