File: hardware/electronics/main-pcb/voltageregulatros.kicad_sch (KiCad schematic)
At the start: 79 parts, among them IC6 BQ24133RGYR, IC7 LM5176PWPR, Q10 40V 70A, Q11 30V 71A, Q12 30V 71A, Q13 30V 71A, Q14 30V 71A, Q8 30V 71A, Q9 30V 71A, U1 LD1117S25TR_SOT223, U2 LD1117S33TR_SOT223, U3 LD1117S50TR_SOT223, U4 LD1117S50TR_SOT223

Commit message: added new brake chopper logic, the previous was sketchy, still we might need to find better brake resistors than the one I added
Parts:
- renumbered C11 to C10, C12 to C11, C13 to C12, C14 to C13, C15 to C14, C16 to C15, C17 to C16, C18 to C17, C19 to C18, C20 to C19, C21 to C20, C22 to C21, C23 to C22, C24 to C23, C25 to C24, C26 to C25, C27 to C26, C28 to C27, C29 to C28, C30 to C29, C31 to C30, C32 to C31, C33 to C32, C34 to C33, C35 to C34, C36 to C35, C37 to C36, C38 to C37, C10 to C9, D11 to D10, D5 to D4, D6 to D5, D7 to D6, D8 to D7, D9 to D8, D10 to D9, IC6 to IC5, IC7 to IC6, Q11 to Q10, Q12 to Q11, Q13 to Q12, Q14 to Q13, Q8 to Q7, Q9 to Q8, Q10 to Q9, R15 to R12, R16 to R13, R17 to R14, R18 to R15, R19 to R16, R20 to R17, R21 to R18, R22 to R19, R23 to R20, R24 to R21, R25 to R22, R26 to R23, R27 to R24, R28 to R25, R29 to R26, R30 to R27, R31 to R28, R32 to R29, R33 to R30, R34 to R31, R35 to R32, R36 to R33, R37 to R34, R38 to R35, R39 to R36, R40 to R37, R41 to R38, R42 to R39

Commit message: saved here
Parts:
- renumbered C9 to C10, C10 to C11, C11 to C12, C12 to C13, C13 to C14, C14 to C15, C15 to C16, C16 to C17, C17 to C18, C18 to C19, C19 to C20, C20 to C21, C21 to C22, C22 to C23, C23 to C24, C24 to C25, C25 to C26, C26 to C27, C27 to C28, C28 to C29, C29 to C30, C30 to C31, C31 to C32, C32 to C33, C33 to C34, C34 to C36, C36 to C37, C37 to C38, R35 to R33, R36 to R35, R38 to R36, R33 to R38
Connections:
- net IC5_VREF: now also R22.1; no longer R22.2
- net SW2: now also C37.1; no longer C37.2
- net at IC5.13 (ISET), R23.1: now also R22.2; no longer R22.1
- net BOOT2: now reaches D9.1 (K), IC6.20 (BOOT2)
- net BOOT2: now also C37.2; no longer C37.1
- net VCC: now reaches D10.2 (A), D9.2 (A), IC6.23 (VCC), R36.1
- net COMP: now reaches C33.2, IC6.9 (COMP), R37.2
- net BOOT1: now reaches C35.1, D10.1 (K), IC6.26 (BOOT1)
- net OVPSET: now reaches IC5.18 (OVPSET), R14.1, R15.2
- net PGOOD: now reaches IC6.17 (PGOOD), R36.2
- net RT: now reaches IC6.6 (RT), R38.2
- net SLOPE: now reaches C36.2, IC6.7 (SLOPE)
- net SS: now reaches C34.2, IC6.8 (SS)
Other:
- note removed: "Decoupling caps"
- moved on the sheet: C15, C18, C32, C33, C34, C35, C36, C37, D10, D9, R14, R15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

Commit message: wip
Parts:
- renumbered R18 to R17, R19 to R18, R17 to R19
