File: hardware/electronics/core-pcb/IO.kicad_sch (KiCad schematic)
At the start: 23 parts, among them J1 IMU1, J2 IMU2, J3 Conn_01x04_Socket, J4 XT60-M, P1 USB_C_Plug_USB2.0, SW1 PUSH

Commit message: started work on pcbv2 work in progress
Parts:
- renumbered R40 to R29, R41 to R30, R42 to R31
Connections:
- net BATTVIN renamed BATTERY_P
