File: hardware/electronics/core-pcb/brake.kicad_sch (KiCad schematic)
At the start: 6 parts, among them IC12 LM5109BSDX_NOPB, Q20 30V 71A

Commit message: started work on pcbv2 work in progress
Parts:
- removed Q20: 30V 71A, kuben-footprints:IPD047N03LF2SATMA1, symbol IPD047N03LF2SATMA1:IPD047N03LF2SATMA1
- added Q16: NMOS 30V 70A, footprints:IPD047N03LF2SATMA1, symbol Device:Q_NMOS
- renumbered C119 to C110, D57 to D54, IC12 to IC11, R87 to R75, R88 to R76
Connections:
- net GND: now also Q16.3 (S); no longer D54.2 (A), R76.2
- net at R75.1: now also Q16.2 (G)
- new net: D54.2 (A), Q16.1 (D), R76.2
