File: hardware/electronics/core-pcb/motordriver.kicad_pcb (KiCad board)
At the start: 4 copper layers, 122 x 122 mm, 419 parts, among them IC1 LM5109BSDX_NOPB, IC10 LM5109BSDX_NOPB, IC11 INA2181A2IDGSR, IC12 LM5109BSDX_NOPB, IC13 LM5109BSDX_NOPB, IC14 LM5109BSDX_NOPB, IC15 LM5109BSDX_NOPB, IC16 INA2181A2IDGSR, IC2 LM5109BSDX_NOPB, IC3 LM5109BSDX_NOPB, IC4 INA2181A2IDGSR, IC5 BQ24133RGYR, IC6 LM5176PWPR, IC7 ATSAME53J18A-MF, IC8 LM5109BSDX_NOPB, IC9 LM5109BSDX_NOPB, J1 IMU1, J2 IMU2, J3 Conn_01x04_Socket, J4 XT60-M, J5 1-84952-1, J6 1-84952-1, J7 1-84952-1, P1 USB_C_Plug_USB2.0, Q1 30V 71A, Q10 30V 71A, Q11 30V 71A, Q12 30V 71A, Q13 30V 71A, Q14 30V 71A, Q15 30V 71A, Q16 30V 71A, Q17 30V 71A, Q18 30V 71A, Q19 30V 71A, Q2 30V 71A, Q20 30V 71A, Q21 30V 71A, Q22 30V 71A, Q23 30V 71A, Q24 30V 71A, Q25 30V 71A, Q26 30V 71A, Q3 30V 71A, Q4 30V 71A, Q5 30V 71A, Q6 30V 71A, Q7 30V 71A, Q8 30V 71A, Q9 40V 70A, SW1 PUSH, U1 LD1117S25TR_SOT223, U2 LD1117S33TR_SOT223, U3 LD1117S50TR_SOT223, U4 LD1117S50TR_SOT223, U5 TMC4671-LA, U6 ATSAMD11D14A-M, U7 TMC4671-LA, U8 TMC4671-LA, Y1 DSC6001CI2B-025.0000T

Commit message: started work on pcbv2 work in progress
Parts:
- removed L2: 1µH 22A, kuben-footprints:INDPM6965X300N
- removed the Q20 at (182.2, 125.5)
- added Q16: NMOS 30V 70A, footprints:IPD047N03LF2SATMA1, B.Cu at (182.7, 126.1)
- C17: renamed from C21; value 0.047µF -> 47nF
- C22: value 100nF -> 10µF
- C26: value 10uF -> 220µF 35V
- C30: value 10nF -> 100nF
- C32: value 33nF -> 100nF
- C33: value 470pF -> 100nF
- C34: value 15nF -> 100pF
- C36: value 220pF -> 100nF
- C37: value 100nF -> 100pF
- D7: value 4.7Vf 0.5A -> PWR; footprint kuben-footprints:DIOC1709X85N -> Diode_SMD:D_0603_1608Metric
- IC6: value LM5176PWPR -> ATSAME53J18A-MF
- Q7, Q8: value 30V 71A -> NMOS 30V 70A
- Q9: value 40V 70A -> PMOS 40V 70A
- R28: value 10Ω -> 1kΩ
- R30: value 240kΩ -> 5.1kΩ
- R31: value 133kΩ -> 10kΩ
- R32: value 93.1kΩ -> 4.7kΩ
- R33: value 2kΩ -> 4.7kΩ
- R34: value 280kΩ -> 4.7kΩ
- R35: value 20kΩ -> 1kΩ
- R36: value 10kΩ -> 1kΩ
- R37: value 9.09kΩ -> 1kΩ
- R38: value 23.2kΩ -> 10kΩ
- R39: value 2mΩ -> 1kΩ
- R60: value 1kΩ -> 10kΩ
- U3: value LD1117S50TR_SOT223 -> LD1117S25TR_SOT223
- renumbered C12 to C10, C109 to C100, C110 to C101, C111 to C102, C112 to C103, C113 to C104, C114 to C105, C115 to C106, C116 to C107, C117 to C108, C118 to C109, C119 to C110, C120 to C111, C121 to C112, C122 to C113, C123 to C114, C124 to C115, C125 to C116, C126 to C117, C127 to C118, C128 to C119, C14 to C12, C129 to C120, C130 to C121, C131 to C122, C132 to C123, C133 to C124, C134 to C125, C135 to C126, C136 to C127, C137 to C128, C138 to C129, C15 to C13, C139 to C130, C140 to C131, C141 to C132, C142 to C133, C143 to C134, C144 to C135, C145 to C136, C146 to C137, C147 to C138, C148 to C139, C17 to C14, C149 to C140, C150 to C141, C151 to C142, C152 to C143, C153 to C144, C154 to C145, C155 to C146, C18 to C15, C19 to C16, C23 to C18, C24 to C19, C25 to C20, C27 to C21, C29 to C22, C28 to C23, C16 to C24, C31 to C25, C38 to C26, C20 to C27, C10 to C28, C13 to C29, C39 to C30, C40 to C31, C41 to C32, C42 to C33, C43 to C34, C44 to C35, C45 to C36, C46 to C37, C47 to C38, C48 to C39, C49 to C40, C50 to C41, C51 to C42, C52 to C43, C53 to C44, C54 to C45, C55 to C46, C56 to C47, C57 to C48, C58 to C49, C59 to C50, C60 to C51, C61 to C52, C62 to C53, C63 to C54, C64 to C55, C65 to C56, C66 to C57, C67 to C58, C68 to C59, C69 to C60, C70 to C61, C71 to C62, C72 to C63, C73 to C64, C74 to C65, C75 to C66, C76 to C67, C77 to C68, C78 to C69, C79 to C70, C80 to C71, C81 to C72, C82 to C73, C83 to C74, C84 to C75, C85 to C76, C86 to C77, C87 to C78, C88 to C79, C89 to C80, C90 to C81, C91 to C82, C92 to C83, C93 to C84, C94 to C85, C95 to C86, C96 to C87, C97 to C88, C98 to C89, C99 to C90, C100 to C91, C101 to C92, C102 to C93, C103 to C94, C104 to C95, C105 to C96, C106 to C97, C107 to C98, C108 to C99, D13 to D10, D14 to D11, D15 to D12, D16 to D13, D17 to D14, D18 to D15, D19 to D16, D20 to D17, D21 to D18, D22 to D19, D23 to D20, D24 to D21, D25 to D22, D26 to D23, D27 to D24, D28 to D25, D29 to D26, D30 to D27, D31 to D28, D32 to D29, D33 to D30, D34 to D31, D35 to D32, D36 to D33, D37 to D34, D38 to D35, D39 to D36, D40 to D37, D41 to D38, D42 to D39, D43 to D40, D44 to D41, D45 to D42, D46 to D43, D47 to D44, D48 to D45, D49 to D46, D50 to D47, D51 to D48, D52 to D49, D53 to D50, D54 to D51, D55 to D52, D56 to D53, D57 to D54, D58 to D55, D59 to D56, D60 to D57, D61 to D58, D62 to D59, D63 to D60, D64 to D61, D65 to D62, D66 to D63, D67 to D64, D68 to D65, D69 to D66, D70 to D67, D71 to D68, D72 to D69, D8 to D7, D73 to D70, D74 to D71, D75 to D72, D76 to D73, D77 to D74, D78 to D75, D11 to D8, D12 to D9, IC11 to IC10, IC12 to IC11, IC13 to IC12, IC14 to IC13, IC15 to IC14, IC16 to IC15, IC7 to IC6, IC8 to IC7, IC9 to IC8, IC10 to IC9, Q14 to Q10, Q15 to Q11, Q16 to Q12, Q17 to Q13, Q18 to Q14, Q19 to Q15, Q21 to Q17, Q22 to Q18, Q23 to Q19, Q24 to Q20, Q25 to Q21, Q26 to Q22, R19 to R17, R17 to R18, R18 to R19, R29 to R28, R40 to R29, R41 to R30, R42 to R31, R43 to R32, R44 to R33, R45 to R34, R46 to R35, R47 to R36, R48 to R37, R49 to R38, R50 to R39, R51 to R40, R52 to R41, R53 to R42, R54 to R43, R55 to R44, R56 to R45, R57 to R46, R58 to R47, R59 to R48, R61 to R49, R62 to R50, R63 to R51, R64 to R52, R65 to R53, R66 to R54, R67 to R55, R68 to R56, R69 to R57, R70 to R58, R71 to R59, R72 to R60, R73 to R61, R74 to R62, R75 to R63, R76 to R64, R77 to R65, R78 to R66, R79 to R67, R80 to R68, R81 to R69, R82 to R70, R83 to R71, R84 to R72, R85 to R73, R86 to R74, R87 to R75, R89 to R77, R90 to R78, R91 to R79, R92 to R80, R93 to R81, R94 to R82, R95 to R83, R96 to R84, R97 to R85, R98 to R86, R99 to R87, R100 to R88, R101 to R89, R102 to R90, R103 to R91, R104 to R92, R105 to R93, R106 to R94, R107 to R95, R108 to R96, R109 to R97, R110 to R98, R111 to R99, U4 to U1, U1 to U3, U5 to U4, U6 to U5, U7 to U6, U8 to U7
Connections:
- net /voltageregulators/IC5_VREF renamed Net-(IC5-CELL)
- net /voltageregulators/OVPSET renamed Net-(IC5-OVPSET)
- net Net-(IC5-ACDRV) renamed /voltageregulators/ACDRV
- net Net-(IC5-CMSRC) renamed /voltageregulators/CMSRC
- net Net-(IC7-PB30) renamed /microcontrollers/SWO
- C12 pad 1: Net-(D7-A) -> Net-(IC5-PVCC_1)
- C14 pad 1: Net-(IC5-ACP) -> Net-(Q7-S)
- C14 pad 2: Net-(D7-A) -> /voltageregulators/ACP
- C16 pad 1: Net-(D7-A) -> /voltageregulators/ACP
- C20 pad 2: /IO/BATTVIN -> BATTERY_P
- C21 pad 1: /IO/BATTVIN -> BATTERY_P
- C22 pad 1: +12V -> BATTERY_P
- C22 pad 1: /IO/BATTVIN -> BATTERY_P
- C26 pad 1: +5V -> +12V
- C30 pad 1: Net-(IC6-VIN) -> GND
- C30 pad 2: GND -> +3.3V
- C32 pad 2: Net-(C32-Pad2) -> +3.3V
- C33 pad 2: /voltageregulators/COMP -> +3.3V
- C34 pad 2: /voltageregulators/SS -> /servo1/HALL_U_FILT
- C35 pad 1: /voltageregulators/BOOT1 -> GND
- C35 pad 2: /voltageregulators/SW1 -> +3.3V
- C36 pad 2: Net-(U5-VCCCORE3) -> Net-(U4-VCCCORE3)
- C36 pad 2: /voltageregulators/SLOPE -> Net-(U4-VCCCORE3)
- C37 pad 1: /voltageregulators/SW2 -> GND
- C37 pad 2: /voltageregulators/BOOT2 -> /servo1/HALL_V_FILT
- C72 pad 1: /IO/RESETN -> /microcontrollers/RESETN
- C87 pad 1: Net-(U7-NRST) (its old number) -> Net-(U6-NRST)
- D10 pad 1: /voltageregulators/BOOT1 -> +5VA
- D10 pad 2: /voltageregulators/VCC -> /servo1/ADC_I1_POS
- D20 pad 2: Net-(D23-A) (its old number) -> Net-(D20-A)
- D4 pad 2: /IO/BATTVIN -> BATTERY_P
- D54 pad 2: GND -> Net-(D54-A)
- D7 pad 1: Net-(D7-K) -> GND
- D7 pad 2: Net-(D8-A) -> Net-(D7-A)
- D9 pad 1: /voltageregulators/BOOT2 -> /servo1/ADC_I0_POS
- D9 pad 2: /voltageregulators/VCC -> GND
- IC10 pad 3: Net-(IC11-IN+1) -> Net-(IC10-IN+1)
- IC10 pad 7: Net-(IC11-IN+2) -> Net-(IC10-IN+2)
- IC5 pad 15: /IO/BATTVIN -> BATTERY_P
- IC5 pad 19: Net-(IC5-~{BATDRV}) -> Net-(IC5-SRP)
- IC5 pad 2: Net-(D7-A) -> Net-(IC5-PVCC_1)
- IC5 pad 3: Net-(D7-A) -> Net-(IC5-PVCC_1)
- IC5 pad 5: Net-(D7-A) -> /voltageregulators/ACP
- IC5 pad 6: Net-(IC5-ACP) -> /voltageregulators/ACP
- IC6 pad 11: unconnected-(IC7-PB08-Pad11) -> unconnected-(IC6-PB08-Pad11)
- IC6 pad 12: unconnected-(IC7-PB09-Pad12) -> unconnected-(IC6-PB09-Pad12)
- IC6 pad 13: unconnected-(IC7-PA04-Pad13) -> unconnected-(IC6-PA04-Pad13)
- IC6 pad 14: unconnected-(IC7-PA05-Pad14) -> unconnected-(IC6-PA05-Pad14)
- IC6 pad 15: unconnected-(IC7-PA06-Pad15) -> unconnected-(IC6-PA06-Pad15)
- IC6 pad 16: unconnected-(IC7-PA07-Pad16) -> unconnected-(IC6-PA07-Pad16)
- IC6 pad 19: unconnected-(IC7-PA10-Pad19) -> unconnected-(IC6-PA10-Pad19)
- IC6 pad 20: unconnected-(IC7-PA11-Pad20) -> unconnected-(IC6-PA11-Pad20)
- IC6 pad 23: unconnected-(IC7-PB10-Pad23) -> unconnected-(IC6-PB10-Pad23)
- IC6 pad 28: unconnected-(IC7-PB15-Pad28) -> unconnected-(IC6-PB15-Pad28)
- IC6 pad 52: /IO/RESETN -> /microcontrollers/RESETN
- IC6 pad 57: Net-(IC7-PA30) -> /microcontrollers/CLK
- IC6 pad 58: Net-(IC7-PA31) -> /microcontrollers/DIO
- IC6 pad 1: Net-(IC6-EN/UVLO) -> /microcontrollers/PROCLED
- IC6 pad 10: GND -> /IO/INT_IMU2
- IC6 pad 11: Net-(IC6-FB) -> unconnected-(IC6-PB08-Pad11)
- IC6 pad 12: +12V -> unconnected-(IC6-PB09-Pad12)
- IC6 pad 13: GND -> unconnected-(IC6-PA04-Pad13)
- IC6 pad 14: GND -> unconnected-(IC6-PA05-Pad14)
- IC6 pad 15: GND -> unconnected-(IC6-PA06-Pad15)
- IC6 pad 16: Net-(IC6-CS) -> unconnected-(IC6-PA07-Pad16)
- IC6 pad 17: /voltageregulators/PGOOD -> /IO/SDA_IMU1
- IC6 pad 18: /voltageregulators/SW2 -> /IO/SCL_IMU1
- IC6 pad 19: /voltageregulators/HDRV2 -> unconnected-(IC6-PA10-Pad19)
- IC6 pad 2: Net-(IC6-VIN) -> /microcontrollers/ERRLED
- IC6 pad 20: /voltageregulators/BOOT2 -> unconnected-(IC6-PA11-Pad20)
- IC6 pad 21: /voltageregulators/LDRV2 -> +3.3V
- IC6 pad 23: /voltageregulators/VCC -> unconnected-(IC6-PB10-Pad23)
- IC6 pad 24: +12V -> SERVO_ENI
- IC6 pad 25: /voltageregulators/LDRV1 -> TMC_DB_MISO
- IC6 pad 26: /voltageregulators/BOOT1 -> TMC_DB_MOSI
- IC6 pad 27: /voltageregulators/HDRV1 -> TMC_DB_SCK
- IC6 pad 28: /voltageregulators/SW1 -> unconnected-(IC6-PB15-Pad28)
- IC6 pad 29: unconnected-(IC6-EPAD-Pad29) -> /IO/OLED_SDA
- IC6 pad 3: Net-(IC6-VISNS) -> /microcontrollers/SERVO1_DB_CS
- IC6 pad 4: Net-(IC6-MODE) -> /microcontrollers/SERVO1_STATUS
- IC6 pad 5: GND -> /microcontrollers/SERVO2_STATUS
- IC6 pad 6: /voltageregulators/RT -> /microcontrollers/SERVO3_STATUS
- IC6 pad 7: /voltageregulators/SLOPE -> GND
- IC6 pad 8: /voltageregulators/SS -> +3.3V
- IC6 pad 9: /voltageregulators/COMP -> /IO/INT_IMU1
- J4 pad P: /IO/BATTVIN -> BATTERY_P
- Q10 pad 1: /voltageregulators/HDRV1 -> Net-(Q10-G)
- Q10 pad 2: Net-(D7-A) -> +12V
- Q10 pad 3: /voltageregulators/SW1 -> Net-(IC10-IN+1)
- Q10 pad 1: Net-(Q14-G) (its old number) -> Net-(Q10-G)
- Q10 pad 3: Net-(IC11-IN+1) -> Net-(IC10-IN+1)
- Q11 pad 1: /voltageregulators/LDRV1 -> Net-(Q11-G)
- Q11 pad 2: /voltageregulators/SW1 -> Net-(IC10-IN+1)
- Q11 pad 3: Net-(IC6-CS) -> GND
- Q11 pad 1: Net-(Q15-G) (its old number) -> Net-(Q11-G)
- Q11 pad 2: Net-(IC11-IN+1) -> Net-(IC10-IN+1)
- Q12 pad 1: /voltageregulators/HDRV2 -> Net-(Q12-G)
- Q12 pad 3: /voltageregulators/SW2 -> Net-(IC10-IN+2)
- Q12 pad 1: Net-(Q16-G) (its old number) -> Net-(Q12-G)
- Q12 pad 3: Net-(IC11-IN+2) -> Net-(IC10-IN+2)
- Q13 pad 1: /voltageregulators/LDRV2 -> Net-(Q13-G)
- Q13 pad 2: /voltageregulators/SW2 -> Net-(IC10-IN+2)
- Q13 pad 3: Net-(IC6-CS) -> GND
- Q13 pad 1: Net-(Q17-G) (its old number) -> Net-(Q13-G)
- Q13 pad 2: Net-(IC11-IN+2) -> Net-(IC10-IN+2)
- Q7 pad 1: Net-(Q7-G) -> /IO/USBVIN
- Q7 pad 2: /IO/USBVIN -> Net-(Q7-G)
- Q7 pad 3: Net-(IC5-ACP) -> Net-(Q7-S)
- Q8 pad 1: Net-(Q7-G) -> unconnected-(Q8-D-Pad1)
- Q8 pad 2: Net-(IC5-ACP) -> Net-(Q7-G)
- Q8 pad 3: Net-(IC5-ACP) -> Net-(Q7-S)
- Q9 pad 2: /IO/BATTVIN -> BATTERY_P
- Q9 pad 3: Net-(D7-A) -> unconnected-(Q9-S-Pad3)
- R13 pad 1: Net-(C11-Pad1) -> /IO/USBVIN
- R13 pad 2: /IO/USBVIN -> Net-(C11-Pad1)
- R20 pad 2: Net-(IC5-ACP) -> Net-(Q7-S)
- R21 pad 1: Net-(D7-A) -> /voltageregulators/ACP
- R21 pad 2: Net-(IC5-ACP) -> Net-(Q7-S)
- R26 pad 2: Net-(IC5-~{BATDRV}) -> Net-(IC5-SRP)
- R27 pad 1: /IO/BATTVIN -> BATTERY_P
- R28 pad 1: Net-(IC6-VIN) -> Net-(D7-A)
- R28 pad 2: Net-(D7-K) -> +3.3V
- R28 pad 1: Net-(D8-A) -> Net-(D7-A)
- R30 pad 1: Net-(IC6-EN/UVLO) -> GND
- R30 pad 2: Net-(D7-A) -> Net-(P1-PadB5)
- R31 pad 2: /IO/RESETN -> /microcontrollers/RESETN
- R31 pad 1: GND -> +3.3V
- R31 pad 2: Net-(IC6-EN/UVLO) -> /microcontrollers/RESETN
- R32 pad 1: GND -> +5VA
- R32 pad 2: Net-(IC6-MODE) -> /motorIO/HALL_A3
- R33 pad 1: Net-(IC6-VISNS) -> +5VA
- R33 pad 2: Net-(D7-A) -> /motorIO/HALL_B3
- R34 pad 1: Net-(IC6-FB) -> +5VA
- R34 pad 2: +12V -> /motorIO/HALL_C3
- R35 pad 1: GND -> /motorIO/HALL_C3
- R35 pad 2: Net-(IC6-FB) -> /servo1/HALL_W_FILT
- R36 pad 1: /voltageregulators/VCC -> /motorIO/HALL_B3
- R36 pad 2: /voltageregulators/PGOOD -> /servo1/HALL_V_FILT
- R37 pad 1: Net-(C32-Pad2) -> /motorIO/HALL_A3
- R37 pad 2: /voltageregulators/COMP -> /servo1/HALL_U_FILT
- R38 pad 1: GND -> SERVO_ENI
- R38 pad 2: /voltageregulators/RT -> GND
- R39 pad 1: Net-(D23-A) (its old number) -> Net-(D20-A)
- R39 pad 2: Net-(U5-GPIO2_/_ADC_VM_MCD) -> Net-(U4-GPIO2_/_ADC_VM_MCD)
- R39 pad 1: GND -> Net-(D20-A)
- R39 pad 2: Net-(IC6-CS) -> Net-(U4-GPIO2_/_ADC_VM_MCD)
- R42 pad 1: +12V -> BATTERY_P
- R60 pad 1: Net-(IC7-PA31) -> Net-(U6-NRST)
- R60 pad 1: Net-(U7-NRST) (its old number) -> Net-(U6-NRST)
- R62 pad 1: +12V -> BATTERY_P
- R68 pad 2: Net-(Q16-G) (its old number) -> Net-(Q12-G)
- R69 pad 1: Net-(Q17-G) (its old number) -> Net-(Q13-G)
- R71 pad 2: Net-(Q14-G) (its old number) -> Net-(Q10-G)
- R72 pad 1: Net-(Q15-G) (its old number) -> Net-(Q11-G)
- R73 pad 2: Net-(IC11-IN+1) -> Net-(IC10-IN+1)
- R74 pad 2: Net-(IC11-IN+2) -> Net-(IC10-IN+2)
- R87 pad 1: +12V -> BATTERY_P
- SW1 pad 1: /IO/RESETN -> /microcontrollers/RESETN
- U3 pad 2: +5V -> +2.5V
- U4 pad 63: Net-(U5-VCCCORE3) -> Net-(U4-VCCCORE3)
- U4 pad 74: Net-(U5-GPIO2_/_ADC_VM_MCD) -> Net-(U4-GPIO2_/_ADC_VM_MCD)
- U5 pad 3: Net-(IC7-PA30) -> /microcontrollers/DIO
- U5 pad 4: /IO/RESETN -> /microcontrollers/RESETN
- U5 pad 7: Net-(IC7-PA31) -> /microcontrollers/CLK
- U6 pad 50: Net-(U7-NRST) (its old number) -> Net-(U6-NRST)
Routing:
- net (no net): track 0.00 -> 533.2 mm, vias 0 -> 2
- net /IO/RESETN: track 81.7 -> 0.00 mm, vias 4 -> 0
- net GND: track 590.8 -> 672.5 mm, vias 183 -> 187
- net BATTERY_P: track 0.00 -> 77.9 mm
- net /IO/BATTVIN: track 77.9 -> 0.00 mm
- net Net-(IC7-PA31): track 76.2 -> 0.00 mm, vias 2 -> 0
- net Net-(IC7-PA30): track 68.7 -> 0.00 mm, vias 2 -> 0
- net Net-(IC5-ACP): track 49.0 -> 0.00 mm
- net Net-(IC11-IN+2): track 44.6 -> 0.00 mm, vias 2 -> 0
- net Net-(IC10-IN+2): track 0.00 -> 44.6 mm, vias 0 -> 6
- net Net-(D7-K): track 38.4 -> 0.00 mm
- net /voltageregulators/HDRV2: track 35.3 -> 0.00 mm
- net Net-(IC6-EN/UVLO): track 31.1 -> 0.00 mm
- net /voltageregulators/SW2: track 28.3 -> 0.00 mm, vias 4 -> 0
- net Net-(IC5-~{BATDRV}): track 27.6 -> 0.00 mm
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- added copper zone on F.Cu, net BATTERY_P
- added copper zone on F.Cu, net GND
- added copper zone on F.Cu, net Net-(IC10-IN+1)
- added copper zone on F.Cu, net Net-(IC10-IN+2)
- removed copper zone on F.Cu, net /IO/BATTVIN
- removed copper zone on F.Cu, net /voltageregulators/SW1
- removed copper zone on F.Cu, net /voltageregulators/SW2
- removed copper zone on F.Cu, net Net-(IC6-CS)
