File: hardware/electronics/core-pcb/servocontroller.kicad_sch (KiCad schematic)
At the start: 59 parts, among them U5 TMC4671-LA

Commit message: started work on pcbv2 work in progress
Parts:
- renumbered C39 to C30, C40 to C31, C41 to C32, C42 to C33, C43 to C34, C44 to C35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
Connections:
- net +12V renamed BATTERY_P
Other:
- moved on the sheet: C55, C57
